File: hardware/mcphail-photodiode-emitter/mcphail-photodiode-emitter.kicad_pcb (KiCad board)
At the start: 2 copper layers, 0 parts

Commit message: Updated README to include hardware design notes.
Other:
- board outline added: 76 x 11 mm
- rule trace_clearance: 0.1524 -> 0.254
Changed lines of the file:
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@@
-(kicad_pcb (version 4) (host pcbnew 4.0.4+e1-6308~48~ubuntu14.04.1-stable)
+(kicad_pcb (version 4) (host pcbnew 4.0.5-e0-6337~49~ubuntu16.04.1)
   (general
     (links 0)
@@
     (area 104.572999 74.854999 178.510001 123.265001)
     (thickness 1.6)
-    (drawings 17)
+    (drawings 61)
     (tracks 0)
     (zones 0)
@@
     (title "McPhail Trap Photodiode Emitter Board")
     (date "19 Jul 2017")
-    (rev "1.0")
+    (rev 1.0)
     (company "CERN Open Hardware License v1.2")
-    (comment 1 "jenner@wickerbox.net")
-    (comment 2 "http://wickerbox.net")
+    (comment 1 jenner@wickerbox.net)
+    (comment 2 http://wickerbox.net)
     (comment 3 "Wickerbox Electronics")
   )
@@
     (user_trace_width 0.762)
     (user_trace_width 1.27)
-    (trace_clearance 0.1524)
+    (trace_clearance 0.254)
     (zone_clearance 0.508)
     (zone_45_only no)
@@
     (uvia_drill 0.3302)
   )
+  (gr_line (start 180 103) (end 180 92) (layer Edge.Cuts) (width 0.1524))
+  (gr_line (start 104 103) (end 180 103) (layer Edge.Cuts) (width 0.1524))
+  (gr_line (start 104 92) (end 104 103) (layer Edge.Cuts) (width 0.1524))
+  (gr_line (start 180 92) (end 104 92) (layer Edge.Cuts) (width 0.1524))
+  (gr_line (start 109 95) (end 109 100) (layer F.Fab) (width 0.1524))
+  (gr_line (start 114 95) (end 109 95) (layer F.Fab) (width 0.1524))
+  (gr_line (start 114 100) (end 114 95) (layer F.Fab) (width 0.1524))
+  (gr_line (start 109 100) (end 114 100) (layer F.Fab) (width 0.1524))
+  (gr_line (start 116 95) (end 116 100) (layer F.Fab) (width 0.1524))
+  (gr_line (start 121 95) (end 116 95) (layer F.Fab) (width 0.1524))
+  (gr_line (start 121 100) (end 121 95) (layer F.Fab) (width 0.1524))
+  (gr_line (start 116 100) (end 121 100) (layer F.Fab) (width 0.1524))
+  (gr_line (start 123 95) (end 123 100) (layer F.Fab) (width 0.1524))
+  (gr_line (start 128 95) (end 123 95) (layer F.Fab) (width 0.1524))
+  (gr_line (start 128 100) (end 128 95) (layer F.Fab) (width 0.1524))
+  (gr_line (start 123 100) (end 128 100) (layer F.Fab) (width 0.1524))
+  (gr_line (start 172 95) (end 172 100) (layer F.Fab) (width 0.1524))
+  (gr_line (start 177 95) (end 172 95) (layer F.Fab) (width 0.1524))
+  (gr_line (start 177 100) (end 177 95) (layer F.Fab) (width 0.1524))
+  (gr_line (start 172 100) (end 177 100) (layer F.Fab) (width 0.1524))
+  (gr_line (start 165 95) (end 165 100) (layer F.Fab) (width 0.1524))
+  (gr_line (start 170 95) (end 165 95) (layer F.Fab) (width 0.1524))
+  (gr_line (start 170 100) (end 170 95) (layer F.Fab) (width 0.1524))
+  (gr_line (start 165 100) (end 170 100) (layer F.Fab) (width 0.1524))
+  (gr_line (start 158 95) (end 158 100) (layer F.Fab) (width 0.1524))
+  (gr_line (start 163 95) (end 158 95) (layer F.Fab) (width 0.1524))
+  (gr_line (start 163 100) (end 163 95) (layer F.Fab) (width 0.1524))
+  (gr_line (start 158 100) (end 163 100) (layer F.Fab) (width 0.1524))
+  (gr_line (start 151 95) (end 151 100) (layer F.Fab) (width 0.1524))
+  (gr_line (start 156 95) (end 151 95) (layer F.Fab) (width 0.1524))
+  (gr_line (start 156 100) (end 156 95) (layer F.Fab) (width 0.1524))
+  (gr_line (start 151 100) (end 156 100) (layer F.Fab) (width 0.1524))
+  (gr_line (start 144 95) (end 144 100) (layer F.Fab) (width 0.1524))
+  (gr_line (start 149 95) (end 144 95) (layer F.Fab) (width 0.1524))
+  (gr_line (start 149 100) (end 149 95) (layer F.Fab) (width 0.1524))
+  (gr_line (start 144 100) (end 149 100) (layer F.Fab) (width 0.1524))
+  (gr_line (start 137 95) (end 137 100) (layer F.Fab) (width 0.1524))
+  (gr_line (start 142 95) (end 137 95) (layer F.Fab) (width 0.1524))
+  (gr_line (start 142 100) (end 142 95) (layer F.Fab) (width 0.1524))
+  (gr_line (start 137 100) (end 142 100) (layer F.Fab) (width 0.1524))
+  (gr_line (start 130 95) (end 130 100) (layer F.Fab) (width 0.1524))
+  (gr_line (start 135 95) (end 130 95) (layer F.Fab) (width 0.1524))
+  (gr_line (start 135 100) (end 135 95) (layer F.Fab) (width 0.1524))
+  (gr_line (start 130 100) (end 135 100) (layer F.Fab) (width 0.1524))
   (gr_circle (center 117.348 76.962) (end 118.618 76.962) (layer Dwgs.User) (width 0.15))
   (gr_line (start 114.427 78.994) (end 114.427 74.93) (angle 90) (layer Dwgs.User) (width 0.15))
