File: hardware/mcphail-photodiode-detector-board/mcphail-photodiode-detector-board.sch (KiCad schematic (older format))
At the start: 11 parts, among them J1 TO MCU

Commit message: Release v1.0 Mcphail IR 940nm Emitter Board.
Parts:
- J1: footprint CONN-1x02-2.54MM-TH -> Wickerlib:CONN-HEADER-STRAIGHT-P2.54MM-1x02
- LED1, LED10, LED2, LED3, LED4, LED5, LED6, LED7, LED8, LED9: footprint Wickerlib:LED-D5MM-2PIN -> Wickerlib:TEMD5110X01
Connections:
- net A: now reaches J1.1 (P1), LED1.2, LED10.2, LED2.2, LED3.2, LED4.2, LED5.2, LED6.2, LED7.2, LED8.2, LED9.2
- net K: now reaches J1.2 (P2), LED1.1, LED10.1, LED2.1, LED3.1, LED4.1, LED5.1, LED6.1, LED7.1, LED8.1, LED9.1
Changed lines of the file:
@@
 EESchema Schematic File Version 2
 LIBS:wickerlib
+LIBS:mcphail-photodiode-detector-board-cache
 EELAYER 25 0
 EELAYER END
@@
 F 0 "J1" H 2150 3950 50  0000 L CNN
 F 1 "TO MCU" H 2150 3650 50  0000 L CNN
-F 2 "CONN-1x02-2.54MM-TH" H 2250 3450 50  0001 C CIN
+F 2 "Wickerlib:CONN-HEADER-STRAIGHT-P2.54MM-1x02" H 2250 3450 50  0001 C CIN
 F 3 "https://cdn.harwin.com/pdfs/60page140.pdf" H 2200 3800 5   0001 C CNN
 F 4 "HEADER MALE 2POS TH 1x02 0.1IN" H 2250 3450 50  0001 C CIN "Description"
@@
 F 0 "LED1" H 2925 3875 50  0000 L CNN
 F 1 "940NM" H 2925 3775 50  0000 L CNN
-F 2 "Wickerlib:LED-D5MM-2PIN" H 2850 3450 50  0001 C CIN
+F 2 "Wickerlib:TEMD5110X01" H 2850 3450 50  0001 C CIN
 F 3 "http://www.vishay.com/docs/84658/temd5110.pdf" V 2850 3800 5   0001 C CNN
 F 4 "PHOTODIODE IR 940NM SMD TEMD5110X01" H 2850 3450 50  0001 C CIN "Description"
@@
 F 0 "LED2" H 3350 3875 50  0000 L CNN
 F 1 "940NM" H 3350 3775 50  0000 L CNN
-F 2 "Wickerlib:LED-D5MM-2PIN" H 3275 3450 50  0001 C CIN
+F 2 "Wickerlib:TEMD5110X01" H 3275 3450 50  0001 C CIN
 F 3 "http://www.vishay.com/docs/84658/temd5110.pdf" V 3275 3800 5   0001 C CNN
 F 4 "PHOTODIODE IR 940NM SMD TEMD5110X01" H 3275 3450 50  0001 C CIN "Description"
@@
 F 0 "LED3" H 3750 3875 50  0000 L CNN
 F 1 "940NM" H 3750 3775 50  0000 L CNN
-F 2 "Wickerlib:LED-D5MM-2PIN" H 3675 3450 50  0001 C CIN
+F 2 "Wickerlib:TEMD5110X01" H 3675 3450 50  0001 C CIN
 F 3 "http://www.vishay.com/docs/84658/temd5110.pdf" V 3675 3800 5   0001 C CNN
 F 4 "PHOTODIODE IR 940NM SMD TEMD5110X01" H 3675 3450 50  0001 C CIN "Description"
@@
 F 0 "LED4" H 4150 3875 50  0000 L CNN
 F 1 "940NM" H 4150 3775 50  0000 L CNN
-F 2 "Wickerlib:LED-D5MM-2PIN" H 4075 3450 50  0001 C CIN
+F 2 "Wickerlib:TEMD5110X01" H 4075 3450 50  0001 C CIN
 F 3 "http://www.vishay.com/docs/84658/temd5110.pdf" V 4075 3800 5   0001 C CNN
 F 4 "PHOTODIODE IR 940NM SMD TEMD5110X01" H 4075 3450 50  0001 C CIN "Description"
@@
 F 0 "LED5" H 4550 3875 50  0000 L CNN
 F 1 "940NM" H 4550 3775 50  0000 L CNN
-F 2 "Wickerlib:LED-D5MM-2PIN" H 4475 3450 50  0001 C CIN
+F 2 "Wickerlib:TEMD5110X01" H 4475 3450 50  0001 C CIN
 F 3 "http://www.vishay.com/docs/84658/temd5110.pdf" V 4475 3800 5   0001 C CNN
 F 4 "PHOTODIODE IR 940NM SMD TEMD5110X01" H 4475 3450 50  0001 C CIN "Description"
@@
 F 0 "LED6" H 4950 3875 50  0000 L CNN
 F 1 "940NM" H 4950 3775 50  0000 L CNN
-F 2 "Wickerlib:LED-D5MM-2PIN" H 4875 3450 50  0001 C CIN
+F 2 "Wickerlib:TEMD5110X01" H 4875 3450 50  0001 C CIN
 F 3 "http://www.vishay.com/docs/84658/temd5110.pdf" V 4875 3800 5   0001 C CNN
 F 4 "PHOTODIODE IR 940NM SMD TEMD5110X01" H 4875 3450 50  0001 C CIN "Description"
@@
 F 0 "LED7" H 5325 3875 50  0000 L CNN
 F 1 "940NM" H 5325 3775 50  0000 L CNN
-F 2 "Wickerlib:LED-D5MM-2PIN" H 5250 3450 50  0001 C CIN
+F 2 "Wickerlib:TEMD5110X01" H 5250 3450 50  0001 C CIN
 F 3 "http://www.vishay.com/docs/84658/temd5110.pdf" V 5250 3800 5   0001 C CNN
 F 4 "PHOTODIODE IR 940NM SMD TEMD5110X01" H 5250 3450 50  0001 C CIN "Description"
@@
 F 0 "LED8" H 5750 3875 50  0000 L CNN
 F 1 "940NM" H 5750 3775 50  0000 L CNN
-F 2 "Wickerlib:LED-D5MM-2PIN" H 5675 3450 50  0001 C CIN
+F 2 "Wickerlib:TEMD5110X01" H 5675 3450 50  0001 C CIN
 F 3 "http://www.vishay.com/docs/84658/temd5110.pdf" V 5675 3800 5   0001 C CNN
 F 4 "PHOTODIODE IR 940NM SMD TEMD5110X01" H 5675 3450 50  0001 C CIN "Description"
@@
 F 0 "LED9" H 6125 3875 50  0000 L CNN
 F 1 "940NM" H 6125 3775 50  0000 L CNN
-F 2 "Wickerlib:LED-D5MM-2PIN" H 6050 3450 50  0001 C CIN
+F 2 "Wickerlib:TEMD5110X01" H 6050 3450 50  0001 C CIN
 F 3 "http://www.vishay.com/docs/84658/temd5110.pdf" V 6050 3800 5   0001 C CNN
 F 4 "PHOTODIODE IR 940NM SMD TEMD5110X01" H 6050 3450 50  0001 C CIN "Description"
@@
 F 0 "LED10" H 6550 3875 50  0000 L CNN
 F 1 "940NM" H 6550 3775 50  0000 L CNN
-F 2 "Wickerlib:LED-D5MM-2PIN" H 6475 3450 50  0001 C CIN
+F 2 "Wickerlib:TEMD5110X01" H 6475 3450 50  0001 C CIN
 F 3 "http://www.vishay.com/docs/84658/temd5110.pdf" V 6475 3800 5   0001 C CNN
 F 4 "PHOTODIODE IR 940NM SMD TEMD5110X01" H 6475 3450 50  0001 C CIN "Description"
@@
 $EndComp
 Wire Wire Line
-	6475 3700 6475 3575
-Wire Wire Line
-	6475 3575 6050 3575
-Wire Wire Line
-	6050 3575 5675 3575
-Wire Wire Line
-	5675 3575 5250 3575
-Wire Wire Line
-	5250 3575 4875 3575
-Wire Wire Line
-	4875 3575 4475 3575
-Wire Wire Line
-	4475 3575 4075 3575
-Wire Wire Line
-	4075 3575 3675 3575
-Wire Wire Line
-	3675 3575 3275 3575
-Wire Wire Line
-	3275 3575 2850 3575
-Wire Wire Line
-	2850 3575 2575 3575
+	6475 3575 6475 3700
+Wire Wire Line
+	2575 3575 6475 3575
 Wire Wire Line
 	2575 3575 2575 3750
@@
 	2575 3850 2575 4025
 Wire Wire Line
-	2575 4025 2850 4025
-Wire Wire Line
-	2850 4025 3275 4025
-Wire Wire Line
-	3275 4025 3675 4025
-Wire Wire Line
-	3675 4025 4075 4025
-Wire Wire Line
-	4075 4025 4475 4025
-Wire Wire Line
-	4475 4025 4875 4025
-Wire Wire Line
-	4875 4025 5250 4025
-Wire Wire Line
-	5250 4025 5675 4025
-Wire Wire Line
-	5675 4025 6050 4025
-Wire Wire Line
-	6050 4025 6475 4025
+	2575 4025 6475 4025
 Wire Wire Line
 	6475 4025 6475 3900
@@
 	6050 3900 6050 4025
 Connection ~ 6050 4025
+Text Label 2450 3750 0    50   ~ 0
+A
+Text Label 2450 3850 0    50   ~ 0
+K
 $EndSCHEMATC
