File: hardware/mcphail-photodiode-detector-board/mcphail-photodiode-detector-board.kicad_pcb (KiCad board)
At the start: 2 copper layers, 0 parts

Commit message: Release v1.0 Mcphail IR 940nm Emitter Board.
Parts:
- added J1: TO MCU, Wickerlib:CONN-HEADER-STRAIGHT-P2.54MM-1x02, F.Cu at (97.8, 89.0)
- added LED1: 940NM, Wickerlib:TEMD5110X01, F.Cu at (105.0, 90.0)
- added LED10: 940NM, Wickerlib:TEMD5110X01, F.Cu at (159.0, 90.0)
- added LED2: 940NM, Wickerlib:TEMD5110X01, F.Cu at (111.0, 90.0)
- added LED3: 940NM, Wickerlib:TEMD5110X01, F.Cu at (117.0, 90.0)
- added LED4: 940NM, Wickerlib:TEMD5110X01, F.Cu at (123.0, 90.0)
- added LED5: 940NM, Wickerlib:TEMD5110X01, F.Cu at (129.0, 90.0)
- added LED6: 940NM, Wickerlib:TEMD5110X01, F.Cu at (135.0, 90.0)
- added LED7: 940NM, Wickerlib:TEMD5110X01, F.Cu at (141.0, 90.0)
- added LED8: 940NM, Wickerlib:TEMD5110X01, F.Cu at (147.0, 90.0)
- added LED9: 940NM, Wickerlib:TEMD5110X01, F.Cu at (153.0, 90.0)
Routing:
- net /A: track 0.00 -> 61.7 mm
- net /K: track 0.00 -> 61.2 mm
Other:
- board outline added: 68.6 x 12.7 mm
- rule trace_clearance: 0.1524 -> 0.254
- board text added: "+"
- board text added: "-"
- board text added: "940nm Photodiode Receiver Board v1.0"

Commit message: Release v1.0 McPhail Photodiode Detector Board
Parts:
- moved J1 59.5 mm to (38.7, 96.0)
- moved LED1 59.5 mm to (45.9, 97.0)
- moved LED10 59.5 mm to (99.9, 97.0)
- moved LED2 59.5 mm to (51.9, 97.0)
- moved LED3 59.5 mm to (57.9, 97.0)
- moved LED4 59.5 mm to (63.9, 97.0)
- moved LED5 59.5 mm to (69.9, 97.0)
- moved LED6 59.5 mm to (75.9, 97.0)
- moved LED7 59.5 mm to (81.9, 97.0)
- moved LED8 59.5 mm to (87.9, 97.0)
- moved LED9 59.5 mm to (93.9, 97.0)
Other:
- board text added: "FABRICATION NOTES 1. THIS IS A 2 LAYER BOARD. 2. EXTERNAL LAYERS SHALL HAVE 1 OZ COPPER. 3. MATERIAL: FR4 AND 0.062 INCH +/- 10% THICK. 4. BOARDS SHALL BE ROHS COMPLIANT. 5. MANUFACTURE IN ACCORDANCE WITH IPC-6012 CLASS 2 6. MASK: BOTH SIDES OF THE BOARD SHALL HAVE SOLDER MASK (ANY COLOR) OVER BARE COPPER. 7. SILK: BOTH SIDES OF THE BOARD SHALL HAVE WHITE SILKSCREEN. DO NOT PLACE SILK OVER BARE C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"
