File: hardware/mcphail-ir-emitter-board/mcphail-ir-emitter-board.sch (KiCad schematic (older format))
At the start: 11 parts, among them J1 TO MCU

Commit message: Release v1.0 Mcphail IR 940nm Emitter Board.
Parts:
- J1: footprint CONN-1x02-2.54MM-TH -> Wickerlib:CONN-HEADER-STRAIGHT-P2.54MM-1x02
Changed lines of the file:
@@
 EESchema Schematic File Version 2
 LIBS:wickerlib
+LIBS:mcphail-ir-emitter-board-cache
 EELAYER 25 0
 EELAYER END
@@
 F 0 "J1" H 2375 4000 50  0000 L CNN
 F 1 "TO MCU" H 2375 3700 50  0000 L CNN
-F 2 "CONN-1x02-2.54MM-TH" H 2475 3500 50  0001 C CIN
+F 2 "Wickerlib:CONN-HEADER-STRAIGHT-P2.54MM-1x02" H 2475 3500 50  0001 C CIN
 F 3 "https://cdn.harwin.com/pdfs/60page140.pdf" H 2425 3850 5   0001 C CNN
 F 4 "HEADER MALE 2POS TH 1x02 0.1IN" H 2475 3500 50  0001 C CIN "Description"

Commit message: Release v1.0 Mcphail IR 940nm Detector Board.
Parts:
- LED1: footprint Wickerlib:LED-D5MM-2PIN -> Wickerlib:LED-D5MM-2PIN-SH4356
- LED10: renamed from LED2; footprint Wickerlib:LED-D5MM-2PIN -> Wickerlib:LED-D5MM-2PIN-SH4356
- LED2: renamed from LED3; footprint Wickerlib:LED-D5MM-2PIN -> Wickerlib:LED-D5MM-2PIN-SH4356
- LED3: renamed from LED5; footprint Wickerlib:LED-D5MM-2PIN -> Wickerlib:LED-D5MM-2PIN-SH4356
- LED4: renamed from LED7; footprint Wickerlib:LED-D5MM-2PIN -> Wickerlib:LED-D5MM-2PIN-SH4356
- LED5: renamed from LED9; footprint Wickerlib:LED-D5MM-2PIN -> Wickerlib:LED-D5MM-2PIN-SH4356
- LED6: renamed from LED10; footprint Wickerlib:LED-D5MM-2PIN -> Wickerlib:LED-D5MM-2PIN-SH4356
- LED7: renamed from LED8; footprint Wickerlib:LED-D5MM-2PIN -> Wickerlib:LED-D5MM-2PIN-SH4356
- LED8: renamed from LED6; footprint Wickerlib:LED-D5MM-2PIN -> Wickerlib:LED-D5MM-2PIN-SH4356
- LED9: renamed from LED4; footprint Wickerlib:LED-D5MM-2PIN -> Wickerlib:LED-D5MM-2PIN-SH4356
Changed lines of the file:
@@
 F 0 "LED1" V 3350 3625 50  0000 C CNN
 F 1 "IR 850NM" V 3100 3625 50  0000 C CNN
-F 2 "Wickerlib:LED-D5MM-2PIN" H 3250 3275 50  0001 C CIN
-F 3 "http://www.mouser.com/ds/2/311/SFH%204356,%20Lead%20(Pb)%20Free%20Product%20-%20RoHS%20Compliant-532102.pdf" V 3250 3625 5   0001 C CNN
+F 2 "Wickerlib:LED-D5MM-2PIN-SH4356" H 3250 3275 50  0001 C CIN
+F 3 "http://www.mouser.com/ds/2/311/SFH%204356,%20Lead%20(Pb)%20Free%20Product%20-%20RoHS%20Compliant-532102.pdf" V 3250 3625 10  0001 C CNN
 F 4 "LED IR 850NM TH SFH4356" H 3250 3275 50  0001 C CIN "Description"
 F 5 "OSRAM Opto" H 3250 3275 50  0001 C CIN "MF_Name"
@@
 	2750 3625 3150 3625
 $Comp
-L LED-IR-850NM-2PIN-TH-SFH4356 LED3
+L LED-IR-850NM-2PIN-TH-SFH4356 LED2
 U 1 1 5987BFBB
 P 3750 3625
-F 0 "LED3" V 3850 3625 50  0000 C CNN
+F 0 "LED2" V 3850 3625 50  0000 C CNN
 F 1 "IR 850NM" V 3600 3625 50  0000 C CNN
-F 2 "Wickerlib:LED-D5MM-2PIN" H 3750 3275 50  0001 C CIN
+F 2 "Wickerlib:LED-D5MM-2PIN-SH4356" H 3750 3275 50  0001 C CIN
 F 3 "http://www.mouser.com/ds/2/311/SFH%204356,%20Lead%20(Pb)%20Free%20Product%20-%20RoHS%20Compliant-532102.pdf" V 3750 3625 5   0001 C CNN
 F 4 "LED IR 850NM TH SFH4356" H 3750 3275 50  0001 C CIN "Description"
@@
 	3850 3625 4125 3625
 $Comp
-L LED-IR-850NM-2PIN-TH-SFH4356 LED5
+L LED-IR-850NM-2PIN-TH-SFH4356 LED3
 U 1 1 5987BFF3
 P 4225 3625
-F 0 "LED5" V 4325 3625 50  0000 C CNN
+F 0 "LED3" V 4325 3625 50  0000 C CNN
 F 1 "IR 850NM" V 4075 3625 50  0000 C CNN
-F 2 "Wickerlib:LED-D5MM-2PIN" H 4225 3275 50  0001 C CIN
+F 2 "Wickerlib:LED-D5MM-2PIN-SH4356" H 4225 3275 50  0001 C CIN
 F 3 "http://www.mouser.com/ds/2/311/SFH%204356,%20Lead%20(Pb)%20Free%20Product%20-%20RoHS%20Compliant-532102.pdf" V 4225 3625 5   0001 C CNN
 F 4 "LED IR 850NM TH SFH4356" H 4225 3275 50  0001 C CIN "Description"
@@
 $EndComp
 $Comp
-L LED-IR-850NM-2PIN-TH-SFH4356 LED7
+L LED-IR-850NM-2PIN-TH-SFH4356 LED4
 U 1 1 5987C073
 P 4725 3625
-F 0 "LED7" V 4825 3625 50  0000 C CNN
+F 0 "LED4" V 4825 3625 50  0000 C CNN
 F 1 "IR 850NM" V 4575 3625 50  0000 C CNN
-F 2 "Wickerlib:LED-D5MM-2PIN" H 4725 3275 50  0001 C CIN
+F 2 "Wickerlib:LED-D5MM-2PIN-SH4356" H 4725 3275 50  0001 C CIN
 F 3 "http://www.mouser.com/ds/2/311/SFH%204356,%20Lead%20(Pb)%20Free%20Product%20-%20RoHS%20Compliant-532102.pdf" V 4725 3625 5   0001 C CNN
 F 4 "LED IR 850NM TH SFH4356" H 4725 3275 50  0001 C CIN "Description"
@@
 	4325 3625 4625 3625
 $Comp
-L LED-IR-850NM-2PIN-TH-SFH4356 LED9
+L LED-IR-850NM-2PIN-TH-SFH4356 LED5
 U 1 1 5987C0CE
 P 5150 3625
-F 0 "LED9" V 5250 3625 50  0000 C CNN
+F 0 "LED5" V 5250 3625 50  0000 C CNN
 F 1 "IR 850NM" V 5000 3625 50  0000 C CNN
-F 2 "Wickerlib:LED-D5MM-2PIN" H 5150 3275 50  0001 C CIN
+F 2 "Wickerlib:LED-D5MM-2PIN-SH4356" H 5150 3275 50  0001 C CIN
 F 3 "http://www.mouser.com/ds/2/311/SFH%204356,%20Lead%20(Pb)%20Free%20Product%20-%20RoHS%20Compliant-532102.pdf" V 5150 3625 5   0001 C CNN
 F 4 "LED IR 850NM TH SFH4356" H 5150 3275 50  0001 C CIN "Description"
@@
 	5550 4075 5250 4075
 $Comp
-L LED-IR-850NM-2PIN-TH-SFH4356 LED2
+L LED-IR-850NM-2PIN-TH-SFH4356 LED10
 U 1 1 5987C223
 P 3250 4075
-F 0 "LED2" V 3350 4075 50  0000 C CNN
+F 0 "LED10" V 3350 4075 50  0000 C CNN
 F 1 "IR 850NM" V 3100 4075 50  0000 C CNN
-F 2 "Wickerlib:LED-D5MM-2PIN" H 3250 3725 50  0001 C CIN
+F 2 "Wickerlib:LED-D5MM-2PIN-SH4356" H 3250 3725 50  0001 C CIN
 F 3 "http://www.mouser.com/ds/2/311/SFH%204356,%20Lead%20(Pb)%20Free%20Product%20-%20RoHS%20Compliant-532102.pdf" V 3250 4075 5   0001 C CNN
 F 4 "LED IR 850NM TH SFH4356" H 3250 3725 50  0001 C CIN "Description"
@@
 	3350 4075 3650 4075
 $Comp
-L LED-IR-850NM-2PIN-TH-SFH4356 LED4
+L LED-IR-850NM-2PIN-TH-SFH4356 LED9
 U 1 1 5987C22F
 P 3750 4075
-F 0 "LED4" V 3850 4075 50  0000 C CNN
+F 0 "LED9" V 3850 4075 50  0000 C CNN
 F 1 "IR 850NM" V 3600 4075 50  0000 C CNN
-F 2 "Wickerlib:LED-D5MM-2PIN" H 3750 3725 50  0001 C CIN
+F 2 "Wickerlib:LED-D5MM-2PIN-SH4356" H 3750 3725 50  0001 C CIN
 F 3 "http://www.mouser.com/ds/2/311/SFH%204356,%20Lead%20(Pb)%20Free%20Product%20-%20RoHS%20Compliant-532102.pdf" V 3750 4075 5   0001 C CNN
 F 4 "LED IR 850NM TH SFH4356" H 3750 3725 50  0001 C CIN "Description"
@@
 	3850 4075 4125 4075
 $Comp
-L LED-IR-850NM-2PIN-TH-SFH4356 LED6
+L LED-IR-850NM-2PIN-TH-SFH4356 LED8
 U 1 1 5987C23B
 P 4225 4075
-F 0 "LED6" V 4325 4075 50  0000 C CNN
+F 0 "LED8" V 4325 4075 50  0000 C CNN
 F 1 "IR 850NM" V 4075 4075 50  0000 C CNN
-F 2 "Wickerlib:LED-D5MM-2PIN" H 4225 3725 50  0001 C CIN
+F 2 "Wickerlib:LED-D5MM-2PIN-SH4356" H 4225 3725 50  0001 C CIN
 F 3 "http://www.mouser.com/ds/2/311/SFH%204356,%20Lead%20(Pb)%20Free%20Product%20-%20RoHS%20Compliant-532102.pdf" V 4225 4075 5   0001 C CNN
 F 4 "LED IR 850NM TH SFH4356" H 4225 3725 50  0001 C CIN "Description"
@@
 $EndComp
 $Comp
-L LED-IR-850NM-2PIN-TH-SFH4356 LED8
+L LED-IR-850NM-2PIN-TH-SFH4356 LED7
 U 1 1 5987C246
 P 4725 4075
-F 0 "LED8" V 4825 4075 50  0000 C CNN
+F 0 "LED7" V 4825 4075 50  0000 C CNN
 F 1 "IR 850NM" V 4575 4075 50  0000 C CNN
-F 2 "Wickerlib:LED-D5MM-2PIN" H 4725 3725 50  0001 C CIN
+F 2 "Wickerlib:LED-D5MM-2PIN-SH4356" H 4725 3725 50  0001 C CIN
 F 3 "http://www.mouser.com/ds/2/311/SFH%204356,%20Lead%20(Pb)%20Free%20Product%20-%20RoHS%20Compliant-532102.pdf" V 4725 4075 5   0001 C CNN
 F 4 "LED IR 850NM TH SFH4356" H 4725 3725 50  0001 C CIN "Description"
@@
 	4325 4075 4625 4075
 $Comp
-L LED-IR-850NM-2PIN-TH-SFH4356 LED10
+L LED-IR-850NM-2PIN-TH-SFH4356 LED6
 U 1 1 5987C252
 P 5150 4075
-F 0 "LED10" V 5250 4075 50  0000 C CNN
+F 0 "LED6" V 5250 4075 50  0000 C CNN
 F 1 "IR 850NM" V 5000 4075 50  0000 C CNN
-F 2 "Wickerlib:LED-D5MM-2PIN" H 5150 3725 50  0001 C CIN
+F 2 "Wickerlib:LED-D5MM-2PIN-SH4356" H 5150 3725 50  0001 C CIN
 F 3 "http://www.mouser.com/ds/2/311/SFH%204356,%20Lead%20(Pb)%20Free%20Product%20-%20RoHS%20Compliant-532102.pdf" V 5150 4075 5   0001 C CNN
 F 4 "LED IR 850NM TH SFH4356" H 5150 3725 50  0001 C CIN "Description"
