File: hardware/mcphail-ir-emitter-board/mcphail-ir-emitter-board.kicad_pcb (KiCad board)
At the start: 2 copper layers, 0 parts

Commit message: Release v1.0 Mcphail IR 940nm Emitter Board.
Parts:
- added J1: TO MCU, Wickerlib:CONN-HEADER-STRAIGHT-P2.54MM-1x02, F.Cu at (104.1, 81.3)
- added LED1: IR 850NM, Wickerlib:LED-D5MM-2PIN-SH4356, F.Cu at (109.2, 83.8)
- added LED10: IR 850NM, Wickerlib:LED-D5MM-2PIN-SH4356, F.Cu at (166.4, 83.8)
- added LED2: IR 850NM, Wickerlib:LED-D5MM-2PIN-SH4356, F.Cu at (115.6, 83.8)
- added LED3: IR 850NM, Wickerlib:LED-D5MM-2PIN-SH4356, F.Cu at (121.9, 83.8)
- added LED4: IR 850NM, Wickerlib:LED-D5MM-2PIN-SH4356, F.Cu at (128.3, 83.8)
- added LED5: IR 850NM, Wickerlib:LED-D5MM-2PIN-SH4356, F.Cu at (134.6, 83.8)
- added LED6: IR 850NM, Wickerlib:LED-D5MM-2PIN-SH4356, F.Cu at (141.0, 83.8)
- added LED7: IR 850NM, Wickerlib:LED-D5MM-2PIN-SH4356, F.Cu at (147.3, 83.8)
- added LED8: IR 850NM, Wickerlib:LED-D5MM-2PIN-SH4356, F.Cu at (153.7, 83.8)
- added LED9: IR 850NM, Wickerlib:LED-D5MM-2PIN-SH4356, F.Cu at (160.0, 83.8)
Routing:
- net Net-(J1-Pad2): track 0.00 -> 65.7 mm
- net Net-(LED8-Pad1): track 0.00 -> 7.40 mm
- net Net-(LED2-Pad1): track 0.00 -> 7.40 mm
- net Net-(LED3-Pad1): track 0.00 -> 7.40 mm
- net Net-(LED7-Pad1): track 0.00 -> 7.40 mm
- net Net-(LED6-Pad1): track 0.00 -> 7.40 mm
- net Net-(LED1-Pad1): track 0.00 -> 7.40 mm
- net Net-(LED5-Pad1): track 0.00 -> 7.40 mm
- net Net-(LED4-Pad1): track 0.00 -> 7.40 mm
- net Net-(LED10-Pad2): track 0.00 -> 7.40 mm
- net Net-(J1-Pad1): track 0.00 -> 5.08 mm
Other:
- board outline added: 68.6 x 12.7 mm
- rule trace_clearance: 0.1524 -> 0.254
- board text added: "+"
- board text added: "-"
- board text added: "940nm IR Emitter Board v1.0"

Commit message: Release v1.0 McPhail IR Emitter Board
Parts:
- moved J1 75.9 mm to (29.1, 70.5)
- moved LED1 75.9 mm to (34.1, 73.0)
- moved LED10 75.9 mm to (91.3, 73.0)
- moved LED3 75.9 mm to (46.8, 73.0)
- moved LED4 75.9 mm to (53.2, 73.0)
- moved LED5 75.9 mm to (59.5, 73.0)
- moved LED9 75.9 mm to (84.9, 73.0)
- moved LED2 75.9 mm to (40.5, 73.0)
- moved LED6 75.9 mm to (65.9, 73.0)
- moved LED7 75.9 mm to (72.2, 73.0)
- moved LED8 75.9 mm to (78.6, 73.0)
Other:
- board text added: "FABRICATION NOTES 1. THIS IS A 2 LAYER BOARD. 2. EXTERNAL LAYERS SHALL HAVE 1 OZ COPPER. 3. MATERIAL: FR4 AND 0.062 INCH +/- 10% THICK. 4. BOARDS SHALL BE ROHS COMPLIANT. 5. MANUFACTURE IN ACCORDANCE WITH IPC-6012 CLASS 2 6. MASK: BOTH SIDES OF THE BOARD SHALL HAVE SOLDER MASK (ANY COLOR) OVER BARE COPPER. 7. SILK: BOTH SIDES OF THE BOARD SHALL HAVE WHITE SILKSCREEN. DO NOT PLACE SILK OVER BARE C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"
