File: hardware/mcphail-main-board/microcontroller.sch (KiCad schematic (older format))
At the start: 0 parts

Commit message: Release main board sch with BOM and layout estimates.
Parts:
- added BAT1: 3V, Wickerlib:BATT-HOLDER-CR1220-BK-916, symbol BATT-CR1220-HOLDER-SMT-FLATPIN
- added C30, C31, C32, C36, C37, C38, C39: 100nF, Wickerlib:RLC-0603-SMD, symbol CAP-CER-0.1UF-100V-X7R-0603
- added C33, C35: 22pF, Wickerlib:RLC-0603-SMD, symbol CAP-CER-22PF-50V-NP0-0603
- added C34: 1uF, Wickerlib:RLC-0805-SMD, symbol CAP-CER-1UF-25V-X7R-0805
- added C40, C42: 2pF, Wickerlib:RLC-0603-SMD, symbol CAP-CER-2PF-50V-C0G-NP0-0603
- added C41: 100pF, Wickerlib:RLC-0603-SMD, symbol CAP-CER-100PF-50V-C0G-NP0-0603
- added D1: 20V 1A, Wickerlib:DIODE-SMA, symbol DIODE-SCHOTTKY-20V-1A-SS12-SMA
- added D2, D3: CG0603MLC-05E, Wickerlib:RLC-0603-SMD, symbol DIODE-TVS-CG0603MLC-05E
- added F1: 500mA, Wickerlib:RLC-1812-SMD, symbol FUSE-RESET-500MA-15V-MF-MSMF
- added J4: MICRO SD, Wickerlib:CONN-SD-MICRO-MOLEX-0475710001, symbol CONN-MICRO-SD-CARD-PUSH-PULL
- added J5: MICRO USB, Wickerlib:CONN-USB-MICRO-B-AMPHENOL-10118193-0001LF, symbol CONN-USB-MICRO-B-10118193
- added J6: ISP, Wickerlib:CONN-HEADER-STRAIGHT-P2.54MM-2x03, symbol HEADER-MALE-6POS-TH-2x3-P0.1IN
- added J7: FONA 808, Wickerlib:BREAKOUT-ADAFRUIT-FONA808-CELL-GPS, symbol ADAFRUIT-FONA-808-GPS
- added L1: FERRITE, Wickerlib:RLC-0402-SMD, symbol FERRITE-BEAD-220-OHM-0402-1LN
- added R31, R32: 22, Wickerlib:RLC-0603-SMD, symbol RES-22-OHM-5%-1/10W-0603
- added R33, R36: 10K, Wickerlib:RLC-0603-SMD, symbol RES-10K-1%-1/8W-0603
- added R34, R35: 2K, Wickerlib:RLC-0603-SMD, symbol RES-2K-1%-1/8W-0603
- added R37: 1K, Wickerlib:RLC-0603-SMD, symbol RES-1K-1%-1/10W-0603
- added S1: RESET, Wickerlib:SWITCH-OMRON-MOMENTARY-SMD-B3U-1000P, symbol SWITCH-MOMENT-SPST-NO-0.05A-12V-SMT-B3U-1000P
- added U5: TXB0104, Wickerlib:SOIC-14-3.9x8.7MM-P1.27MM, symbol IC-VOLT-LEVEL-TRANSLATOR-TXB0104-SOIC14
- added U6: ATMEGA32U4-TQFP44, Wickerlib:TQFP-44-10x10MM-P0.8MM, symbol IC-MCU-ATMEGA32U4-TQFP44-CUSTOM2
- added U7: 24AA1025 EEPROM, Wickerlib:SOIC-8-3.9x4.9MM-P1.27MM, symbol IC-EEPROM-1MBIT-400KHZ-24AA1025-SOIC8
- added U8: MCP7940N RTC, Wickerlib:SOIC-8-3.9x4.9MM-P1.27MM, symbol IC-RTC-MCP7940N-SOIC8
- added X1: 16MHz, Wickerlib:CRYSTAL-CTS-4SMD, symbol CRYSTAL-16MHZ-18PF-40OHM-CTS-4SMD
- added X2: 32.768kHz, Wickerlib:CRYSTAL-HC49-TH, symbol CRYSTAL-32.768KHZ-7PF-CFS206-TH
Connections:
- net labels added: +3.3V, +5V, 3.3V, 5V, A0, A1, A2, D4_CS, EEPROM_A0, EEPROM_A1, EEPROM_A2, FONA_NS, FONA_PS, FONA_RI, FONA_RST, FONA_RTS, FONA_RX, FONA_TX, GND, MFP, MISO, MOSI, SCL, SCLK, SDA, SD_CS, SD_MISO, SD_MOSI, SD_SCLK, USB_D+, USB_D-, USB_GND, VUSB, VUSB_IN, ~PG, ~RESET
- wire segments 0 -> 195
- no-connect marks 0 -> 10
Other:
- note added: "ATMEGA32u4"
- note added: "CELL"
- note added: "EEPROM"
- note added: "RTC\n"

Commit message: Added ADS1118 (ADC with temp sensor) to Atmega32u4.
Parts:
- added C?: 100nF, Wickerlib:RLC-0603-SMD, symbol CAP-CER-0.1UF-100V-X7R-0603
- added U6: IC-MCU-ATSAMD21G18A-TQFP48-CUSTOM1, Wickerlib:UNDEFINED, symbol IC-MCU-ATSAMD21G18A-TQFP48-CUSTOM1
- added U?: ADS1118, Wickerlib:SOIC-14-3.9x8.7MM-P1.27MM, symbol IC-ADC-16BIT-SPI-ADS1118-10MSOP
Connections:
- net labels added: D7_CS
- wire segments 195 -> 260
- no-connect marks 10 -> 9
Other:
- note added: "SHEET 3: MICROCONTROLLER"

Commit message: Switched all to 3.3V, things got simple, cheaper.
Parts:
- removed C30, C31: 100nF, Wickerlib:RLC-0603-SMD, symbol CAP-CER-0.1UF-100V-X7R-0603
- removed C34: 1uF, Wickerlib:RLC-0805-SMD, symbol CAP-CER-1UF-25V-X7R-0805
- removed J6: ISP, Wickerlib:CONN-HEADER-STRAIGHT-P2.54MM-2x03, symbol HEADER-MALE-6POS-TH-2x3-P0.1IN
- removed R31, R32: 22, Wickerlib:RLC-0603-SMD, symbol RES-22-OHM-5%-1/10W-0603
- removed U5: TXB0104, Wickerlib:SOIC-14-3.9x8.7MM-P1.27MM, symbol IC-VOLT-LEVEL-TRANSLATOR-TXB0104-SOIC14
Connections:
- net labels removed: 3.3V, 5V, SD_CS, SD_MISO, SD_MOSI, SD_SCLK, USB_GND
- wire segments 260 -> 196
- no-connect marks 9 -> 10
Other:
- note added: "16-bit ADC"
- note added: "5V is to charge the Fona's\n3.7V LiPO Battery\n\nVio sets the voltage\nlevel for the Fona \npins to 3.3V"
- note added: "MicroSD"
- note added: "and Temp Sensor"
- moved on the sheet: D1, D2, D3, F1, J4, J5, L1, U6

Commit message: Hooked up pins to ATSAMD21G18 Cortex M0, fixed AGND throughout.
Parts:
- removed L1: FERRITE, Wickerlib:RLC-0402-SMD, symbol FERRITE-BEAD-220-OHM-0402-1LN
- removed U6: ATMEGA32U4-TQFP44, Wickerlib:TQFP-44-10x10MM-P0.8MM, symbol IC-MCU-ATMEGA32U4-TQFP44-CUSTOM2
- added C31: 10uF, Wickerlib:RLC-0805-SMD, symbol CAP-CER-10UF-16V-X7R-0805
- added C34: 1uF, Wickerlib:RLC-0805-SMD, symbol CAP-CER-1UF-25V-X7R-0805
- added C51, C52: 100nF, Wickerlib:RLC-0603-SMD, symbol CAP-CER-0.1UF-100V-X7R-0603
- added J10: BREAKOUT, Wickerlib:CONN-HEADER-STRAIGHT-P2.54MM-1x10, symbol HEADER-FEMALE-10POS-TH-1x10-P0.1IN
- added J6: SWD, Wickerlib:CONN-HEADER-STRAIGHT-P2.54MM-1x05, symbol HEADER-MALE-5POS-TH-1x05-P0.1IN
- added L1, L3, L4: FERRITE, Wickerlib:RLC-0805-SMD, symbol FERRITE-BEAD-30-OHM-0805-1LN
- added R31: 330, Wickerlib:RLC-0603-SMD, symbol RES-330-5%-1/10W-0603
- added R32: 1K, Wickerlib:RLC-0603-SMD, symbol RES-1K-1%-1/10W-0603
- U6: value IC-MCU-ATSAMD21G18A-TQFP48-CUSTOM1 -> ATSAMD21G18A
- gave numbers to parts that had none: 2
Connections:
- net D7_CS is gone; now on net D4_CS: U5.2 (~CS)
- net +3V3: now also U6.17 (VDDIO), U6.36 (VDDIO), U6.44 (VDDIN), J10.1 (P1), J6.1 (P1), L4.2, R32.1
- net A0: now also U6.12 (PA07/AIN7)
- net A1: now also U6.11 (PA06/AIN6)
- net A2: now also U6.10 (PA05/AIN5)
- net D4_CS: now also U6.13 (PA08/I2C/AIN16), U6.30 (PA21)
- net EEPROM_A0: now also U6.1 (PA00/XIN32)
- net EEPROM_A1: now also U6.48 (PB03/AIN11)
- net EEPROM_A2: now also U6.47 (PB02/AIN10)
- net FONA_NS: now also U6.27 (PA18)
- net FONA_PS: now also U6.28 (PA19)
- net FONA_RI: now also U6.38 (PB23)
- net FONA_RST: now also U6.22 (PA13/I2C)
- net FONA_RTS: now also U6.37 (PB22)
- net FONA_RX: now also U6.31 (PA22/I2C)
- net FONA_TX: now also U6.29 (PA20)
- net GND: now also U6.18 (GND), U6.35 (GND), U6.42 (GND), C34.2, C51.2, J10.10 (P10), J6.5 (P5), L1.2, L3.1
- net MFP: now also U6.14 (PA09/I2C/AIN17)
- net MISO: now also U6.21 (PA12/I2C)
- net MOSI: now also U6.19 (PB10)
- net SCL: now also U6.26 (PA17/I2C)
- net SCLK: now also U6.20 (PB11)
- net SDA: now also U6.25 (PA16/I2C)
- net USB_D+: now also U6.34 (PA25/USBDP)
- net USB_D-: now also U6.33 (PA24/USBDM)
- net ~RESET: now also U6.40 (~RESET), C51.1, J6.4 (P4), R31.1; no longer S1.1
- net at C35.1, X1.3 (OUT): now also U6.24 (PA15/XOUT)
- net at C33.1, X1.1 (EN): now also U6.23 (PA14/XIN)
- net at J5.5 (GND): now also L1.1
- net at U6.2 (PA01/XOUT32): now also J10.7 (P7)
- net at U6.3 (PA02/AIN0): now also J10.8 (P8)
- net at U6.39 (PA27): now also J10.2 (P2)
- net at U6.4 (PA03/AIN1): now also J10.9 (P9)
- net at U6.41 (PA28): now also J10.3 (P3)
- net at U6.43 (VDDCORE): now also C34.1
- net SWCLK: now reaches U6.45 (PA30/SWCLK)
- net SWCLK: now also J6.3 (P3), R32.2
- net SWDIO: now reaches U6.46 (PA31/SWDIO)
- net SWDIO: now also J6.2 (P2)
- net AGND: now reaches U6.5 (GNDANA)
- net AGND: now also C31.2, C52.2, L3.2
- net VDDANA: now reaches U6.6 (VDDANA)
- net VDDANA: now also C31.1, C52.1, L4.1
- net at U6.7 (PB08/AIN2): now also J10.4 (P4)
- net at U6.8 (PB09/AIN3): now also J10.5 (P5)
- net at U6.9 (PA04/AIN4): now also J10.6 (P6)
- new net: R31.2, S1.1
- no-connect marks 10 -> 8
Other:
- note added: "ATSAM21G18 Cortex M0\n(Arduino-compatible)"
- note added: "Programming"
- note removed: "ATMEGA32u4"
- moved on the sheet: BAT1, C32, C40, C41, C42, D1, D2, D3, F1, J5, R33, R34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

Commit message: All footprints good. Changed op amps slightly for footprints.
Parts:
- U6: footprint Wickerlib:UNDEFINED -> Wickerlib:TQFP-48_7x7mm_Pitch0.5mm

Commit message: Lots more layout work, needs rework.
Parts:
- removed C32: 100nF, Wickerlib:RLC-0603-SMD, symbol CAP-CER-0.1UF-100V-X7R-0603
- removed J10: BREAKOUT, Wickerlib:CONN-HEADER-STRAIGHT-P2.54MM-1x10, symbol HEADER-FEMALE-10POS-TH-1x10-P0.1IN
- removed J6: SWD, Wickerlib:CONN-HEADER-STRAIGHT-P2.54MM-1x05, symbol HEADER-MALE-5POS-TH-1x05-P0.1IN
- added FID1, FID2, FID3: FIDUCIAL, Wickerlib:FIDUCIAL-2MM, symbol FIDUCIAL
- added J6: PROG/BOOT, Wickerlib:CONN-HEADER-STRAIGHT-P2.54MM-2x03, symbol HEADER-FEMALE-6POS-TH-2x3-P0.1IN
- U5: footprint Wickerlib:SOIC-14-3.9x8.7MM-P1.27MM -> Wickerlib:MSOP-10-3x3MM-P0.5MM
Connections:
- net +3V3: now also J6.1 (P1)
- net AGND: now also C30.2, U5.3 (GND)
- net D4_CS: no longer J4.2 (CS), U6.30 (PA21)
- net GND: now also J6.5 (P5); no longer C30.2, U5.3 (GND)
- net SWCLK: now also J6.4 (P4)
- net SWDIO: now also J6.2 (P2)
- net ~PG: now also U6.15 (PA10/AIN18)
- net ~RESET: now also J6.6 (P6)
- net USB_D+ renamed D+
- net USB_D- renamed D-
- new net D7_CS: J4.2 (CS), U6.30 (PA21)
- no-connect marks 8 -> 17
Other:
- note removed: "Programming"
- moved on the sheet: J4

Commit message: Saving main board layout before major rework.
Other:
- moved on the sheet: C39
Changed lines of the file:
@@
 L CAP-CER-0.1UF-100V-X7R-0603 C39
 U 1 1 597B3976
-P 9625 5000
-F 0 "C39" H 9725 5050 50  0000 L CNN
-F 1 "100nF" H 9725 4950 50  0000 L CNN
-F 2 "Wickerlib:RLC-0603-SMD" H 9625 4650 50  0001 C CIN
-F 3 "http://search.murata.co.jp/Ceramy/image/img/A01X/partnumbering_e_01.pdf" H 9625 5000 5   0001 C CNN
-F 4 "CAP CER 0.1UF 100V X7R 0603" H 9625 4650 50  0001 C CIN "Description"
-F 5 "Murata" H 9625 4650 50  0001 C CIN "MF_Name"
-F 6 "GRM188R72A104KA35D" H 9625 4650 50  0001 C CIN "MF_PN"
-F 7 "Digikey" H 9625 4650 50  0001 C CIN "S1_Name"
-F 8 "490-3285-1-ND" H 9625 4650 50  0001 C CIN "S1_PN"
-	1    9625 5000
+P 9625 4950
+F 0 "C39" H 9725 5000 50  0000 L CNN
+F 1 "100nF" H 9725 4900 50  0000 L CNN
+F 2 "Wickerlib:RLC-0603-SMD" H 9625 4600 50  0001 C CIN
+F 3 "http://search.murata.co.jp/Ceramy/image/img/A01X/partnumbering_e_01.pdf" H 9625 4950 5   0001 C CNN
+F 4 "CAP CER 0.1UF 100V X7R 0603" H 9625 4600 50  0001 C CIN "Description"
+F 5 "Murata" H 9625 4600 50  0001 C CIN "MF_Name"
+F 6 "GRM188R72A104KA35D" H 9625 4600 50  0001 C CIN "MF_PN"
+F 7 "Digikey" H 9625 4600 50  0001 C CIN "S1_Name"
+F 8 "490-3285-1-ND" H 9625 4600 50  0001 C CIN "S1_PN"
+	1    9625 4950
 	-1   0    0    -1
 $EndComp
@@
 L GND #PWR059
 U 1 1 597B3A1E
-P 9625 5100
-F 0 "#PWR059" H 9625 4850 50  0001 C CNN
-F 1 "GND" H 9625 4950 50  0000 C CNN
-F 2 "" H 9625 5100 50  0000 C CNN
-F 3 "" H 9625 5100 50  0000 C CNN
-	1    9625 5100
+P 9625 5050
+F 0 "#PWR059" H 9625 4800 50  0001 C CNN
+F 1 "GND" H 9625 4900 50  0000 C CNN
+F 2 "" H 9625 5050 50  0000 C CNN
+F 3 "" H 9625 5050 50  0000 C CNN
+	1    9625 5050
 	-1   0    0    -1
 $EndComp
@@
 L +3.3V #PWR066
 U 1 1 597C75DE
-P 9125 4950
-F 0 "#PWR066" H 9125 4800 50  0001 C CNN
-F 1 "+3.3V" H 9125 5090 50  0000 C CNN
-F 2 "" H 9125 4950 50  0000 C CNN
-F 3 "" H 9125 4950 50  0000 C CNN
-	1    9125 4950
+P 9125 4725
+F 0 "#PWR066" H 9125 4575 50  0001 C CNN
+F 1 "+3.3V" H 9125 4865 50  0000 C CNN
+F 2 "" H 9125 4725 50  0000 C CNN
+F 3 "" H 9125 4725 50  0000 C CNN
+	1    9125 4725
 	1    0    0    -1
 $EndComp
@@
 SWCLK
 Wire Wire Line
-	3300 2025 3300 3700
+	3300 2025 3300 3275
+Wire Wire Line
+	3300 3275 3300 3700
 Wire Wire Line
 	7650 4875 8275 4875
@@
 Connection ~ 9050 2725
 Wire Wire Line
-	9050 1275 9050 2800
+	9050 1275 9050 2725
+Wire Wire Line
+	9050 2725 9050 2800
 Wire Wire Line
 	9050 2725 9125 2725
@@
 	8800 1075 9125 1075
 Wire Wire Line
-	9050 725  9050 875
+	9050 725  9050 775
+Wire Wire Line
+	9050 775  9050 875
 Wire Wire Line
 	9050 875  9125 875
@@
 Connection ~ 10450 4175
 Wire Wire Line
-	10925 3825 10925 4425
+	10925 3825 10925 4175
+Wire Wire Line
+	10925 4175 10925 4425
 Wire Wire Line
 	10450 4175 10450 4425
@@
 	10925 4625 10925 4950
 Wire Wire Line
-	10400 4175 10525 4175
+	10400 4175 10450 4175
+Wire Wire Line
+	10450 4175 10525 4175
 Wire Wire Line
 	10400 3825 10925 3825
 Connection ~ 8450 3925
 Wire Wire Line
-	8450 3650 8450 5725
+	8450 3650 8450 3925
+Wire Wire Line
+	8450 3925 8450 4325
+Wire Wire Line
+	8450 4325 8450 5725
 Connection ~ 8750 3825
 Wire Wire Line
-	8750 3650 8750 5575
+	8750 3650 8750 3825
+Wire Wire Line
+	8750 3825 8750 4225
+Wire Wire Line
+	8750 4225 8750 5575
 Connection ~ 9050 4025
 Wire Wire Line
-	9050 3650 9050 4425
+	9050 3650 9050 4025
+Wire Wire Line
+	9050 4025 9050 4425
 Wire Wire Line
 	11000 3675 10400 3675
@@
 	10300 3300 10300 3225
 Wire Wire Line
-	10300 2825 10300 2925
+	10300 2825 10300 2875
+Wire Wire Line
+	10300 2875 10300 2925
 Wire Wire Line
 	10150 5725 10700 5725
@@
 	9150 5875 9050 5875
 Wire Wire Line
-	9125 4950 9125 5425
+	9125 4725 9125 4775
+Wire Wire Line
+	9125 4775 9125 5425
 Wire Wire Line
 	9125 5425 9150 5425
@@
 	4575 1925 4450 1925
 Wire Wire Line
-	4575 1800 4575 1975
+	4575 1800 4575 1925
+Wire Wire Line
+	4575 1925 4575 1975
 Wire Wire Line
 	3975 1200 3975 1225
 Wire Wire Line
-	3400 2125 3400 3800
+	3400 2125 3400 3175
+Wire Wire Line
+	3400 3175 3400 3800
 Wire Wire Line
 	2675 2125 3400 2125
@@
 	3600 2875 3600 2325
 Wire Wire Line
-	3500 2225 3500 3500
+	3500 2225 3500 3075
+Wire Wire Line
+	3500 3075 3500 3500
 Wire Wire Line
 	2675 2225 3500 2225
@@
 	4150 3725 4025 3725
 Wire Wire Line
-	4025 3625 4025 3875
+	4025 3625 4025 3725
+Wire Wire Line
+	4025 3725 4025 3875
 Wire Wire Line
 	4150 3625 4025 3625
@@
 	5200 3800 5200 3725
 Wire Wire Line
-	4650 3725 5450 3725
-Wire Wire Line
-	4650 3625 5450 3625
+	4650 3725 5200 3725
+Wire Wire Line
+	5200 3725 5450 3725
+Wire Wire Line
+	4650 3625 4825 3625
+Wire Wire Line
+	4825 3625 5450 3625
 Wire Wire Line
 	3900 6000 3900 5950
@@
 	3025 5550 3025 5100
 Wire Wire Line
-	5350 5400 4550 5400
+	5350 5400 4825 5400
+Wire Wire Line
+	4825 5400 4550 5400
 Wire Wire Line
 	4375 5100 4375 4475
@@
 	4475 5200 4475 4575
 Wire Wire Line
-	2875 5200 4475 5200
-Wire Wire Line
-	2875 5100 4375 5100
+	2875 5200 3900 5200
+Wire Wire Line
+	3900 5200 4475 5200
+Wire Wire Line
+	2875 5100 3025 5100
+Wire Wire Line
+	3025 5100 4375 5100
 Wire Wire Line
 	2875 5400 4350 5400
@@
 Wire Wire Line
 	6575 1450 6575 1600
-Connection ~ 9125 5000
+Connection ~ 9125 4775
 Wire Wire Line
 	10900 5425 10900 6350
@@
 	8625 2825 8625 1975
 Wire Wire Line
-	9125 5000 9525 4825
-Wire Wire Line
-	9525 4825 9625 4825
-Wire Wire Line
-	9625 4825 9625 4900
+	9125 4775 9525 4775
+Wire Wire Line
+	9525 4775 9625 4775
+Wire Wire Line
+	9625 4775 9625 4850
 Wire Wire Line
 	3500 3500 2825 3500
@@
 	1400 3500 1525 3500
 Wire Wire Line
-	1400 3275 1400 3950
+	1400 3275 1400 3350
+Wire Wire Line
+	1400 3350 1400 3500
+Wire Wire Line
+	1400 3500 1400 3950
 Wire Wire Line
 	1400 3950 1525 3950
@@
 	8800 1025 8800 1075
 Wire Wire Line
-	5375 1175 5375 2525
+	5375 1175 5375 1225
+Wire Wire Line
+	5375 1225 5375 1450
+Wire Wire Line
+	5375 1450 5375 2325
+Wire Wire Line
+	5375 2325 5375 2425
+Wire Wire Line
+	5375 2425 5375 2525
 Wire Wire Line
 	5450 4775 4725 4775
@@
 	5450 5125 5350 5125
 Wire Wire Line
-	5350 5125 5350 5400
+	5350 5125 5350 5225
+Wire Wire Line
+	5350 5225 5350 5325
+Wire Wire Line
+	5350 5325 5350 5400
 Wire Wire Line
 	5450 5325 5350 5325
@@
 Connection ~ 5350 5225
 Wire Wire Line
-	5275 5025 5275 6325
+	5275 5025 5275 6000
+Wire Wire Line
+	5275 6000 5275 6225
+Wire Wire Line
+	5275 6225 5275 6325
 Wire Wire Line
 	5275 5025 5450 5025
 Wire Wire Line
-	4825 5400 4825 6325
+	4825 5400 4825 6000
+Wire Wire Line
+	4825 6000 4825 6225
+Wire Wire Line
+	4825 6225 4825 6325
 Wire Wire Line
 	5275 6225 5150 6225
@@
 Connection ~ 4825 5400
 Wire Wire Line
-	4425 2225 5450 2225
+	4425 2225 4875 2225
+Wire Wire Line
+	4875 2225 4950 2225
+Wire Wire Line
+	4950 2225 5450 2225
 Wire Wire Line
 	4875 2225 4875 2300
@@
 Connection ~ 4950 2225
 Wire Wire Line
-	3975 1425 3975 1575
+	3975 1425 3975 1500
+Wire Wire Line
+	3975 1500 3975 1575
 Wire Wire Line
 	3975 1775 3975 1925
@@
 	4575 1500 4575 1600
 Wire Wire Line
-	3875 1500 4575 1500
+	3875 1500 3975 1500
+Wire Wire Line
+	3975 1500 4575 1500
 Connection ~ 3975 1500
 Wire Wire Line
@@
 	7950 5625 7650 5625
 Wire Wire Line
-	6075 6425 8050 6425
+	6075 6425 6725 6425
+Wire Wire Line
+	6725 6425 8050 6425
 Wire Wire Line
 	8050 6425 8050 5525
@@
 $EndComp
 Wire Wire Line
-	5250 1450 6575 1450
+	5250 1450 5375 1450
+Wire Wire Line
+	5375 1450 5600 1450
+Wire Wire Line
+	5600 1450 6075 1450
+Wire Wire Line
+	6075 1450 6575 1450
 $Comp
 L FIDUCIAL FID1
