File: hardware/mcphail-main-board/microcontroller.sch (KiCad schematic (older format))
At the start: 43 parts, among them J4 MICRO SD, J5 MICRO USB, J6 PROG/BOOT, J7 FONA 808, U5 ADS1118, U6 ATSAMD21G18A, U7 24AA1025 EEPROM, U8 MCP7940N RTC, X1 16MHz, X2 32.768kHz

Commit message: Regenerated sch pdf. Converted to 4 layer.
Connections:
- wire segments 240 -> 198
Changed lines of the file:
@@
 SWCLK
 Wire Wire Line
-	3300 2025 3300 3275
-Wire Wire Line
-	3300 3275 3300 3700
+	3300 2025 3300 3700
 Wire Wire Line
 	7650 4875 8275 4875
@@
 Connection ~ 9050 2725
 Wire Wire Line
-	9050 1275 9050 2725
-Wire Wire Line
-	9050 2725 9050 2800
+	9050 1275 9050 2800
 Wire Wire Line
 	9050 2725 9125 2725
@@
 	8800 1075 9125 1075
 Wire Wire Line
-	9050 725  9050 775
-Wire Wire Line
-	9050 775  9050 875
+	9050 725  9050 875
 Wire Wire Line
 	9050 875  9125 875
@@
 Connection ~ 10450 4175
 Wire Wire Line
-	10925 3825 10925 4175
-Wire Wire Line
-	10925 4175 10925 4425
+	10925 3825 10925 4425
 Wire Wire Line
 	10450 4175 10450 4425
@@
 	10925 4625 10925 4950
 Wire Wire Line
-	10400 4175 10450 4175
-Wire Wire Line
-	10450 4175 10525 4175
+	10400 4175 10525 4175
 Wire Wire Line
 	10400 3825 10925 3825
 Connection ~ 8450 3925
 Wire Wire Line
-	8450 3650 8450 3925
-Wire Wire Line
-	8450 3925 8450 4325
-Wire Wire Line
-	8450 4325 8450 5725
+	8450 3650 8450 5725
 Connection ~ 8750 3825
 Wire Wire Line
-	8750 3650 8750 3825
-Wire Wire Line
-	8750 3825 8750 4225
-Wire Wire Line
-	8750 4225 8750 5575
+	8750 3650 8750 5575
 Connection ~ 9050 4025
 Wire Wire Line
-	9050 3650 9050 4025
-Wire Wire Line
-	9050 4025 9050 4425
+	9050 3650 9050 4425
 Wire Wire Line
 	11000 3675 10400 3675
@@
 	10300 3300 10300 3225
 Wire Wire Line
-	10300 2825 10300 2875
-Wire Wire Line
-	10300 2875 10300 2925
+	10300 2825 10300 2925
 Wire Wire Line
 	10150 5725 10700 5725
@@
 	9150 5875 9050 5875
 Wire Wire Line
-	9125 4725 9125 4775
-Wire Wire Line
-	9125 4775 9125 5425
+	9125 4725 9125 5425
 Wire Wire Line
 	9125 5425 9150 5425
@@
 	4575 1925 4450 1925
 Wire Wire Line
-	4575 1800 4575 1925
-Wire Wire Line
-	4575 1925 4575 1975
+	4575 1800 4575 1975
 Wire Wire Line
 	3975 1200 3975 1225
 Wire Wire Line
-	3400 2125 3400 3175
-Wire Wire Line
-	3400 3175 3400 3800
+	3400 2125 3400 3800
 Wire Wire Line
 	2675 2125 3400 2125
@@
 	3600 2875 3600 2325
 Wire Wire Line
-	3500 2225 3500 3075
-Wire Wire Line
-	3500 3075 3500 3500
+	3500 2225 3500 3500
 Wire Wire Line
 	2675 2225 3500 2225
@@
 	4150 3725 4025 3725
 Wire Wire Line
-	4025 3625 4025 3725
-Wire Wire Line
-	4025 3725 4025 3875
+	4025 3625 4025 3875
 Wire Wire Line
 	4150 3625 4025 3625
@@
 	5200 3800 5200 3725
 Wire Wire Line
-	4650 3725 5200 3725
-Wire Wire Line
-	5200 3725 5450 3725
-Wire Wire Line
-	4650 3625 4825 3625
-Wire Wire Line
-	4825 3625 5450 3625
+	4650 3725 5450 3725
+Wire Wire Line
+	4650 3625 5450 3625
 Wire Wire Line
 	3900 6000 3900 5950
@@
 	3025 5550 3025 5100
 Wire Wire Line
-	5350 5400 4825 5400
-Wire Wire Line
-	4825 5400 4550 5400
+	5350 5400 4550 5400
 Wire Wire Line
 	4375 5100 4375 4475
@@
 	4475 5200 4475 4575
 Wire Wire Line
-	2875 5200 3900 5200
-Wire Wire Line
-	3900 5200 4475 5200
-Wire Wire Line
-	2875 5100 3025 5100
-Wire Wire Line
-	3025 5100 4375 5100
+	2875 5200 4475 5200
+Wire Wire Line
+	2875 5100 4375 5100
 Wire Wire Line
 	2875 5400 4350 5400
@@
 	8625 2825 8625 1975
 Wire Wire Line
-	9125 4775 9525 4775
-Wire Wire Line
-	9525 4775 9625 4775
+	9125 4775 9625 4775
 Wire Wire Line
 	9625 4775 9625 4850
@@
 	1400 3500 1525 3500
 Wire Wire Line
-	1400 3275 1400 3350
-Wire Wire Line
-	1400 3350 1400 3500
-Wire Wire Line
-	1400 3500 1400 3950
+	1400 3275 1400 3950
 Wire Wire Line
 	1400 3950 1525 3950
@@
 	8800 1025 8800 1075
 Wire Wire Line
-	5375 1175 5375 1225
-Wire Wire Line
-	5375 1225 5375 1450
-Wire Wire Line
-	5375 1450 5375 2325
-Wire Wire Line
-	5375 2325 5375 2425
-Wire Wire Line
-	5375 2425 5375 2525
+	5375 1175 5375 2525
 Wire Wire Line
 	5450 4775 4725 4775
@@
 	5450 5125 5350 5125
 Wire Wire Line
-	5350 5125 5350 5225
-Wire Wire Line
-	5350 5225 5350 5325
-Wire Wire Line
-	5350 5325 5350 5400
+	5350 5125 5350 5400
 Wire Wire Line
 	5450 5325 5350 5325
@@
 Connection ~ 5350 5225
 Wire Wire Line
-	5275 5025 5275 6000
-Wire Wire Line
-	5275 6000 5275 6225
-Wire Wire Line
-	5275 6225 5275 6325
+	5275 5025 5275 6325
 Wire Wire Line
 	5275 5025 5450 5025
 Wire Wire Line
-	4825 5400 4825 6000
-Wire Wire Line
-	4825 6000 4825 6225
-Wire Wire Line
-	4825 6225 4825 6325
+	4825 5400 4825 6325
 Wire Wire Line
 	5275 6225 5150 6225
@@
 Connection ~ 4825 5400
 Wire Wire Line
-	4425 2225 4875 2225
-Wire Wire Line
-	4875 2225 4950 2225
-Wire Wire Line
-	4950 2225 5450 2225
+	4425 2225 5450 2225
 Wire Wire Line
 	4875 2225 4875 2300
@@
 Connection ~ 4950 2225
 Wire Wire Line
-	3975 1425 3975 1500
-Wire Wire Line
-	3975 1500 3975 1575
+	3975 1425 3975 1575
 Wire Wire Line
 	3975 1775 3975 1925
@@
 	4575 1500 4575 1600
 Wire Wire Line
-	3875 1500 3975 1500
-Wire Wire Line
-	3975 1500 4575 1500
+	3875 1500 4575 1500
 Connection ~ 3975 1500
 Wire Wire Line
@@
 	7950 5625 7650 5625
 Wire Wire Line
-	6075 6425 6725 6425
-Wire Wire Line
-	6725 6425 8050 6425
+	6075 6425 8050 6425
 Wire Wire Line
 	8050 6425 8050 5525
@@
 $EndComp
 Wire Wire Line
-	5250 1450 5375 1450
-Wire Wire Line
-	5375 1450 5600 1450
-Wire Wire Line
-	5600 1450 6075 1450
-Wire Wire Line
-	6075 1450 6575 1450
+	5250 1450 6575 1450
 $Comp
 L FIDUCIAL FID1

Commit message: Reworking main board, power rails routed next.
Connections:
- net labels added: EEPROM_ADD0, EEPROM_ADD1, EEPROM_ADD2
- net labels removed: EEPROM_A0, EEPROM_A1, EEPROM_A2

Commit message: Generate Main Board with traces done. Needs silk.
Parts:
- added L5: FERRITE, Wickerlib:RLC-0805-SMD, symbol FERRITE-BEAD-30-OHM-0805-1LN
Connections:
- wire segments 198 -> 200
- no-connect marks 17 -> 19
Other:
- moved on the sheet: J7
Changed lines of the file:
@@
 L GND #PWR038
 U 1 1 5976AADE
-P 4825 6325
-F 0 "#PWR038" H 4825 6075 50  0001 C CNN
-F 1 "GND" H 4825 6175 50  0000 C CNN
-F 2 "" H 4825 6325 50  0000 C CNN
-F 3 "" H 4825 6325 50  0000 C CNN
-	1    4825 6325
+P 4825 6625
+F 0 "#PWR038" H 4825 6375 50  0001 C CNN
+F 1 "GND" H 4825 6475 50  0000 C CNN
+F 2 "" H 4825 6625 50  0000 C CNN
+F 3 "" H 4825 6625 50  0000 C CNN
+	1    4825 6625
 	1    0    0    -1
 $EndComp
@@
 L ADAFRUIT-FONA-808-GPS J7
 U 1 1 5983CEDF
-P 9525 1175
-F 0 "J7" H 9300 1625 50  0000 L CNN
-F 1 "FONA 808" H 9275 -525 50  0000 L CNN
-F 2 "Wickerlib:BREAKOUT-ADAFRUIT-FONA808-CELL-GPS" H 9525 825 50  0001 C CIN
-F 3 "https://www.adafruit.com/products/2542" H 9525 1175 5   0001 C CNN
-F 4 "ADAFRUIT FONA 808 + GPS" H 9525 825 50  0001 C CIN "Description"
-F 5 "Adafruit" H 9525 825 50  0001 C CIN "MF_Name"
-F 6 "FONA808+GPS" H 9525 825 50  0001 C CIN "MF_PN"
-F 7 "Adafruit" H 9525 825 50  0001 C CIN "S1_Name"
-F 8 "2542" H 9525 825 50  0001 C CIN "S1_PN"
-	1    9525 1175
+P 9525 1275
+F 0 "J7" H 9300 1725 50  0000 L CNN
+F 1 "FONA 808" H 9275 -425 50  0000 L CNN
+F 2 "Wickerlib:BREAKOUT-ADAFRUIT-FONA808-CELL-GPS" H 9525 925 50  0001 C CIN
+F 3 "https://www.adafruit.com/products/2542" H 9525 1275 5   0001 C CNN
+F 4 "ADAFRUIT FONA 808 + GPS" H 9525 925 50  0001 C CIN "Description"
+F 5 "Adafruit" H 9525 925 50  0001 C CIN "MF_Name"
+F 6 "FONA808+GPS" H 9525 925 50  0001 C CIN "MF_PN"
+F 7 "Adafruit" H 9525 925 50  0001 C CIN "S1_Name"
+F 8 "2542" H 9525 925 50  0001 C CIN "S1_PN"
+	1    9525 1275
 	-1   0    0    -1
 $EndComp
@@
 L +5V #PWR055
 U 1 1 5983D1B8
-P 9050 725
-F 0 "#PWR055" H 9050 575 50  0001 C CNN
-F 1 "+5V" H 9050 865 50  0000 C CNN
-F 2 "" H 9050 725 50  0000 C CNN
-F 3 "" H 9050 725 50  0000 C CNN
-	1    9050 725
-	1    0    0    -1
-$EndComp
-NoConn ~ 9125 975
-NoConn ~ 9125 2275
+P 9050 825
+F 0 "#PWR055" H 9050 675 50  0001 C CNN
+F 1 "+5V" H 9050 965 50  0000 C CNN
+F 2 "" H 9050 825 50  0000 C CNN
+F 3 "" H 9050 825 50  0000 C CNN
+	1    9050 825
+	1    0    0    -1
+$EndComp
+NoConn ~ 9125 1075
 NoConn ~ 9125 2375
 NoConn ~ 9125 2475
 NoConn ~ 9125 2575
+NoConn ~ 9125 2675
 $Comp
 L GND #PWR056
 U 1 1 5983ED2F
-P 9050 2800
-F 0 "#PWR056" H 9050 2550 50  0001 C CNN
-F 1 "GND" H 9050 2650 50  0000 C CNN
-F 2 "" H 9050 2800 50  0000 C CNN
-F 3 "" H 9050 2800 50  0000 C CNN
-	1    9050 2800
-	1    0    0    -1
-$EndComp
-Text Label 8625 1375 0    50   ~ 0
+P 9050 2900
+F 0 "#PWR056" H 9050 2650 50  0001 C CNN
+F 1 "GND" H 9050 2750 50  0000 C CNN
+F 2 "" H 9050 2900 50  0000 C CNN
+F 3 "" H 9050 2900 50  0000 C CNN
+	1    9050 2900
+	1    0    0    -1
+$EndComp
+Text Label 8625 1475 0    50   ~ 0
 FONA_RST
-Text Label 8625 1475 0    50   ~ 0
+Text Label 8625 1575 0    50   ~ 0
 FONA_NS
-Text Label 8625 1575 0    50   ~ 0
+Text Label 8625 1675 0    50   ~ 0
 FONA_PS
-Text Label 8625 1675 0    50   ~ 0
+Text Label 8625 1775 0    50   ~ 0
 FONA_RX
-Text Label 8625 1775 0    50   ~ 0
+Text Label 8625 1875 0    50   ~ 0
 FONA_TX
-Text Label 8625 1875 0    50   ~ 0
+Text Label 8625 1975 0    50   ~ 0
 FONA_RTS
-Text Label 8625 1975 0    50   ~ 0
+Text Label 8625 2075 0    50   ~ 0
 FONA_RI
 Text HLabel 7875 5375 2    50   Input ~ 0
@@
 Text Notes 5925 4100 0    50   ~ 0
 ATSAM21G18 Cortex M0\n(Arduino-compatible)
-Text Notes 3750 925  0    200  ~ 0
+Text Notes 2575 925  0    200  ~ 0
 SHEET 3: MICROCONTROLLER
 $Comp
@@
 L +3.3V #PWR058
 U 1 1 597C444B
-P 8800 1025
-F 0 "#PWR058" H 8800 875 50  0001 C CNN
-F 1 "+3.3V" H 8800 1165 50  0000 C CNN
-F 2 "" H 8800 1025 50  0000 C CNN
-F 3 "" H 8800 1025 50  0000 C CNN
-	1    8800 1025
+P 8800 1125
+F 0 "#PWR058" H 8800 975 50  0001 C CNN
+F 1 "+3.3V" H 8800 1265 50  0000 C CNN
+F 2 "" H 8800 1125 50  0000 C CNN
+F 3 "" H 8800 1125 50  0000 C CNN
+	1    8800 1125
 	1    0    0    -1
 $EndComp
@@
 $EndComp
 NoConn ~ 7650 4625
-NoConn ~ 5450 4375
 $Comp
 L CAP-CER-1UF-25V-X7R-0805 C34
@@
 L AGND #PWR067
 U 1 1 598244CE
-P 5275 6325
-F 0 "#PWR067" H 5275 6075 50  0001 C CNN
-F 1 "AGND" H 5275 6175 50  0000 C CNN
-F 2 "" H 5275 6325 50  0000 C CNN
-F 3 "" H 5275 6325 50  0000 C CNN
-	1    5275 6325
+P 5275 6625
+F 0 "#PWR067" H 5275 6375 50  0001 C CNN
+F 1 "AGND" H 5275 6475 50  0000 C CNN
+F 2 "" H 5275 6625 50  0000 C CNN
+F 3 "" H 5275 6625 50  0000 C CNN
+	1    5275 6625
 	1    0    0    -1
 $EndComp
@@
 	9050 3400 9050 3450
 Wire Wire Line
-	7650 2625 8325 2625
-Wire Wire Line
-	7650 2525 8425 2525
-Wire Wire Line
 	7650 5175 7875 5175
 Wire Wire Line
@@
 Wire Wire Line
 	7850 4525 7650 4525
-Connection ~ 9050 2725
-Wire Wire Line
-	9050 1275 9050 2800
-Wire Wire Line
-	9050 2725 9125 2725
-Wire Wire Line
-	9125 1975 8625 1975
-Wire Wire Line
-	9125 1875 8525 1875
-Wire Wire Line
-	8425 1775 9125 1775
-Wire Wire Line
-	8325 1675 9125 1675
-Wire Wire Line
-	8225 1575 9125 1575
-Wire Wire Line
-	8125 1475 9125 1475
-Wire Wire Line
-	8025 1375 9125 1375
-Wire Wire Line
-	9125 1275 9050 1275
-Wire Wire Line
-	8800 1075 9125 1075
-Wire Wire Line
-	9050 725  9050 875
-Wire Wire Line
-	9050 875  9125 875
+Connection ~ 9050 2825
+Wire Wire Line
+	9050 1375 9050 2900
+Wire Wire Line
+	9050 2825 9125 2825
+Wire Wire Line
+	9125 2075 8625 2075
+Wire Wire Line
+	9125 1975 8525 1975
+Wire Wire Line
+	8425 1875 9125 1875
+Wire Wire Line
+	8325 1775 9125 1775
+Wire Wire Line
+	8225 1675 9125 1675
+Wire Wire Line
+	8125 1575 9125 1575
+Wire Wire Line
+	8025 1475 9125 1475
+Wire Wire Line
+	9125 1375 9050 1375
+Wire Wire Line
+	8800 1175 9125 1175
+Wire Wire Line
+	9050 825  9050 975
+Wire Wire Line
+	9050 975  9125 975
 Wire Wire Line
 	4825 6000 4925 6000
@@
 	8350 4775 7650 4775
 Wire Wire Line
-	7650 2225 8025 2225
-Wire Wire Line
-	8025 2225 8025 1375
-Wire Wire Line
-	8125 1475 8125 2325
-Wire Wire Line
-	8125 2325 7650 2325
-Wire Wire Line
-	7650 2425 8225 2425
-Wire Wire Line
-	8225 2425 8225 1575
-Wire Wire Line
-	8325 2625 8325 1675
-Wire Wire Line
-	8425 2525 8425 1775
-Wire Wire Line
-	8525 1875 8525 2725
-Wire Wire Line
-	8525 2725 7650 2725
-Wire Wire Line
-	7650 2825 8625 2825
-Wire Wire Line
-	8625 2825 8625 1975
+	7650 2250 8025 2250
+Wire Wire Line
+	8025 2250 8025 1475
+Wire Wire Line
+	8125 1575 8125 2850
+Wire Wire Line
+	8225 1675 8225 2750
+Wire Wire Line
+	8325 2350 8325 1775
+Wire Wire Line
+	8425 2450 8425 1875
+Wire Wire Line
+	8525 1975 8525 2550
+Wire Wire Line
+	8625 2075 8625 2650
 Wire Wire Line
 	9125 4775 9625 4775
@@
 	3300 2025 2675 2025
 Wire Wire Line
-	8800 1025 8800 1075
+	8800 1125 8800 1175
 Wire Wire Line
 	5375 1175 5375 2525
@@
 Connection ~ 5350 5225
 Wire Wire Line
-	5275 5025 5275 6325
+	5275 5025 5275 6625
 Wire Wire Line
 	5275 5025 5450 5025
 Wire Wire Line
-	4825 5400 4825 6325
+	4825 5400 4825 6625
 Wire Wire Line
 	5275 6225 5150 6225
@@
 3.3V
 Wire Wire Line
-	9050 775  8875 775
-Connection ~ 9050 775
-Text HLabel 8875 775  0    50   Input ~ 0
+	9050 875  8875 875
+Connection ~ 9050 875
+Text HLabel 8875 875  0    50   Input ~ 0
 5V
 $Comp
@@
 	9050 4125 7650 4125
 Connection ~ 9050 4025
+$Comp
+L FERRITE-BEAD-30-OHM-0805-1LN L5
+U 1 1 598AB532
+P 5050 6475
+F 0 "L5" V 5125 6475 50  0000 C CNN
+F 1 "FERRITE" V 4975 6475 50  0000 C CNN
+F 2 "Wickerlib:RLC-0805-SMD" H 5050 6125 50  0001 C CIN
+F 3 "http://www.bourns.com/docs/Product-Datasheets/mh.pdf" H 5050 6475 5   0001 C CNN
+F 4 "FERRITE BEAD 30 OHM 0805 1LN" H 5050 6125 50  0001 C CIN "Description"
+F 5 "Bourns" H 5050 6125 50  0001 C CIN "MF_Name"
+F 6 "MH2029-300Y" H 5050 6125 50  0001 C CIN "MF_PN"
+F 7 "Digikey" H 5050 6125 50  0001 C CIN "S1_Name"
+F 8 "MH2029-300YCT-ND" H 5050 6125 50  0001 C CIN "S1_PN"
+	1    5050 6475
+	0    -1   -1   0
+$EndComp
+Wire Wire Line
+	5150 6475 5275 6475
+Connection ~ 5275 6475
+Wire Wire Line
+	4950 6475 4825 6475
+Connection ~ 4825 6475
+Wire Wire Line
+	7650 2350 8325 2350
+Wire Wire Line
+	8125 2850 7650 2850
+Wire Wire Line
+	8225 2750 7650 2750
+Wire Wire Line
+	8625 2650 7650 2650
+Wire Wire Line
+	8525 2550 7650 2550
+Wire Wire Line
+	8425 2450 7650 2450
+NoConn ~ 7650 2975
+NoConn ~ 7650 3075
+NoConn ~ 7650 3975
 $EndSCHEMATC

Commit message: Commit.
Connections:
- net ~PG: now also U6.41 (PA28)
- no-connect marks 19 -> 17
Changed lines of the file:
@@
 EESchema Schematic File Version 2
 LIBS:wickerlib
-LIBS:mcphail-main-board-cache
 EELAYER 25 0
 EELAYER END
@@
 Text HLabel 7875 5175 2    50   Input ~ 0
 A2
-Text HLabel 7850 4525 2    50   Input ~ 0
+Text HLabel 7850 3275 2    50   Input ~ 0
 ~PG
 Text Label 7725 5375 0    50   ~ 0
@@
 Text Label 1450 3850 0    50   ~ 0
 A2
-Text Label 7725 4525 0    50   ~ 0
+Text Label 7725 3275 0    50   ~ 0
 ~PG
 $Comp
@@
 	1    0    0    -1
 $EndComp
-NoConn ~ 7650 4625
 $Comp
 L CAP-CER-1UF-25V-X7R-0805 C34
@@
 	7650 5375 7875 5375
 Wire Wire Line
-	7850 4525 7650 4525
+	7850 3275 7650 3275
 Connection ~ 9050 2825
 Wire Wire Line
@@
 $EndComp
 NoConn ~ 7650 3175
-NoConn ~ 7650 3275
 NoConn ~ 7650 3375
 NoConn ~ 7650 3475

Commit message: temp
Parts:
- J6: MF_Name TE Conn -> Harwin; MF_PN 7-215079-6 -> M20-9720345; S1_PN A30729CT-ND -> 952-1921-ND
Changed lines of the file:
@@
 F 3 "http://www.te.com/commerce/DocumentDelivery/DDEController?Action=srchrtrv&DocNm=215079&DocType=Customer+Drawing&DocLang=English" H 5825 6425 5   0001 C CNN
 F 4 "HEADER FEMALE 6POS 2x3 0.1IN" H 5825 6075 50  0001 C CIN "Description"
-F 5 "TE Conn" H 5825 6075 50  0001 C CIN "MF_Name"
-F 6 "7-215079-6" H 5825 6075 50  0001 C CIN "MF_PN"
+F 5 "Harwin" H 5825 6075 50  0001 C CIN "MF_Name"
+F 6 "M20-9720345" H 5825 6075 50  0001 C CIN "MF_PN"
 F 7 "Digikey" H 5825 6075 50  0001 C CIN "S1_Name"
-F 8 "A30729CT-ND" H 5825 6075 50  0001 C CIN "S1_PN"
+F 8 "952-1921-ND" H 5825 6075 50  0001 C CIN "S1_PN"
 	1    5825 6425
 	1    0    0    -1
