File: hardware/mcphail-main-board/mcphail-main-board.kicad_pcb (KiCad board)
At the start: 2 copper layers, 101.6 x 101.6 mm, 141 parts, among them J1 INSECT DETECTION, J10 BREAKOUT, J2 EMITTERS, J3 BREAKOUT, J4 MICRO SD, J5 MICRO USB, J6 SWD, J7 FONA 808, J8 INPUT 6V-9V, J9 JST PH, U1 MCP6004, U10 BUCK-BOOST 5V TPS63060, U11 MCP1703, U2 MCP6004, U3 TLV274, U4 MCP6001, U5 ADS1118, U6 ATSAMD21G18A, U7 24AA1025 EEPROM, U8 MCP7940N RTC, U9 MCP73871, X1 16MHz, X2 32.768kHz

Commit message: Lots more layout work, needs rework.
Parts:
- removed C32: 100nF, Wickerlib:RLC-0603-SMD
- removed J10: BREAKOUT, Wickerlib:CONN-HEADER-STRAIGHT-P2.54MM-1x10
- added FID1: FIDUCIAL, Wickerlib:FIDUCIAL-2MM, F.Cu at (171.8, 51.1)
- added FID2: FIDUCIAL, Wickerlib:FIDUCIAL-2MM, F.Cu at (243.8, 95.5)
- added FID3: FIDUCIAL, Wickerlib:FIDUCIAL-2MM, F.Cu at (171.2, 95.5)
- J6: value SWD -> PROG/BOOT; footprint Wickerlib:CONN-HEADER-STRAIGHT-P2.54MM-1x05 -> Wickerlib:CONN-HEADER-STRAIGHT-P2.54MM-2x03
- U5: footprint Wickerlib:SOIC-14-3.9x8.7MM-P1.27MM -> Wickerlib:MSOP-10-3x3MM-P0.5MM
- moved J1 227.0 mm to (237.7, 82.0), turned to 270 degrees
- moved C2 199.9 mm to (235.7, 85.2), turned to 0 degrees
- moved C7 197.6 mm to (232.2, 91.3), turned to 90 degrees
- moved R2 196.2 mm to (234.9, 87.5), turned to 0 degrees
- moved C3 195.2 mm to (236.3, 89.5), turned to 180 degrees
- moved C16 192.4 mm to (229.1, 91.6)
- moved C17 192.2 mm to (229.1, 86.8), turned to 270 degrees
- moved C19 191.8 mm to (225.9, 84.8), turned to 270 degrees
- moved U4 191.5 mm to (235.7, 92.0), turned to 0 degrees
- moved L3 191.3 mm to (207.0, 77.5), turned to 180 degrees
- moved C13 186.6 mm to (228.1, 95.2), turned to 180 degrees
- moved R16 184.7 mm to (223.3, 85.5), turned to 270 degrees
- moved J9 184.2 mm to (204.5, 47.6), turned to 180 degrees
- moved R12 183.9 mm to (226.6, 92.3), turned to 90 degrees
- moved C20 183.5 mm to (221.8, 82.7)
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Connections:
- net /Microcontroller/USB_D+ renamed /Microcontroller/D+
- net /Microcontroller/USB_D- renamed /Microcontroller/D-
- C25 pad 2: GND -> AGND
- C26 pad 2: GND -> AGND
- C30 pad 2: GND -> AGND
- J4 pad 2: /Microcontroller/D4_CS -> /Microcontroller/D7_CS
- J6 pad 3: /Microcontroller/SWCLK -> (no net)
- J6 pad 4: /Microcontroller/~RESET -> /Microcontroller/SWCLK
- R41 pad 2: /~PG -> /Input Power/~PG1
- U2 pad 13: Net-(C18-Pad2) -> Net-(C8-Pad2)
- U2 pad 14: /Photodiode Signal Input Conditioning/LINE_IN -> Net-(C8-Pad1)
- U2 pad 6: Net-(C8-Pad2) -> Net-(C18-Pad2)
- U2 pad 7: Net-(C8-Pad1) -> /Photodiode Signal Input Conditioning/LINE_IN
- U3 pad 10: Net-(U3-Pad10) -> (no net)
- U3 pad 12: (no net) -> Net-(U3-Pad12)
- U3 pad 13: (no net) -> /A1
- U3 pad 14: (no net) -> /A2
- U3 pad 3: Net-(U3-Pad10) -> Net-(U3-Pad12)
- U3 pad 6: Net-(U3-Pad10) -> Net-(U3-Pad12)
- U3 pad 7: Net-(U3-Pad10) -> Net-(U3-Pad12)
- U3 pad 8: /A2 -> (no net)
- U3 pad 9: /A1 -> (no net)
- U5 pad 3: GND -> AGND
- U6 pad 1: Net-(J10-Pad6) -> /Microcontroller/EEPROM_A0
- U6 pad 10: /Microcontroller/EEPROM_A2 -> /A2
- U6 pad 11: /Microcontroller/EEPROM_A1 -> /A1
- U6 pad 12: /Microcontroller/EEPROM_A0 -> /A0
- U6 pad 14: /A2 -> /Microcontroller/MFP
- U6 pad 15: /A1 -> /~PG
- U6 pad 16: /A0 -> (no net)
- U6 pad 2: Net-(J10-Pad7) -> (no net)
- U6 pad 25: /Microcontroller/SCL -> /Microcontroller/SDA
- U6 pad 26: /Microcontroller/MFP -> /Microcontroller/SCL
- U6 pad 3: Net-(J10-Pad8) -> (no net)
- U6 pad 30: /Microcontroller/D4_CS -> /Microcontroller/D7_CS
- U6 pad 39: Net-(J10-Pad2) -> (no net)
- U6 pad 4: Net-(J10-Pad9) -> (no net)
- U6 pad 41: Net-(J10-Pad3) -> (no net)
- U6 pad 47: Net-(J10-Pad4) -> /Microcontroller/EEPROM_A2
- U6 pad 48: Net-(J10-Pad5) -> /Microcontroller/EEPROM_A1
- U6 pad 7: /Microcontroller/SDA -> (no net)
- U6 pad 8: /~PG -> (no net)
- U9 pad 6: /~PG -> /Input Power/~PG1
Routing:
- net GND: track 0.00 -> 183.9 mm, vias 0 -> 46
- net +5V: track 0.00 -> 144.0 mm, vias 0 -> 9
- net +3V3: track 0.00 -> 127.4 mm, vias 0 -> 7
- net /Photodiode Signal Input Conditioning/VREF: track 0.00 -> 82.3 mm, vias 0 -> 4
- net /A0: track 0.00 -> 54.3 mm, vias 0 -> 1
- net AGND: track 0.00 -> 50.9 mm, vias 0 -> 20
- net /Microcontroller/D-: track 0.00 -> 50.6 mm, vias 0 -> 2
- net /Microcontroller/D+: track 0.00 -> 49.6 mm, vias 0 -> 2
- net /A2: track 0.00 -> 48.1 mm, vias 0 -> 2
- net VIN: track 0.00 -> 40.2 mm, vias 0 -> 6
- net /Input Power/VCC: track 0.00 -> 38.9 mm, vias 0 -> 5
- net /~PG: track 0.00 -> 35.4 mm, vias 0 -> 2
- net /A1: track 0.00 -> 35.3 mm, vias 0 -> 2
- net /Microcontroller/~RESET: track 0.00 -> 31.6 mm
- net /Microcontroller/D7_CS: track 0.00 -> 31.1 mm, vias 0 -> 2
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- added copper zone on B.Cu, net AGND
- added copper zone on F.Cu, net AGND
Other:
- board size 101.6 x 101.6 mm -> 80.6 x 56.6 mm
- net class Default: clearance 0.2032 -> 0.0254
- rule trace_clearance: 0.2032 -> 0.0254
- board text added: "9V MAX"
- board text added: "GND"
- board text added: "SIG"
- board text removed: "EMITTER"

Commit message: Saving main board layout before major rework.
Parts:
- moved C22 33.3 mm to (202.9, 78.4)
- moved L3 11.3 mm to (196.2, 74.0), turned to 270 degrees
- moved J3 4.44 mm to (186.8, 77.0)
Routing:
- net +5V: track 144.0 -> 267.5 mm, vias 9 -> 10
- net +3V3: track 127.4 -> 196.2 mm, vias 7 -> 8
- net /Microcontroller/MISO: track 3.34 -> 46.0 mm, vias 2 -> 3
- net /Microcontroller/MOSI: track 2.77 -> 41.0 mm, vias 2 -> 3
- net /Microcontroller/MFP: track 6.69 -> 35.1 mm, vias 0 -> 2
- net /Microcontroller/SCLK: track 11.1 -> 37.3 mm
- net Net-(BAT1-Pad1): track 15.7 -> 38.7 mm
- net /A1: track 35.3 -> 55.4 mm, vias 2 -> 1
- net /A2: track 48.1 -> 53.4 mm, vias 2 -> 1
- net VIN: track 40.2 -> 45.2 mm
- net /Photodiode Signal Input Conditioning/LINE_IN: track 4.41 -> 9.27 mm
- net /A0: track 54.3 -> 57.1 mm, vias 1 -> 2
- net Net-(C2-Pad1): track 5.72 -> 8.02 mm
- net GND: track 183.9 -> 181.8 mm, vias 46 -> 47
- net (no net): track 0.00 -> 0.87 mm

Commit message: Regenerated sch pdf. Converted to 4 layer.
Routing:
- net /Microcontroller/MISO: track 46.0 -> 37.8 mm
- net GND: track 181.8 -> 182.3 mm
- added copper zone on In1.Cu, net AGND
- added copper zone on In2.Cu, net AGND
Other:
- copper layers 2 -> 4
Changed lines of the file:
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@@
     (thickness 1.6)
     (drawings 28)
-    (tracks 1354)
+    (tracks 1353)
     (zones 0)
     (modules 142)
@@
   (layers
     (0 F.Cu signal)
+    (1 In1.Cu signal)
+    (2 In2.Cu signal)
     (31 B.Cu signal)
     (34 B.Paste user)
@@
   (segment (start 237.1624 70.5398) (end 237.1624 69.8858) (width 0.254) (layer F.Cu) (net 1))
   (segment (start 237.1624 69.8858) (end 237.1624 65.6898) (width 0.254) (layer F.Cu) (net 1))
-  (segment (start 211.973929 71.098749) (end 211.488996 71.098749) (width 0.254) (layer B.Cu) (net 2))
-  (segment (start 211.984251 71.098749) (end 211.973929 71.098749) (width 0.254) (layer B.Cu) (net 2))
-  (via (at 211.488996 71.098749) (size 0.6858) (drill 0.3302) (layers F.Cu B.Cu) (net 2))
-  (segment (start 211.488996 70.613816) (end 211.488996 71.098749) (width 0.254) (layer F.Cu) (net 2))
-  (segment (start 211.488996 70.285656) (end 211.488996 70.613816) (width 0.254) (layer F.Cu) (net 2))
-  (segment (start 212.217 70.866) (end 211.984251 71.098749) (width 0.254) (layer B.Cu) (net 2))
-  (segment (start 211.440298 70.236958) (end 211.488996 70.285656) (width 0.254) (layer F.Cu) (net 2))
+  (segment (start 211.922615 71.443129) (end 211.922615 70.958196) (width 0.254) (layer B.Cu) (net 2))
+  (segment (start 211.440298 70.236958) (end 211.440298 70.761958) (width 0.254) (layer F.Cu) (net 2))
+  (via (at 211.922615 71.443129) (size 0.6858) (drill 0.3302) (layers F.Cu B.Cu) (net 2))
+  (segment (start 212.014811 70.866) (end 212.217 70.866) (width 0.254) (layer B.Cu) (net 2))
+  (segment (start 211.922615 71.244275) (end 211.922615 71.443129) (width 0.254) (layer F.Cu) (net 2))
+  (segment (start 211.922615 70.958196) (end 212.014811 70.866) (width 0.254) (layer B.Cu) (net 2))
+  (segment (start 211.440298 70.761958) (end 211.922615 71.244275) (width 0.254) (layer F.Cu) (net 2))
   (segment (start 242.824 49.716) (end 242.824 51.562) (width 0.254) (layer F.Cu) (net 2))
   (segment (start 242.934 49.606) (end 242.824 49.716) (width 0.254) (layer F.Cu) (net 2))
@@
   (segment (start 185.877156 87.324614) (end 187.970856 87.324614) (width 0.254) (layer F.Cu) (net 53))
   (segment (start 187.970856 87.324614) (end 187.995556 87.299914) (width 0.254) (layer F.Cu) (net 53))
-  (segment (start 213.332399 71.594059) (end 206.317992 71.594059) (width 0.254) (layer B.Cu) (net 54))
-  (segment (start 213.675298 71.936958) (end 213.332399 71.594059) (width 0.254) (layer B.Cu) (net 54))
-  (segment (start 206.161433 71.4375) (end 205.6765 71.4375) (width 0.254) (layer B.Cu) (net 54))
-  (segment (start 206.317992 71.594059) (end 206.161433 71.4375) (width 0.254) (layer B.Cu) (net 54))
   (segment (start 200.938193 70.013776) (end 202.361917 71.4375) (width 0.254) (layer F.Cu) (net 54))
   (segment (start 202.361917 71.4375) (end 205.6765 71.4375) (width 0.254) (layer F.Cu) (net 54))
@@
   (segment (start 204.104298 70.248958) (end 208.928298 70.248958) (width 0.254) (layer F.Cu) (net 56))
   (segment (start 208.928298 70.248958) (end 208.940298 70.236958) (width 0.254) (layer F.Cu) (net 56))
-  (segment (start 205.995459 72.089369) (end 206.480392 72.089369) (width 0.254) (layer F.Cu) (net 57))
-  (segment (start 199.628192 71.478068) (end 200.239493 72.089369) (width 0.254) (layer F.Cu) (net 57))
-  (segment (start 200.239493 72.089369) (end 205.995459 72.089369) (width 0.254) (layer F.Cu) (net 57))
-  (segment (start 212.59302 71.41468) (end 212.59302 71.604436) (width 0.254) (layer F.Cu) (net 57))
-  (via (at 212.59302 72.089369) (size 0.6858) (drill 0.3302) (layers F.Cu B.Cu) (net 57))
-  (via (at 206.480392 72.089369) (size 0.6858) (drill 0.3302) (layers F.Cu B.Cu) (net 57))
-  (segment (start 212.59302 71.604436) (end 212.59302 72.089369) (width 0.254) (layer F.Cu) (net 57))
-  (segment (start 211.940298 70.761958) (end 212.59302 71.41468) (width 0.254) (layer F.Cu) (net 57))
-  (segment (start 211.940298 70.236958) (end 211.940298 70.761958) (width 0.254) (layer F.Cu) (net 57))
-  (segment (start 212.59302 72.089369) (end 206.480392 72.089369) (width 0.254) (layer B.Cu) (net 57))
+  (via (at 206.883 71.8185) (size 0.6858) (drill 0.3302) (layers F.Cu B.Cu) (net 57))
+  (segment (start 212.190365 71.936958) (end 212.675298 71.936958) (width 0.254) (layer B.Cu) (net 57))
+  (segment (start 206.540101 72.161399) (end 206.883 71.8185) (width 0.254) (layer F.Cu) (net 57))
+  (segment (start 212.188884 71.938439) (end 212.190365 71.936958) (width 0.254) (layer B.Cu) (net 57))
+  (segment (start 211.548821 71.8185) (end 211.66876 71.938439) (width 0.254) (layer B.Cu) (net 57))
+  (segment (start 212.675298 71.462764) (end 212.675298 71.936958) (width 0.254) (layer F.Cu) (net 57))
+  (segment (start 211.66876 71.938439) (end 212.188884 71.938439) (width 0.254) (layer B.Cu) (net 57))
+  (segment (start 199.628192 71.478068) (end 200.311523 72.161399) (width 0.254) (layer F.Cu) (net 57))
+  (segment (start 200.311523 72.161399) (end 206.540101 72.161399) (width 0.254) (layer F.Cu) (net 57))
+  (segment (start 211.940298 70.236958) (end 211.940298 70.727764) (width 0.254) (layer F.Cu) (net 57))
+  (segment (start 211.940298 70.727764) (end 212.675298 71.462764) (width 0.254) (layer F.Cu) (net 57))
+  (segment (start 206.883 71.8185) (end 211.548821 71.8185) (width 0.254) (layer B.Cu) (net 57))
+  (via (at 212.675298 71.936958) (size 0.6858) (drill 0.3302) (layers F.Cu B.Cu) (net 57))
   (segment (start 223.8375 60.3885) (end 221.9325 62.2935) (width 0.254) (layer F.Cu) (net 57))
   (segment (start 223.8375 58.8645) (end 223.8375 60.3885) (width 0.254) (layer F.Cu) (net 57))
@@
     (polygon
       (pts
-        (xy 248.92 41.91) (xy 167.64 41.91) (xy 167.64 99.06) (xy 250.19 99.06)
-      )
-    )
-  )
-  (zone (net 2) (net_name GND) (layer B.Cu) (hatch edge 0.508)
-    (connect_pads (clearance 0.508))
-    (min_thickness 0.254)
-    (fill yes (arc_segments 16) (thermal_gap 0.508) (thermal_bridge_width 0.508))
-    (polygon
-      (pts
-        (xy 248.92 41.91) (xy 167.64 41.91) (xy 167.64 99.06) (xy 250.19 99.06)
+        (xy 248.92 41.91) (xy 167.64 41.91) (xy 167.64 99.06) (xy 247.65 99.06)
       )
     )
@@
     (priority 1)
     (connect_pads (clearance 0.508))
+    (min_thickness 0.254)
+    (fill yes (arc_segments 16) (thermal_gap 0.508) (thermal_bridge_width 0.508))
+    (polygon
+      (pts
+        (xy 171.45 74.295) (xy 200.66 74.295) (xy 200.66 63.5) (xy 205.74 63.5) (xy 207.264 63.5)
+        (xy 207.264 76.2) (xy 207.264 78.74) (xy 241.3 78.74) (xy 241.3 95.25) (xy 171.45 95.25)
+      )
+    )
+  )
+  (zone (net 2) (net_name GND) (layer B.Cu) (hatch edge 0.508)
+    (connect_pads (clearance 0.508))
+    (min_thickness 0.254)
+    (fill yes (arc_segments 16) (thermal_gap 0.508) (thermal_bridge_width 0.508))
+    (polygon
+      (pts
+        (xy 248.92 41.91) (xy 167.64 41.91) (xy 167.64 99.06) (xy 247.65 99.06)
+      )
+    )
+  )
+  (zone (net 7) (net_name AGND) (layer In1.Cu) (hatch edge 0.508)
+    (priority 1)
+    (connect_pads (clearance 0.508))
+    (min_thickness 0.254)
+    (fill yes (arc_segments 16) (thermal_gap 0.508) (thermal_bridge_width 0.508))
+    (polygon
+      (pts
+        (xy 171.45 74.295) (xy 200.66 74.295) (xy 200.66 63.5) (xy 205.74 63.5) (xy 207.264 63.5)
+        (xy 207.264 76.2) (xy 207.264 78.74) (xy 241.3 78.74) (xy 241.3 95.25) (xy 171.45 95.25)
+      )
+    )
+  )
+  (zone (net 7) (net_name AGND) (layer In2.Cu) (hatch edge 0.508)
+    (priority 1)
+    (connect_pads (clearance 0.508))
