File: hardware/mcphail-main-board/mcphail-main-board.kicad_pcb (KiCad board)
At the start: 4 copper layers, 80.6 x 56.6 mm, 142 parts, among them J1 INSECT DETECTION, J2 EMITTERS, J3 BREAKOUT, J4 MICRO SD, J5 MICRO USB, J6 PROG/BOOT, J7 FONA 808, J8 INPUT 6V-9V, J9 JST PH, U1 MCP6004, U10 BUCK-BOOST 5V TPS63060, U11 MCP1703, U2 MCP6004, U3 TLV274, U4 MCP6001, U5 ADS1118, U6 ATSAMD21G18A, U7 24AA1025 EEPROM, U8 MCP7940N RTC, U9 MCP73871, X1 16MHz, X2 32.768kHz

Commit message: Reworking main board, power rails routed next.
Parts:
- moved J2 64.4 mm to (228.6, 99.1), turned to 90 degrees
- moved R1 60.1 mm to (230.3, 95.3), turned to 180 degrees
- moved C41 52.6 mm to (258.7, 23.3), turned to 0 degrees
- moved C1 49.7 mm to (229.8, 87.7), turned to 90 degrees
- moved R37 44.3 mm to (252.4, 23.3), turned to 0 degrees
- moved C39 40.4 mm to (234.0, 64.1), turned to 270 degrees
- moved J4 39.1 mm to (217.8, 81.4), turned to 0 degrees
- moved J1 38.9 mm to (201.2, 95.4)
- moved R29 38.3 mm to (173.0, 75.7), turned to 180 degrees
- moved R27 37.1 mm to (173.0, 77.4), turned to 180 degrees
- moved C11 36.5 mm to (187.8, 92.3)
- moved C13 36.5 mm to (191.6, 94.1)
- moved C19 36.5 mm to (189.3, 83.7)
- moved C20 36.5 mm to (185.3, 81.6)
- moved C23 36.5 mm to (176.9, 83.4)
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Connections:
- C25 pad 1: +3V3 -> /VDDANA
- C26 pad 1: +3V3 -> /VDDANA
- C31 pad 1: /Microcontroller/VDDANA -> /VDDANA
- C52 pad 1: /Microcontroller/VDDANA -> /VDDANA
- J3 pad 2: +3V3 -> /VDDANA
- J7 pad 11: /Microcontroller/FONA_PS -> (no net)
- J7 pad 12: /Microcontroller/FONA_NS -> (no net)
- J7 pad 5: /Microcontroller/FONA_RST -> (no net)
- J7 pad 6: /Microcontroller/FONA_RX -> (no net)
- J7 pad 7: /Microcontroller/FONA_TX -> (no net)
- L4 pad 1: /Microcontroller/VDDANA -> /VDDANA
- R18 pad 1: +3V3 -> /VDDANA
- R20 pad 1: +3V3 -> /VDDANA
- U3 pad 4: +3V3 -> /VDDANA
- U6 pad 1: /Microcontroller/EEPROM_A0 -> (no net)
- U6 pad 14: /Microcontroller/MFP -> (no net)
- U6 pad 20: /Microcontroller/SCLK -> /Microcontroller/MFP
- U6 pad 21: /Microcontroller/MISO -> /Microcontroller/SDA
- U6 pad 22: /Microcontroller/FONA_RST -> /Microcontroller/SCL
- U6 pad 25: /Microcontroller/SDA -> (no net)
- U6 pad 26: /Microcontroller/SCL -> (no net)
- U6 pad 27: /Microcontroller/FONA_NS -> /Microcontroller/EEPROM_ADD2
- U6 pad 28: /Microcontroller/FONA_PS -> /Microcontroller/EEPROM_ADD1
- U6 pad 29: /Microcontroller/FONA_TX -> /Microcontroller/EEPROM_ADD0
- U6 pad 31: /Microcontroller/FONA_RX -> (no net)
- U6 pad 47: /Microcontroller/EEPROM_A2 -> (no net)
- U6 pad 48: /Microcontroller/EEPROM_A1 -> (no net)
- U6 pad 6: /Microcontroller/VDDANA -> /VDDANA
- U7 pad 1: /Microcontroller/EEPROM_A0 -> /Microcontroller/EEPROM_ADD0
- U7 pad 2: /Microcontroller/EEPROM_A1 -> /Microcontroller/EEPROM_ADD1
- U7 pad 3: /Microcontroller/EEPROM_A2 -> /Microcontroller/EEPROM_ADD2
Routing:
- net +5V: track 267.5 -> 58.4 mm, vias 10 -> 8
- net +3V3: track 196.2 -> 3.07 mm, vias 8 -> 0
- net GND: track 182.3 -> 4.95 mm, vias 47 -> 2
- net VIN: track 45.2 -> 0.00 mm, vias 6 -> 0
- net /Microcontroller/MOSI: track 41.2 -> 0.00 mm, vias 3 -> 0
- net /Input Power/VCC: track 38.9 -> 0.00 mm, vias 5 -> 0
- net Net-(BAT1-Pad1): track 38.7 -> 0.00 mm, vias 1 -> 0
- net /Microcontroller/MISO: track 37.8 -> 0.00 mm, vias 3 -> 0
- net /Microcontroller/SCLK: track 37.3 -> 0.00 mm, vias 2 -> 0
- net /~PG: track 35.4 -> 0.00 mm, vias 2 -> 0
- net /Microcontroller/MFP: track 35.1 -> 0.00 mm, vias 2 -> 0
- net /A1: track 55.4 -> 20.9 mm, vias 1 -> 2
- net /Microcontroller/~RESET: track 31.6 -> 0.00 mm
- net /Microcontroller/D7_CS: track 31.1 -> 0.00 mm, vias 2 -> 0
- net /VDDANA: track 0.00 -> 27.9 mm, vias 0 -> 2
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- removed copper zone on B.Cu, net AGND
- removed copper zone on B.Cu, net GND
- removed copper zone on F.Cu, net GND

Commit message: Generate Main Board with traces done. Needs silk.
Parts:
- added L5: FERRITE, Wickerlib:RLC-0805-SMD, F.Cu at (211.1, 92.9)
- moved C41 63.0 mm to (231.9, 80.2)
- moved R37 63.0 mm to (225.5, 80.2)
- moved BAT1 62.7 mm to (226.0, 87.4)
- moved U11 34.5 mm to (237.1, 55.2)
- moved C49 34.5 mm to (237.3, 52.2)
- moved C50 34.5 mm to (237.1, 58.2)
- moved C46 30.1 mm to (220.8, 50.8), turned to 270 degrees
- moved C53 29.9 mm to (218.6, 50.8), turned to 270 degrees
- moved J9 28.7 mm to (211.7, 48.4)
- moved L2 28.0 mm to (224.2, 46.0)
- moved C48 28.0 mm to (231.1, 53.6)
- moved C54 28.0 mm to (235.9, 47.0)
- moved R45 28.0 mm to (232.8, 50.5)
- moved R46 28.0 mm to (230.4, 51.2)
- moved R47 28.0 mm to (233.4, 52.8)
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Connections:
- J7 pad 11: (no net) -> /Microcontroller/FONA_PS
- J7 pad 12: (no net) -> /Microcontroller/FONA_NS
- J7 pad 5: (no net) -> /Microcontroller/FONA_RST
- J7 pad 6: (no net) -> /Microcontroller/FONA_RX
- J7 pad 7: (no net) -> /Microcontroller/FONA_TX
- U6 pad 14: (no net) -> /Microcontroller/SCLK
- U6 pad 15: /~PG -> /Microcontroller/MISO
- U6 pad 25: (no net) -> /Microcontroller/D7_CS
- U6 pad 26: (no net) -> /Microcontroller/FONA_NS
- U6 pad 27: /Microcontroller/EEPROM_ADD2 -> /Microcontroller/FONA_PS
- U6 pad 28: /Microcontroller/EEPROM_ADD1 -> /Microcontroller/FONA_RI
- U6 pad 29: /Microcontroller/EEPROM_ADD0 -> /Microcontroller/FONA_RTS
- U6 pad 30: /Microcontroller/D7_CS -> /Microcontroller/FONA_TX
- U6 pad 31: (no net) -> /Microcontroller/FONA_RX
- U6 pad 32: (no net) -> /Microcontroller/FONA_RST
- U6 pad 37: /Microcontroller/FONA_RTS -> /Microcontroller/EEPROM_ADD2
- U6 pad 38: /Microcontroller/FONA_RI -> /Microcontroller/EEPROM_ADD1
- U6 pad 39: (no net) -> /Microcontroller/EEPROM_ADD0
Routing:
- net +3V3: track 3.07 -> 156.1 mm, vias 0 -> 9
- net +5V: track 58.4 -> 205.3 mm, vias 8 -> 10
- net GND: track 4.95 -> 126.2 mm, vias 2 -> 44
- net /Microcontroller/SCLK: track 0.00 -> 40.6 mm, vias 0 -> 3
- net Net-(BAT1-Pad1): track 0.00 -> 38.7 mm, vias 0 -> 1
- net /Microcontroller/FONA_PS: track 0.00 -> 38.5 mm, vias 0 -> 3
- net /Input Power/VCC: track 0.00 -> 38.3 mm
- net /Microcontroller/FONA_NS: track 0.00 -> 36.6 mm, vias 0 -> 2
- net VIN: track 0.00 -> 35.6 mm, vias 0 -> 2
- net /Microcontroller/MISO: track 0.00 -> 34.3 mm, vias 0 -> 2
- net /Microcontroller/D7_CS: track 0.00 -> 30.8 mm, vias 0 -> 2
- net /Microcontroller/FONA_RTS: track 0.00 -> 29.5 mm, vias 0 -> 2
- net /Microcontroller/FONA_RI: track 0.00 -> 28.9 mm
- net /Microcontroller/SDA: track 0.00 -> 28.5 mm, vias 0 -> 6
- net /Microcontroller/MOSI: track 0.00 -> 28.4 mm, vias 0 -> 2
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- added copper zone on B.Cu, net AGND
- added copper zone on B.Cu, net GND
- added copper zone on F.Cu, net GND
- removed copper zone on In1.Cu, net AGND
- removed copper zone on In2.Cu, net AGND
Other:
- copper layers 4 -> 2

Commit message: Major updates to README.
Parts:
- moved C40 0.74 mm to (238.8, 75.6), turned to 270 degrees
- moved C42 0.05 mm to (238.7, 72.4), turned to 90 degrees
Routing:
- net Net-(C42-Pad1): track 7.97 -> 11.2 mm
- net Net-(C40-Pad1): track 11.8 -> 12.7 mm
- net GND: track 126.2 -> 126.7 mm, vias 44 -> 45
Changed lines of the file:
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@@
     (links 335)
     (no_connects 0)
-    (area 167.563799 41.722878 248.365056 98.505056)
+    (area 104.572999 40.039358 248.365056 123.265001)
     (thickness 1.6)
     (drawings 28)
-    (tracks 1457)
+    (tracks 1475)
     (zones 0)
     (modules 143)
@@
   )
   (module Wickerlib:RLC-0603-SMD (layer F.Cu)
-    (at 238.7814 76.3416 90)
+    (at 238.76 75.6038 270)
     (descr "Capacitor SMD RLC-0603-SMD, reflow soldering, AVX (see smccp.pdf)")
     (tags "capacitor RLC-0603-SMD")
     (attr smd)
-    (fp_text reference C40 (at 0.09 0.04 90) (layer F.Fab)
+    (fp_text reference C40 (at 0.09 0.04 270) (layer F.Fab)
       (effects (font (size 0.8 0.8) (thickness 0.15)))
     )
-    (fp_text value 2pF (at 0 1.9 90) (layer F.Fab) hide
+    (fp_text value 2pF (at 0 1.9 270) (layer F.Fab) hide
       (effects (font (size 1 1) (thickness 0.15)))
     )
     (fp_line (start -1.397 -0.635) (end -1.397 0.635) (layer F.SilkS) (width 0.1524))
     (fp_line (start 1.3335 -0.635) (end 1.3335 0.635) (layer F.SilkS) (width 0.1524))
-    (fp_text user %R (at 0.012 1.6256 90) (layer F.SilkS)
+    (fp_text user %R (at 0.012 1.6256 270) (layer F.SilkS)
       (effects (font (size 1 1) (thickness 0.15)))
     )
@@
     (fp_line (start 1.45 -0.75) (end 1.45 0.75) (layer F.Fab) (width 0.05))
     (fp_line (start -1.45 0.75) (end 1.45 0.75) (layer F.Fab) (width 0.05))
-    (pad 1 smd rect (at -0.75 0 90) (size 0.8 0.75) (layers F.Cu F.Paste F.Mask)
+    (pad 1 smd rect (at -0.75 0 270) (size 0.8 0.75) (layers F.Cu F.Paste F.Mask)
       (net 37 "Net-(C40-Pad1)"))
-    (pad 2 smd rect (at 0.75 0 90) (size 0.8 0.75) (layers F.Cu F.Paste F.Mask)
+    (pad 2 smd rect (at 0.75 0 270) (size 0.8 0.75) (layers F.Cu F.Paste F.Mask)
       (net 2 GND))
   )
@@
   )
   (module Wickerlib:RLC-0603-SMD (layer F.Cu)
-    (at 238.7814 72.4554 270)
+    (at 238.7346 72.4274 90)
     (descr "Capacitor SMD RLC-0603-SMD, reflow soldering, AVX (see smccp.pdf)")
     (tags "capacitor RLC-0603-SMD")
     (attr smd)
-    (fp_text reference C42 (at 0.09 0.04 270) (layer F.Fab)
+    (fp_text reference C42 (at 0.09 0.04 90) (layer F.Fab)
       (effects (font (size 0.8 0.8) (thickness 0.15)))
     )
-    (fp_text value 2pF (at 0 1.9 270) (layer F.Fab) hide
+    (fp_text value 2pF (at 0 1.9 90) (layer F.Fab) hide
       (effects (font (size 1 1) (thickness 0.15)))
     )
     (fp_line (start -1.397 -0.635) (end -1.397 0.635) (layer F.SilkS) (width 0.1524))
     (fp_line (start 1.3335 -0.635) (end 1.3335 0.635) (layer F.SilkS) (width 0.1524))
-    (fp_text user %R (at 0.0134 -1.6002 270) (layer F.SilkS)
+    (fp_text user %R (at 0.0134 -1.6002 90) (layer F.SilkS)
       (effects (font (size 1 1) (thickness 0.15)))
     )
@@
     (fp_line (start 1.45 -0.75) (end 1.45 0.75) (layer F.Fab) (width 0.05))
     (fp_line (start -1.45 0.75) (end 1.45 0.75) (layer F.Fab) (width 0.05))
-    (pad 1 smd rect (at -0.75 0 270) (size 0.8 0.75) (layers F.Cu F.Paste F.Mask)
+    (pad 1 smd rect (at -0.75 0 90) (size 0.8 0.75) (layers F.Cu F.Paste F.Mask)
       (net 38 "Net-(C42-Pad1)"))
-    (pad 2 smd rect (at 0.75 0 270) (size 0.8 0.75) (layers F.Cu F.Paste F.Mask)
+    (pad 2 smd rect (at 0.75 0 90) (size 0.8 0.75) (layers F.Cu F.Paste F.Mask)
       (net 2 GND))
   )
@@
   (segment (start 231.1186 80.236) (end 230.0224 80.236) (width 0.254) (layer F.Cu) (net 1))
   (via (at 230.0224 80.236) (size 0.6858) (drill 0.3302) (layers F.Cu B.Cu) (net 1))
+  (segment (start 238.76 76.3538) (end 240.0286 76.3538) (width 0.254) (layer F.Cu) (net 2))
+  (segment (start 240.0286 76.3538) (end 240.0554 76.327) (width 0.254) (layer F.Cu) (net 2))
+  (via (at 240.0554 76.327) (size 0.6858) (drill 0.3302) (layers F.Cu B.Cu) (net 2))
+  (segment (start 238.7346 71.6774) (end 239.3936 71.6774) (width 0.254) (layer F.Cu) (net 2))
+  (segment (start 239.3936 71.6774) (end 240.0554 72.3392) (width 0.254) (layer F.Cu) (net 2))
+  (via (at 240.0554 72.3392) (size 0.6858) (drill 0.3302) (layers F.Cu B.Cu) (net 2))
   (segment (start 211.7344 66.291667) (end 211.7344 65.9638) (width 0.254) (layer B.Cu) (net 2))
   (segment (start 211.7852 66.8274) (end 211.7852 66.342467) (width 0.254) (layer B.Cu) (net 2))
@@
   (segment (start 226.3708 70.9108) (end 226.3648 70.9168) (width 0.3302) (layer F.Cu) (net 2))
   (via (at 226.3648 70.9168) (size 0.6858) (drill 0.3302) (layers F.Cu B.Cu) (net 2))
-  (segment (start 238.7814 74.3712) (end 238.7814 73.2054) (width 0.3302) (layer F.Cu) (net 2))
-  (segment (start 238.7814 75.5916) (end 238.7814 74.3712) (width 0.3302) (layer F.Cu) (net 2))
-  (via (at 238.7814 74.3712) (size 0.6858) (drill 0.3302) (layers F.Cu B.Cu) (net 2))
   (segment (start 211.7852 76.0476) (end 213.7544 76.0476) (width 0.3302) (layer B.Cu) (net 2))
   (segment (start 213.7544 76.0476) (end 213.856 75.946) (width 0.3302) (layer B.Cu) (net 2))
@@
   (segment (start 222.758098 75.235558) (end 220.839498 75.235558) (width 0.254) (layer F.Cu) (net 36))
   (segment (start 220.839498 75.235558) (end 220.485898 75.589158) (width 0.254) (layer F.Cu) (net 36))
-  (segment (start 238.7814 77.0916) (end 235.6032 77.0916) (width 0.3302) (layer F.Cu) (net 37))
-  (segment (start 235.6032 77.0916) (end 234.8698 76.3582) (width 0.3302) (layer F.Cu) (net 37))
+  (segment (start 233.263 74.8538) (end 234.8738 74.8538) (width 0.254) (layer F.Cu) (net 37))
+  (segment (start 234.8738 74.8538) (end 237.4392 74.8538) (width 0.254) (layer F.Cu) (net 37))
+  (segment (start 234.8698 76.3582) (end 234.8698 75.22683) (width 0.254) (layer F.Cu) (net 37))
+  (segment (start 234.8698 75.22683) (end 234.8738 75.22283) (width 0.254) (layer F.Cu) (net 37))
+  (segment (start 234.8738 75.22283) (end 234.8738 74.8538) (width 0.254) (layer F.Cu) (net 37))
+  (segment (start 237.4392 74.8538) (end 237.7186 74.8538) (width 0.254) (layer F.Cu) (net 37))
+  (segment (start 238.76 74.8538) (end 238.131 74.8538) (width 0.254) (layer F.Cu) (net 37))
+  (segment (start 238.131 74.8538) (end 237.4392 74.8538) (width 0.254) (layer F.Cu) (net 37))
+  (segment (start 229.87 71.4608) (end 233.263 74.8538) (width 0.254) (layer F.Cu) (net 37))
   (segment (start 229.87 70.9108) (end 229.87 71.4608) (width 0.3302) (layer F.Cu) (net 37))
-  (segment (start 229.87 71.4608) (end 234.7674 76.3582) (width 0.3302) (layer F.Cu) (net 37))
   (segment (start 234.7674 76.3582) (end 234.8698 76.3582) (width 0.3302) (layer F.Cu) (net 37))
-  (segment (start 238.7814 71.7054) (end 235.097 71.7054) (width 0.3302) (layer F.Cu) (net 38))
+  (segment (start 238.0742 73.1774) (end 238.46389 73.1774) (width 0.254) (layer F.Cu) (net 38))
+  (segment (start 236.1692 73.1774) (end 238.0742 73.1774) (width 0.254) (layer F.Cu) (net 38))
+  (segment (start 238.0742 73.1774) (end 238.7346 73.1774) (width 0.254) (layer F.Cu) (net 38))
+  (segment (start 236.1692 73.1774) (end 236.3724 73.1774) (width 0.254) (layer F.Cu) (net 38))
+  (segment (start 234.7722 73.1774) (end 236.1692 73.1774) (width 0.254) (layer F.Cu) (net 38))
+  (segment (start 233.9856 73.1774) (end 234.7722 73.1774) (width 0.254) (layer F.Cu) (net 38))
+  (segment (start 234.7722 73.1774) (end 234.8698 73.0798) (width 0.254) (layer F.Cu) (net 38))
+  (segment (start 234.8698 73.0798) (end 234.8698 71.4782) (width 0.254) (layer F.Cu) (net 38))
+  (segment (start 231.14 70.9108) (end 231.719 70.9108) (width 0.254) (layer F.Cu) (net 38))
+  (segment (start 231.719 70.9108) (end 233.9856 73.1774) (width 0.254) (layer F.Cu) (net 38))
   (segment (start 235.097 71.7054) (end 234.8698 71.4782) (width 0.3302) (layer F.Cu) (net 38))
-  (segment (start 231.14 70.9108) (end 234.3024 70.9108) (width 0.3302) (layer F.Cu) (net 38))
-  (segment (start 234.3024 70.9108) (end 234.8698 71.4782) (width 0.3302) (layer F.Cu) (net 38))
   (segment (start 193.5748 46.8884) (end 193.5748 48.03) (width 0.508) (layer F.Cu) (net 39))
   (segment (start 193.5748 48.03) (end 191.6684 49.9364) (width 0.508) (layer F.Cu) (net 39))
@@
   (segment (start 226.047242 68.922958) (end 226.06 68.9102) (width 0.254) (layer F.Cu) (net 60))
   (via (at 226.06 68.9102) (size 0.6858) (drill 0.3302) (layers F.Cu B.Cu) (net 60))
+  (segment (start 235.1532 69.507102) (end 235.369102 69.507102) (width 0.254) (layer F.Cu) (net 61))
+  (segment (start 239.5982 70.739) (end 243.738401 74.879201) (width 0.254) (layer F.Cu) (net 61))
+  (segment (start 233.797854 69.507102) (end 235.1532 69.507102) (width 0.254) (layer F.Cu) (net 61))
+  (segment (start 235.1532 69.507102) (end 238.366302 69.507102) (width 0.254) (layer F.Cu) (net 61))
+  (segment (start 239.4458 70.5866) (end 239.5982 70.739) (width 0.254) (layer F.Cu) (net 61))
+  (segment (start 238.366302 69.507102) (end 239.5982 70.739) (width 0.254) (layer F.Cu) (net 61))
   (segment (start 227.294586 68.6816) (end 232.972352 68.6816) (width 0.254) (layer F.Cu) (net 61))
   (segment (start 232.972352 68.6816) (end 233.797854 69.507102) (width 0.254) (layer F.Cu) (net 61))
   (segment (start 243.738401 74.879201) (end 244.5004 75.6412) (width 0.254) (layer F.Cu) (net 61))
-  (segment (start 239.4458 70.5866) (end 243.738401 74.879201) (width 0.254) (layer F.Cu) (net 61))
-  (segment (start 236.4486 70.5866) (end 239.4458 70.5866) (width 0.254) (layer F.Cu) (net 61))
-  (segment (start 233.797854 69.507102) (end 235.369102 69.507102) (width 0.254) (layer F.Cu) (net 61))
-  (segment (start 235.369102 69.507102) (end 236.4486 70.5866) (width 0.254) (layer F.Cu) (net 61))
   (segment (start 226.553228 69.422958) (end 227.294586 68.6816) (width 0.254) (layer F.Cu) (net 61))
   (segment (start 218.783498 69.422958) (end 226.553228 69.422958) (width 0.254) (layer F.Cu) (net 61))
