File: hardware/mcphail-main-board/mcphail-main-board.kicad_pcb (KiCad board)
At the start: 2 copper layers, 80.6 x 56.6 mm, 143 parts, among them J1 INSECT DETECTION, J2 EMITTERS, J3 BREAKOUT, J4 MICRO SD, J5 MICRO USB, J6 PROG/BOOT, J7 FONA 808, J8 INPUT 6V-9V, J9 JST PH, U1 MCP6004, U10 BUCK-BOOST 5V TPS63060, U11 MCP1703, U2 MCP6004, U3 TLV274, U4 MCP6001, U5 ADS1118, U6 ATSAMD21G18A, U7 24AA1025 EEPROM, U8 MCP7940N RTC, U9 MCP73871, X1 16MHz, X2 32.768kHz

Commit message: Commit.
Connections:
- U6 pad 41: (no net) -> /~PG
Routing:
- net /~PG: track 14.9 -> 29.6 mm, vias 0 -> 2
- net GND: track 126.7 -> 127.3 mm
- net +3V3: track 156.1 -> 156.4 mm, vias 9 -> 11
Changed lines of the file:
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@@
 (kicad_pcb (version 4) (host pcbnew 4.0.5-e0-6337~49~ubuntu16.04.1)
   (general
-    (links 335)
+    (links 336)
     (no_connects 0)
-    (area 104.572999 40.039358 248.365056 123.265001)
+    (area 167.563799 41.722878 248.365056 98.505056)
     (thickness 1.6)
     (drawings 28)
-    (tracks 1475)
+    (tracks 1497)
     (zones 0)
     (modules 143)
@@
     (pad 40 smd rect (at 1.25 -4.35 90) (size 1.3 0.25) (layers F.Cu F.Paste F.Mask)
       (net 45 /Microcontroller/~RESET))
-    (pad 41 smd rect (at 0.75 -4.35 90) (size 1.3 0.25) (layers F.Cu F.Paste F.Mask))
+    (pad 41 smd rect (at 0.75 -4.35 90) (size 1.3 0.25) (layers F.Cu F.Paste F.Mask)
+      (net 44 /~PG))
     (pad 42 smd rect (at 0.25 -4.35 90) (size 1.3 0.25) (layers F.Cu F.Paste F.Mask)
       (net 2 GND))
@@
   (segment (start 231.1186 80.236) (end 230.0224 80.236) (width 0.254) (layer F.Cu) (net 1))
   (via (at 230.0224 80.236) (size 0.6858) (drill 0.3302) (layers F.Cu B.Cu) (net 1))
+  (segment (start 216.217501 61.763955) (end 216.217501 60.236099) (width 0.254) (layer F.Cu) (net 2))
+  (segment (start 214.668098 62.322454) (end 214.925654 62.064898) (width 0.254) (layer F.Cu) (net 2))
+  (segment (start 216.217501 60.236099) (end 216.5604 59.8932) (width 0.254) (layer F.Cu) (net 2))
+  (segment (start 214.925654 62.064898) (end 215.916558 62.064898) (width 0.254) (layer F.Cu) (net 2))
+  (segment (start 214.668098 62.903558) (end 214.668098 62.322454) (width 0.254) (layer F.Cu) (net 2))
+  (segment (start 214.683498 62.918958) (end 214.668098 62.903558) (width 0.254) (layer F.Cu) (net 2))
+  (segment (start 214.683498 63.822958) (end 214.683498 62.918958) (width 0.254) (layer F.Cu) (net 2))
+  (segment (start 215.916558 62.064898) (end 216.217501 61.763955) (width 0.254) (layer F.Cu) (net 2))
   (segment (start 238.76 76.3538) (end 240.0286 76.3538) (width 0.254) (layer F.Cu) (net 2))
   (segment (start 240.0286 76.3538) (end 240.0554 76.327) (width 0.254) (layer F.Cu) (net 2))
@@
   (segment (start 222.183642 65.903158) (end 222.1992 65.8876) (width 0.254) (layer F.Cu) (net 2))
   (via (at 222.1992 65.8876) (size 0.6858) (drill 0.3302) (layers F.Cu B.Cu) (net 2))
-  (segment (start 214.683498 63.297958) (end 216.5604 61.421056) (width 0.254) (layer F.Cu) (net 2))
-  (segment (start 214.683498 63.822958) (end 214.683498 63.297958) (width 0.254) (layer F.Cu) (net 2))
-  (segment (start 216.5604 61.421056) (end 216.5604 60.378133) (width 0.254) (layer F.Cu) (net 2))
-  (segment (start 216.5604 60.378133) (end 216.5604 59.8932) (width 0.254) (layer F.Cu) (net 2))
   (segment (start 215.138 59.3852) (end 216.0524 59.3852) (width 0.254) (layer F.Cu) (net 2))
   (segment (start 216.0524 59.3852) (end 216.5604 59.8932) (width 0.254) (layer F.Cu) (net 2))
@@
   (segment (start 173.311629 83.423461) (end 173.311629 83.145461) (width 0.254) (layer F.Cu) (net 29))
   (segment (start 173.311629 83.145461) (end 174.811629 81.645461) (width 0.254) (layer F.Cu) (net 29))
+  (segment (start 213.9696 57.912) (end 213.7664 57.912) (width 0.254) (layer F.Cu) (net 30))
+  (segment (start 213.7664 57.912) (end 213.0044 57.912) (width 0.254) (layer F.Cu) (net 30))
+  (segment (start 219.964 56.3626) (end 218.4146 57.912) (width 0.254) (layer F.Cu) (net 30))
+  (segment (start 218.4146 57.912) (end 213.7664 57.912) (width 0.254) (layer F.Cu) (net 30))
+  (segment (start 222.371 56.388) (end 219.9894 56.388) (width 0.254) (layer B.Cu) (net 30))
+  (segment (start 219.9894 56.388) (end 219.964 56.3626) (width 0.254) (layer B.Cu) (net 30))
+  (via (at 219.964 56.3626) (size 0.6858) (drill 0.3302) (layers F.Cu B.Cu) (net 30))
+  (via (at 222.371 56.388) (size 0.6858) (drill 0.3302) (layers F.Cu B.Cu) (net 30))
   (segment (start 213.6648 70.4342) (end 213.6648 68.4784) (width 0.254) (layer B.Cu) (net 30))
   (segment (start 213.683498 72.522958) (end 213.683498 70.452898) (width 0.254) (layer F.Cu) (net 30))
@@
   (segment (start 204.0636 65.0748) (end 204.216 64.9224) (width 0.254) (layer F.Cu) (net 30))
   (via (at 204.216 64.9224) (size 0.6858) (drill 0.3302) (layers F.Cu B.Cu) (net 30))
-  (segment (start 215.4936 56.388) (end 213.9696 57.912) (width 0.254) (layer F.Cu) (net 30))
-  (segment (start 213.9696 57.912) (end 213.0044 57.912) (width 0.254) (layer F.Cu) (net 30))
-  (segment (start 222.371 56.388) (end 215.4936 56.388) (width 0.254) (layer F.Cu) (net 30))
   (segment (start 222.758 57.404) (end 222.758 56.775) (width 0.254) (layer F.Cu) (net 30))
   (segment (start 222.758 56.775) (end 222.371 56.388) (width 0.254) (layer F.Cu) (net 30))
@@
   (segment (start 230.43888 50.45694) (end 230.41208 50.43014) (width 0.3302) (layer F.Cu) (net 43))
   (segment (start 230.32508 50.51714) (end 230.41208 50.43014) (width 0.3302) (layer F.Cu) (net 43))
+  (segment (start 222.74128 51.99734) (end 224.2312 53.48726) (width 0.3302) (layer F.Cu) (net 44))
+  (segment (start 224.2312 53.48726) (end 225.30314 54.5592) (width 0.3302) (layer F.Cu) (net 44))
+  (segment (start 220.1672 58.5216) (end 220.1672 57.445478) (width 0.254) (layer F.Cu) (net 44))
+  (segment (start 220.1672 57.445478) (end 224.125418 53.48726) (width 0.254) (layer F.Cu) (net 44))
+  (segment (start 224.125418 53.48726) (end 224.2312 53.48726) (width 0.254) (layer F.Cu) (net 44))
+  (segment (start 217.6272 61.0616) (end 220.1672 58.5216) (width 0.254) (layer F.Cu) (net 44))
+  (segment (start 217.0176 61.0616) (end 217.6272 61.0616) (width 0.254) (layer F.Cu) (net 44))
+  (via (at 217.0176 61.0616) (size 0.6858) (drill 0.3302) (layers F.Cu B.Cu) (net 44))
+  (segment (start 216.4842 61.2394) (end 216.8398 61.2394) (width 0.254) (layer B.Cu) (net 44))
+  (segment (start 216.8398 61.2394) (end 217.0176 61.0616) (width 0.254) (layer B.Cu) (net 44))
+  (segment (start 215.1634 62.5602) (end 216.4842 61.2394) (width 0.254) (layer B.Cu) (net 44))
+  (via (at 215.1634 62.5602) (size 0.6858) (drill 0.3302) (layers F.Cu B.Cu) (net 44))
+  (segment (start 215.183498 63.822958) (end 215.183498 62.580298) (width 0.254) (layer F.Cu) (net 44))
+  (segment (start 215.183498 62.580298) (end 215.1634 62.5602) (width 0.254) (layer F.Cu) (net 44))
   (segment (start 225.30314 54.5592) (end 230.82012 54.5592) (width 0.3302) (layer F.Cu) (net 44))
   (segment (start 230.82012 54.5592) (end 231.79818 53.58114) (width 0.3302) (layer F.Cu) (net 44))
   (segment (start 231.79818 53.58114) (end 231.82318 53.58114) (width 0.3302) (layer F.Cu) (net 44))
   (segment (start 222.74128 51.51714) (end 222.74128 51.99734) (width 0.3302) (layer F.Cu) (net 44))
-  (segment (start 222.74128 51.99734) (end 225.30314 54.5592) (width 0.3302) (layer F.Cu) (net 44))
   (segment (start 231.82318 53.58114) (end 231.82318 53.34124) (width 0.3302) (layer F.Cu) (net 44))
   (segment (start 231.82318 53.34124) (end 230.41208 51.93014) (width 0.3302) (layer F.Cu) (net 44))

Commit message: Release v1.0 McPhail Main Board
Parts:
- moved BAT1 144.4 mm to (81.7, 87.8)
- moved C1 144.4 mm to (92.5, 84.9)
- moved C10 144.4 mm to (34.3, 63.5)
- moved C11 144.4 mm to (43.4, 92.6)
- moved C12 144.4 mm to (40.9, 66.5)
- moved C13 144.4 mm to (47.2, 94.4)
- moved C14 144.4 mm to (43.5, 89.2)
- moved C15 144.4 mm to (44.4, 64.6)
- moved C16 144.4 mm to (48.2, 90.9)
- moved C17 144.4 mm to (48.2, 86.0)
- moved C2 144.4 mm to (64.9, 88.1)
- moved C20 144.4 mm to (40.9, 82.0)
- moved C21 144.4 mm to (46.9, 79.1)
- moved C22 144.4 mm to (44.1, 72.7)
- moved C23 144.4 mm to (32.5, 83.8)
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Routing:
- net GND: track 127.3 -> 171.4 mm, vias 45 -> 57
- net AGND: track 52.7 -> 67.3 mm, vias 26 -> 32
- net /Microcontroller/D7_CS: track 30.8 -> 21.0 mm
- net /Microcontroller/MISO: track 34.3 -> 25.8 mm
- net +3V3: track 156.4 -> 150.2 mm, vias 11 -> 10
- net /Microcontroller/SCLK: track 40.6 -> 45.8 mm
- net /Microcontroller/MOSI: track 28.4 -> 30.1 mm
- net (no net): track 1.71 -> 0.00 mm
- net /Microcontroller/SDA: track 28.5 -> 29.2 mm
Other:
- board text added: "3.3V"
- board text added: "5V"
- board text added: "5V VA A2 A1 A0 AG"
- board text added: "AGND"
- board text added: "FABRICATION NOTES 1. THIS IS A 2 LAYER BOARD. 2. EXTERNAL LAYERS SHALL HAVE 1 OZ COPPER. 3. MATERIAL: FR4 AND 0.062 INCH +/- 10% THICK. 4. BOARDS SHALL BE ROHS COMPLIANT. 5. MANUFACTURE IN ACCORDANCE WITH IPC-6012 CLASS 2 6. MASK: BOTH SIDES OF THE BOARD SHALL HAVE SOLDER MASK (ANY COLOR) OVER BARE COPPER. 7. SILK: BOTH SIDES OF THE BOARD SHALL HAVE WHITE SILKSCREEN. DO NOT PLACE SILK OVER BARE C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"
- board text added: "McPhail Trap Main Board v1.0 Kyle Birchard and Jenner Hanni jenner@wickerbox.net"
- board text added: "PIN1"
- board text added: "SIGIN"
- board text added: "SIGOUT"
- board text removed: "9V MAX"
- board text removed: "SIG"

Commit message: Release v1.0 McPhail Main Board
Other:
- board text added: "McPhail Trap Main Board v1.0 Kyle Birchard and Jenner Hanni"
- board text added: "jenner@wickerbox.net"
- board text removed: "McPhail Trap Main Board v1.0 Kyle Birchard and Jenner Hanni jenner@wickerbox.net"
Changed lines of the file:
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@@
     (links 336)
     (no_connects 0)
-    (area 167.563799 41.722878 248.365056 98.505056)
+    (area 23.190199 39.6748 253.588759 108.7628)
     (thickness 1.6)
-    (drawings 19)
+    (drawings 20)
     (tracks 1543)
     (zones 0)
@@
       (net 30 +3V3))
   )
-  (gr_text "McPhail Trap Main Board v1.0\nKyle Birchard and Jenner Hanni\njenner@wickerbox.net" (at 100.7618 47.752) (layer B.SilkS)
+  (gr_text jenner@wickerbox.net (at 36.2204 96.139 360) (layer B.SilkS)
+    (effects (font (size 1.27 1.27) (thickness 0.2032)) (justify mirror))
+  )
+  (gr_text "McPhail Trap Main Board v1.0\nKyle Birchard and Jenner Hanni" (at 100.8634 46.7868) (layer B.SilkS)
     (effects (font (thickness 0.254)) (justify left mirror))
   )
@@
     (effects (font (size 1.016 1.016) (thickness 0.1524)))
   )
-  (gr_text 5V (at 96.393 52.959 360) (layer F.SilkS)
+  (gr_text 5V (at 96.393 52.959) (layer F.SilkS)
     (effects (font (size 1.016 1.016) (thickness 0.1524)))
   )

Commit message: Fixed clearance issues on McPhail Main v1.1
Routing:
- net /Microcontroller/FONA_PS: track 38.5 -> 52.2 mm, vias 3 -> 5
- net AGND: track 67.3 -> 75.7 mm
- net /Microcontroller/SCL: track 27.6 -> 32.1 mm
- net GND: track 171.4 -> 167.8 mm, vias 57 -> 53
- net /Microcontroller/FONA_RTS: track 29.5 -> 26.9 mm, vias 2 -> 0
- net +3V3: track 150.2 -> 152.2 mm
- net VIN: track 35.6 -> 37.3 mm
- net /Photodiode Signal Input Conditioning/VREF: track 68.0 -> 69.5 mm
- net /Microcontroller/MOSI: track 30.1 -> 31.5 mm
- net /Microcontroller/MFP: track 27.6 -> 26.3 mm
- net /Microcontroller/~RESET: track 25.4 -> 26.8 mm
- net /Microcontroller/SDA: track 29.2 -> 28.2 mm, vias 6 -> 5
- net /Microcontroller/FONA_TX: track 26.0 -> 26.9 mm
- net /Microcontroller/D7_CS: track 21.0 -> 21.8 mm
- net /Microcontroller/D-: track 53.9 -> 54.6 mm
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Other:
- net class Default: clearance 0.0254 -> 0.1524; trace_width 0.254 -> 0.1524
- rule trace_clearance: 0.0254 -> 0.1524
- board text added: "McPhail Trap Main Board v1.1 Kyle Birchard and Jenner Hanni"
- board text removed: "McPhail Trap Main Board v1.0 Kyle Birchard and Jenner Hanni"
