File: hardware/mcphail-main-board/signal-conditioning.sch (KiCad schematic (older format))
At the start: 66 parts, among them J1 INSECT DETECTION, J2 EMITTERS, J3 BREAKOUT, U1 MCP6004, U2 MCP6004, U3 TLV274, U4 MCP6001

Commit message: Sch passes rule check. Final netlist. Starting layout.
Changed lines of the file:
@@
 $EndComp
 $Comp
-L +5V #PWR24
+L +5V #PWR013
 U 1 1 596FCAB2
 P 6350 3400
-F 0 "#PWR24" H 6350 3250 50  0001 C CNN
+F 0 "#PWR013" H 6350 3250 50  0001 C CNN
 F 1 "+5V" H 6350 3540 50  0000 C CNN
 F 2 "" H 6350 3400 50  0000 C CNN
@@
 $EndComp
 $Comp
-L +5V #PWR21
+L +5V #PWR014
 U 1 1 596FCB56
 P 3550 4225
-F 0 "#PWR21" H 3550 4075 50  0001 C CNN
+F 0 "#PWR014" H 3550 4075 50  0001 C CNN
 F 1 "+5V" H 3550 4365 50  0000 C CNN
 F 2 "" H 3550 4225 50  0000 C CNN
@@
 $EndComp
 $Comp
-L +5V #PWR34
+L +5V #PWR015
 U 1 1 59701081
 P 12225 3550
-F 0 "#PWR34" H 12225 3400 50  0001 C CNN
+F 0 "#PWR015" H 12225 3400 50  0001 C CNN
 F 1 "+5V" H 12225 3690 50  0000 C CNN
 F 2 "" H 12225 3550 50  0000 C CNN
@@
 $EndComp
 $Comp
-L GND #PWR32
+L GND #PWR016
 U 1 1 597121F8
 P 10425 7375
-F 0 "#PWR32" H 10425 7125 50  0001 C CNN
+F 0 "#PWR016" H 10425 7125 50  0001 C CNN
 F 1 "GND" H 10425 7225 50  0000 C CNN
 F 2 "" H 10425 7375 50  0000 C CNN
@@
 $EndComp
 $Comp
-L GND #PWR33
+L GND #PWR017
 U 1 1 59712329
 P 10825 7375
-F 0 "#PWR33" H 10825 7125 50  0001 C CNN
+F 0 "#PWR017" H 10825 7125 50  0001 C CNN
 F 1 "GND" H 10825 7225 50  0000 C CNN
 F 2 "" H 10825 7375 50  0000 C CNN
@@
 $EndComp
 $Comp
-L +3.3V #PWR27
+L +3.3V #PWR018
 U 1 1 59713790
 P 9325 7350
-F 0 "#PWR27" H 9325 7200 50  0001 C CNN
+F 0 "#PWR018" H 9325 7200 50  0001 C CNN
 F 1 "+3.3V" H 9325 7490 50  0000 C CNN
 F 2 "" H 9325 7350 50  0000 C CNN
@@
 $EndComp
 $Comp
-L +3.3V #PWR29
+L +3.3V #PWR019
 U 1 1 59716A30
 P 9550 5950
-F 0 "#PWR29" H 9550 5800 50  0001 C CNN
+F 0 "#PWR019" H 9550 5800 50  0001 C CNN
 F 1 "+3.3V" H 9550 6090 50  0000 C CNN
 F 2 "" H 9550 5950 50  0000 C CNN
@@
 3.3V
 $Comp
-L +3.3V #PWR36
+L +3.3V #PWR020
 U 1 1 5971ADA4
 P 12425 8225
-F 0 "#PWR36" H 12425 8075 50  0001 C CNN
+F 0 "#PWR020" H 12425 8075 50  0001 C CNN
 F 1 "+3.3V" H 12425 8365 50  0000 C CNN
 F 2 "" H 12425 8225 50  0000 C CNN
@@
 $EndComp
 $Comp
-L +5V #PWR17
+L +5V #PWR021
 U 1 1 5974FCB7
 P 2525 2700
-F 0 "#PWR17" H 2525 2550 50  0001 C CNN
+F 0 "#PWR021" H 2525 2550 50  0001 C CNN
 F 1 "+5V" H 2525 2840 50  0000 C CNN
 F 2 "" H 2525 2700 50  0000 C CNN
@@
 $EndComp
 $Comp
-L +5V #PWR13
+L +5V #PWR022
 U 1 1 59752D6D
 P 1600 850
-F 0 "#PWR13" H 1600 700 50  0001 C CNN
+F 0 "#PWR022" H 1600 700 50  0001 C CNN
 F 1 "+5V" H 1600 990 50  0000 C CNN
 F 2 "" H 1600 850 50  0000 C CNN
@@
 $EndComp
 $Comp
-L GND #PWR16
+L GND #PWR023
 U 1 1 59753228
 P 2125 1250
-F 0 "#PWR16" H 2125 1000 50  0001 C CNN
+F 0 "#PWR023" H 2125 1000 50  0001 C CNN
 F 1 "GND" H 2125 1100 50  0000 C CNN
 F 2 "" H 2125 1250 50  0000 C CNN
@@
 $EndComp
 $Comp
-L GND #PWR14
+L GND #PWR024
 U 1 1 597544D0
 P 1600 1500
-F 0 "#PWR14" H 1600 1250 50  0001 C CNN
+F 0 "#PWR024" H 1600 1250 50  0001 C CNN
 F 1 "GND" H 1600 1350 50  0000 C CNN
 F 2 "" H 1600 1500 50  0000 C CNN
@@
 $EndComp
 $Comp
-L +5V #PWR39
+L +5V #PWR025
 U 1 1 5981F754
 P 12650 8225
-F 0 "#PWR39" H 12650 8075 50  0001 C CNN
+F 0 "#PWR025" H 12650 8075 50  0001 C CNN
 F 1 "+5V" H 12650 8365 50  0000 C CNN
 F 2 "" H 12650 8225 50  0000 C CNN
@@
 Connection ~ 13025 8425
 Wire Wire Line
-	13025 8425 13025 7650
+	13025 7650 13025 8425
 Connection ~ 12925 8325
 Wire Wire Line
@@
 	2825 3300 4350 3300
 $Comp
-L +3.3V #PWR30
+L +3.3V #PWR026
 U 1 1 5983489F
 P 10225 7075
-F 0 "#PWR30" H 10225 6925 50  0001 C CNN
+F 0 "#PWR026" H 10225 6925 50  0001 C CNN
 F 1 "+3.3V" H 10225 7215 50  0000 C CNN
 F 2 "" H 10225 7075 50  0000 C CNN
@@
 SHEET 2: SIGNAL CONDITIONING
 $Comp
-L AGND #PWR28
+L AGND #PWR027
 U 1 1 598790E7
 P 9325 8425
-F 0 "#PWR28" H 9325 8175 50  0001 C CNN
+F 0 "#PWR027" H 9325 8175 50  0001 C CNN
 F 1 "AGND" H 9325 8275 50  0000 C CNN
 F 2 "" H 9325 8425 50  0000 C CNN
@@
 $EndComp
 $Comp
-L AGND #PWR37
+L AGND #PWR028
 U 1 1 598791DA
 P 12425 8775
-F 0 "#PWR37" H 12425 8525 50  0001 C CNN
+F 0 "#PWR028" H 12425 8525 50  0001 C CNN
 F 1 "AGND" H 12425 8625 50  0000 C CNN
 F 2 "" H 12425 8775 50  0000 C CNN
@@
 AGND
 $Comp
-L AGND #PWR22
+L AGND #PWR029
 U 1 1 598796DA
 P 4225 8475
-F 0 "#PWR22" H 4225 8225 50  0001 C CNN
+F 0 "#PWR029" H 4225 8225 50  0001 C CNN
 F 1 "AGND" H 4225 8325 50  0000 C CNN
 F 2 "" H 4225 8475 50  0000 C CNN
@@
 $EndComp
 $Comp
-L AGND #PWR25
+L AGND #PWR030
 U 1 1 59879F07
 P 6350 4225
-F 0 "#PWR25" H 6350 3975 50  0001 C CNN
+F 0 "#PWR030" H 6350 3975 50  0001 C CNN
 F 1 "AGND" H 6350 4075 50  0000 C CNN
 F 2 "" H 6350 4225 50  0000 C CNN
@@
 $EndComp
 $Comp
-L AGND #PWR20
+L AGND #PWR031
 U 1 1 5987A045
 P 3350 4900
-F 0 "#PWR20" H 3350 4650 50  0001 C CNN
+F 0 "#PWR031" H 3350 4650 50  0001 C CNN
 F 1 "AGND" H 3350 4750 50  0000 C CNN
 F 2 "" H 3350 4900 50  0000 C CNN
@@
 $EndComp
 $Comp
-L AGND #PWR23
+L AGND #PWR032
 U 1 1 5987A135
 P 5175 5000
-F 0 "#PWR23" H 5175 4750 50  0001 C CNN
+F 0 "#PWR032" H 5175 4750 50  0001 C CNN
 F 1 "AGND" H 5175 4850 50  0000 C CNN
 F 2 "" H 5175 5000 50  0000 C CNN
@@
 $EndComp
 $Comp
-L AGND #PWR18
+L AGND #PWR033
 U 1 1 5987A303
 P 2525 3600
-F 0 "#PWR18" H 2525 3350 50  0001 C CNN
+F 0 "#PWR033" H 2525 3350 50  0001 C CNN
 F 1 "AGND" H 2525 3450 50  0000 C CNN
 F 2 "" H 2525 3600 50  0000 C CNN
@@
 $EndComp
 $Comp
-L AGND #PWR35
+L AGND #PWR034
 U 1 1 5987F0DC
 P 12225 4175
-F 0 "#PWR35" H 12225 3925 50  0001 C CNN
+F 0 "#PWR034" H 12225 3925 50  0001 C CNN
 F 1 "AGND" H 12225 4025 50  0000 C CNN
 F 2 "" H 12225 4175 50  0000 C CNN
@@
 $EndComp
 $Comp
-L AGND #PWR38
+L AGND #PWR035
 U 1 1 5987F1D1
 P 12550 3650
-F 0 "#PWR38" H 12550 3400 50  0001 C CNN
+F 0 "#PWR035" H 12550 3400 50  0001 C CNN
 F 1 "AGND" H 12550 3500 50  0000 C CNN
 F 2 "" H 12550 3650 50  0000 C CNN
@@
 $EndComp
 $Comp
-L AGND #PWR26
+L AGND #PWR036
 U 1 1 598809E6
 P 6675 3625
-F 0 "#PWR26" H 6675 3375 50  0001 C CNN
+F 0 "#PWR036" H 6675 3375 50  0001 C CNN
 F 1 "AGND" H 6675 3475 50  0000 C CNN
 F 2 "" H 6675 3625 50  0000 C CNN
@@
 $EndComp
 $Comp
-L AGND #PWR31
+L AGND #PWR037
 U 1 1 5988572B
 P 10225 8125
-F 0 "#PWR31" H 10225 7875 50  0001 C CNN
+F 0 "#PWR037" H 10225 7875 50  0001 C CNN
 F 1 "AGND" H 10225 7975 50  0000 C CNN
 F 2 "" H 10225 8125 50  0000 C CNN
@@
 VREF
 $Comp
-L AGND #PWR19
+L AGND #PWR038
 U 1 1 598046F9
 P 2825 2950
-F 0 "#PWR19" H 2825 2700 50  0001 C CNN
+F 0 "#PWR038" H 2825 2700 50  0001 C CNN
 F 1 "AGND" H 2825 2800 50  0000 C CNN
 F 2 "" H 2825 2950 50  0000 C CNN
@@
 $EndComp
 $Comp
-L AGND #PWR15
+L AGND #PWR039
 U 1 1 598047EC
 P 1700 3450
-F 0 "#PWR15" H 1700 3200 50  0001 C CNN
+F 0 "#PWR039" H 1700 3200 50  0001 C CNN
 F 1 "AGND" H 1700 3300 50  0000 C CNN
 F 2 "" H 1700 3450 50  0000 C CNN

Commit message: Lots more layout work, needs rework.
Connections:
- net A1: now also U3.13 (-); no longer U3.9 (-)
- net A2: now also U3.14; no longer U3.8
- net AGND: now also C25.2, C26.2
- net GND: no longer C25.2, C26.2
- net LINE_IN: now also U2.7; no longer U2.14
- net VREF: now also U2.12 (+), U2.5 (+); no longer U2.12 (+), U2.5 (+)
- net at C8.2, R5.1: now also U2.13 (-); no longer U2.6 (-)
- net at C8.1, R6.1, R8.2: now also U2.14; no longer U2.7
- net at C18.2, R13.2, R15.2: now also U2.6 (-); no longer U2.13 (-)
- net at U3.3 (+), U3.6 (-), U3.7: now also U3.12 (+); no longer U3.10 (+)
Changed lines of the file:
@@
 $Comp
 L IC-OPAMP-QUAD-MCP6004-SOIC14 U?
-U 2 1 596FEB1E
+U 4 1 596FEB1E
 P 4650 7450
 AR Path="/596FEB1E" Ref="U?"  Part="2"
-AR Path="/596F9466/596FEB1E" Ref="U2"  Part="2"
+AR Path="/596F9466/596FEB1E" Ref="U2"  Part="4"
 F 0 "U2" H 4700 7600 50  0000 L CNN
 F 1 "MCP6004" H 4700 7300 50  0000 L CNN
@@
 F 7 "Digikey" H 4650 7100 50  0001 C CIN "S1_Name"
 F 8 "MCP6004T-I/SLCT-ND" H 4650 7100 50  0001 C CIN "S1_PN"
-	2    4650 7450
+	4    4650 7450
 	1    0    0    -1
 $EndComp
@@
 $Comp
 L IC-OPAMP-QUAD-MCP6004-SOIC14 U?
-U 4 1 596FEC6B
+U 2 1 596FEC6B
 P 7925 7925
 AR Path="/596FEC6B" Ref="U?"  Part="4"
-AR Path="/596F9466/596FEC6B" Ref="U2"  Part="4"
+AR Path="/596F9466/596FEC6B" Ref="U2"  Part="2"
 F 0 "U2" H 7975 8075 50  0000 L CNN
 F 1 "MCP6004" H 7975 7775 50  0000 L CNN
@@
 F 7 "Digikey" H 7925 7575 50  0001 C CIN "S1_Name"
 F 8 "MCP6004T-I/SLCT-ND" H 7925 7575 50  0001 C CIN "S1_PN"
-	4    7925 7925
+	2    7925 7925
 	1    0    0    -1
 $EndComp
@@
 $EndComp
 $Comp
-L GND #PWR016
-U 1 1 597121F8
-P 10425 7375
-F 0 "#PWR016" H 10425 7125 50  0001 C CNN
-F 1 "GND" H 10425 7225 50  0000 C CNN
-F 2 "" H 10425 7375 50  0000 C CNN
-F 3 "" H 10425 7375 50  0000 C CNN
-	1    10425 7375
-	1    0    0    -1
-$EndComp
-$Comp
-L GND #PWR017
-U 1 1 59712329
-P 10825 7375
-F 0 "#PWR017" H 10825 7125 50  0001 C CNN
-F 1 "GND" H 10825 7225 50  0000 C CNN
-F 2 "" H 10825 7375 50  0000 C CNN
-F 3 "" H 10825 7375 50  0000 C CNN
-	1    10825 7375
-	1    0    0    -1
-$EndComp
-$Comp
 L CAP-CER-2.2UF-25V-X7R-0805 C22
 U 1 1 59713111
@@
 $EndComp
 $Comp
-L +3.3V #PWR018
+L +3.3V #PWR016
 U 1 1 59713790
 P 9325 7350
-F 0 "#PWR018" H 9325 7200 50  0001 C CNN
+F 0 "#PWR016" H 9325 7200 50  0001 C CNN
 F 1 "+3.3V" H 9325 7490 50  0000 C CNN
 F 2 "" H 9325 7350 50  0000 C CNN
@@
 $EndComp
 $Comp
-L +3.3V #PWR019
+L +3.3V #PWR017
 U 1 1 59716A30
 P 9550 5950
-F 0 "#PWR019" H 9550 5800 50  0001 C CNN
+F 0 "#PWR017" H 9550 5800 50  0001 C CNN
 F 1 "+3.3V" H 9550 6090 50  0000 C CNN
 F 2 "" H 9550 5950 50  0000 C CNN
@@
 3.3V
 $Comp
-L +3.3V #PWR020
+L +3.3V #PWR018
 U 1 1 5971ADA4
 P 12425 8225
-F 0 "#PWR020" H 12425 8075 50  0001 C CNN
+F 0 "#PWR018" H 12425 8075 50  0001 C CNN
 F 1 "+3.3V" H 12425 8365 50  0000 C CNN
 F 2 "" H 12425 8225 50  0000 C CNN
@@
 $Comp
 L IC-OPAMP-QUAD-TLV274-SOIC14 U3
-U 3 1 59722405
+U 4 1 59722405
 P 11625 7875
 F 0 "U3" H 11675 8025 50  0000 L CNN
@@
 F 7 "Digikey" H 11625 7525 50  0001 C CIN "S1_Name"
 F 8 "296-39258-1-ND" H 11625 7525 50  0001 C CIN "S1_PN"
-	3    11625 7875
+	4    11625 7875
 	1    0    0    -1
 $EndComp
@@
 $EndComp
 $Comp
-L +5V #PWR021
+L +5V #PWR019
 U 1 1 5974FCB7
 P 2525 2700
-F 0 "#PWR021" H 2525 2550 50  0001 C CNN
+F 0 "#PWR019" H 2525 2550 50  0001 C CNN
 F 1 "+5V" H 2525 2840 50  0000 C CNN
 F 2 "" H 2525 2700 50  0000 C CNN
@@
 $EndComp
 $Comp
-L +5V #PWR022
+L +5V #PWR020
 U 1 1 59752D6D
 P 1600 850
-F 0 "#PWR022" H 1600 700 50  0001 C CNN
+F 0 "#PWR020" H 1600 700 50  0001 C CNN
 F 1 "+5V" H 1600 990 50  0000 C CNN
 F 2 "" H 1600 850 50  0000 C CNN
@@
 $EndComp
 $Comp
-L GND #PWR023
+L GND #PWR021
 U 1 1 59753228
 P 2125 1250
-F 0 "#PWR023" H 2125 1000 50  0001 C CNN
+F 0 "#PWR021" H 2125 1000 50  0001 C CNN
 F 1 "GND" H 2125 1100 50  0000 C CNN
 F 2 "" H 2125 1250 50  0000 C CNN
@@
 $EndComp
 $Comp
-L GND #PWR024
+L GND #PWR022
 U 1 1 597544D0
 P 1600 1500
-F 0 "#PWR024" H 1600 1250 50  0001 C CNN
+F 0 "#PWR022" H 1600 1250 50  0001 C CNN
 F 1 "GND" H 1600 1350 50  0000 C CNN
 F 2 "" H 1600 1500 50  0000 C CNN
@@
 $EndComp
 $Comp
-L +5V #PWR025
+L +5V #PWR023
 U 1 1 5981F754
 P 12650 8225
-F 0 "#PWR025" H 12650 8075 50  0001 C CNN
+F 0 "#PWR023" H 12650 8075 50  0001 C CNN
 F 1 "+5V" H 12650 8365 50  0000 C CNN
 F 2 "" H 12650 8225 50  0000 C CNN
@@
 	2825 3300 4350 3300
 $Comp
-L +3.3V #PWR026
+L +3.3V #PWR024
 U 1 1 5983489F
 P 10225 7075
-F 0 "#PWR026" H 10225 6925 50  0001 C CNN
+F 0 "#PWR024" H 10225 6925 50  0001 C CNN
 F 1 "+3.3V" H 10225 7215 50  0000 C CNN
 F 2 "" H 10225 7075 50  0000 C CNN
@@
 SHEET 2: SIGNAL CONDITIONING
 $Comp
-L AGND #PWR027
+L AGND #PWR025
 U 1 1 598790E7
 P 9325 8425
-F 0 "#PWR027" H 9325 8175 50  0001 C CNN
+F 0 "#PWR025" H 9325 8175 50  0001 C CNN
 F 1 "AGND" H 9325 8275 50  0000 C CNN
 F 2 "" H 9325 8425 50  0000 C CNN
@@
 $EndComp
 $Comp
-L AGND #PWR028
+L AGND #PWR026
 U 1 1 598791DA
 P 12425 8775
-F 0 "#PWR028" H 12425 8525 50  0001 C CNN
+F 0 "#PWR026" H 12425 8525 50  0001 C CNN
 F 1 "AGND" H 12425 8625 50  0000 C CNN
 F 2 "" H 12425 8775 50  0000 C CNN
@@
 AGND
 $Comp
-L AGND #PWR029
+L AGND #PWR027
 U 1 1 598796DA
 P 4225 8475
-F 0 "#PWR029" H 4225 8225 50  0001 C CNN
+F 0 "#PWR027" H 4225 8225 50  0001 C CNN
 F 1 "AGND" H 4225 8325 50  0000 C CNN
 F 2 "" H 4225 8475 50  0000 C CNN
@@
 $EndComp
 $Comp
-L AGND #PWR030
+L AGND #PWR028
 U 1 1 59879F07
 P 6350 4225
-F 0 "#PWR030" H 6350 3975 50  0001 C CNN
+F 0 "#PWR028" H 6350 3975 50  0001 C CNN
 F 1 "AGND" H 6350 4075 50  0000 C CNN
 F 2 "" H 6350 4225 50  0000 C CNN
@@
 $EndComp
 $Comp
-L AGND #PWR031
+L AGND #PWR029
 U 1 1 5987A045
 P 3350 4900
-F 0 "#PWR031" H 3350 4650 50  0001 C CNN
+F 0 "#PWR029" H 3350 4650 50  0001 C CNN
 F 1 "AGND" H 3350 4750 50  0000 C CNN
 F 2 "" H 3350 4900 50  0000 C CNN
@@
 $EndComp
 $Comp
-L AGND #PWR032
+L AGND #PWR030
 U 1 1 5987A135
 P 5175 5000
-F 0 "#PWR032" H 5175 4750 50  0001 C CNN
+F 0 "#PWR030" H 5175 4750 50  0001 C CNN
 F 1 "AGND" H 5175 4850 50  0000 C CNN
 F 2 "" H 5175 5000 50  0000 C CNN
@@
 $EndComp
 $Comp
-L AGND #PWR033
+L AGND #PWR031
 U 1 1 5987A303
 P 2525 3600
-F 0 "#PWR033" H 2525 3350 50  0001 C CNN
+F 0 "#PWR031" H 2525 3350 50  0001 C CNN
 F 1 "AGND" H 2525 3450 50  0000 C CNN
 F 2 "" H 2525 3600 50  0000 C CNN
@@
 $EndComp
 $Comp
-L AGND #PWR034
+L AGND #PWR032
 U 1 1 5987F0DC
 P 12225 4175
-F 0 "#PWR034" H 12225 3925 50  0001 C CNN
+F 0 "#PWR032" H 12225 3925 50  0001 C CNN
 F 1 "AGND" H 12225 4025 50  0000 C CNN
 F 2 "" H 12225 4175 50  0000 C CNN
@@
 $EndComp
 $Comp
-L AGND #PWR035
+L AGND #PWR033
 U 1 1 5987F1D1
 P 12550 3650
-F 0 "#PWR035" H 12550 3400 50  0001 C CNN
+F 0 "#PWR033" H 12550 3400 50  0001 C CNN
 F 1 "AGND" H 12550 3500 50  0000 C CNN
 F 2 "" H 12550 3650 50  0000 C CNN
@@
 $EndComp
 $Comp
-L AGND #PWR036
+L AGND #PWR034
 U 1 1 598809E6
 P 6675 3625
-F 0 "#PWR036" H 6675 3375 50  0001 C CNN
+F 0 "#PWR034" H 6675 3375 50  0001 C CNN
 F 1 "AGND" H 6675 3475 50  0000 C CNN
 F 2 "" H 6675 3625 50  0000 C CNN
@@
 $EndComp
 $Comp
-L AGND #PWR037
+L AGND #PWR035
 U 1 1 5988572B
 P 10225 8125
-F 0 "#PWR037" H 10225 7875 50  0001 C CNN
+F 0 "#PWR035" H 10225 7875 50  0001 C CNN
 F 1 "AGND" H 10225 7975 50  0000 C CNN
 F 2 "" H 10225 8125 50  0000 C CNN
@@
 VREF
 $Comp
-L AGND #PWR038
+L AGND #PWR036
 U 1 1 598046F9
 P 2825 2950
-F 0 "#PWR038" H 2825 2700 50  0001 C CNN
+F 0 "#PWR036" H 2825 2700 50  0001 C CNN
 F 1 "AGND" H 2825 2800 50  0000 C CNN
 F 2 "" H 2825 2950 50  0000 C CNN
@@
 $EndComp
 $Comp
-L AGND #PWR039
+L AGND #PWR037
 U 1 1 598047EC
 P 1700 3450
-F 0 "#PWR039" H 1700 3200 50  0001 C CNN
+F 0 "#PWR037" H 1700 3200 50  0001 C CNN
 F 1 "AGND" H 1700 3300 50  0000 C CNN
 F 2 "" H 1700 3450 50  0000 C CNN
@@
 	1    0    0    -1
 $EndComp
+$Comp
+L AGND #PWR038
+U 1 1 5984484C
+P 10425 7375
+F 0 "#PWR038" H 10425 7125 50  0001 C CNN
+F 1 "AGND" H 10425 7225 50  0000 C CNN
+F 2 "" H 10425 7375 50  0000 C CNN
+F 3 "" H 10425 7375 50  0000 C CNN
+	1    10425 7375
+	1    0    0    -1
+$EndComp
+$Comp
+L AGND #PWR039
+U 1 1 5984493C
+P 10825 7375
+F 0 "#PWR039" H 10825 7125 50  0001 C CNN
+F 1 "AGND" H 10825 7225 50  0000 C CNN
+F 2 "" H 10825 7375 50  0000 C CNN
+F 3 "" H 10825 7375 50  0000 C CNN
+	1    10825 7375
+	1    0    0    -1
+$EndComp
