File: hardware/mcphail-main-board/input-power.sch (KiCad schematic (older format))
At the start: 0 parts

Commit message: Release main board sch with BOM and layout estimates.
Parts:
- added B1: LIPO, Wickerlib:UNDEFINED, symbol BATT-LIPO-3.7V-500MAH-JST-2PIN
- added C43, C44, C45, C46: 4.7uF, Wickerlib:RLC-1206-SMD, symbol CAP-CER-4.7UF-50V-X7R-1206
- added C47: 100nF, Wickerlib:RLC-0603-SMD, symbol CAP-CER-0.1UF-100V-X7R-0603
- added C48: 10pF, Wickerlib:RLC-0603-SMD, symbol CAP-CER-10PF-50V-NP0-0603
- added C49, C50: 1uF, Wickerlib:RLC-0805-SMD, symbol CAP-CER-1UF-25V-X7R-0805
- added D4: 20V 1A, Wickerlib:DIODE-SMA, symbol DIODE-SCHOTTKY-20V-1A-SS12-SMA
- added J8: INPUT 6V-9V, Wickerlib:CONN-BARREL-JACK-2.5x5.5MM-TH, symbol CONN-PWR-JACK-2.5X5.5MM-HIGH-CUR
- added J9: JST PH, Wickerlib:CONN-JST-S2B-PH-SM4-TB, symbol HEADER-FEMALE-2POS-TH-1x02-JST-PH
- added L2: 1uH 11A, Wickerlib:UNDEFINED, symbol FIXED-IND-1UH-11A-XFL4020-102-SMD
- added LED1, LED2, LED3: AMBER, Wickerlib:LED-0603-SMD, symbol LED-AMBER-0603-SMT-L296-Q2R2
- added R38: 0 ohm, Wickerlib:RLC-0603-SMD, symbol RES-0.0-JUMPER-1/8W-0603
- added R39, R40, R41: 470, Wickerlib:RLC-0603-SMD, symbol RES-470-5%-1/4W-0603
- added R42: NTC 10K, Wickerlib:RLC-0402-SMD, symbol THERM-NTC-10K-1%-0402
- added R43: 2K, Wickerlib:RLC-0603-SMD, symbol RES-2K-1%-1/8W-0603
- added R44: 100K, Wickerlib:RLC-0603-SMD, symbol RES-100K-1%-1/10W-0603
- added R45, R47: 1M, Wickerlib:RLC-0603-SMD, symbol RES-1M-5%-1/10W-0603
- added R46: 111K, Wickerlib:RLC-0603-SMD, symbol RES-111K-5%-1/10W-0603
- added U10: BUCK-BOOST 5V TPS63060, Wickerlib:QFN-20-1EP-4x4MM_P0.5MM, symbol IC-REG-BUCK-BOOST-ADJ-2A-TPS63060-10WSON
- added U11: MCP1703, Wickerlib:SOT-23-3, symbol IC-REG-LDO-3.3V-0.25A-MCP1703-SOT23A-3
- added U9: MCP73871, Wickerlib:QFN-20-1EP-4x4MM_P0.5MM, symbol IC-LI-ION-CONTROLLER-MCP73871-QFN20
- added W1: TEST_1P, Wickerlib:HOLE-PLATED-40MIL, symbol TEST_1P
Connections:
- net labels added: +3.3V, +5V, 3.3V, 5V, GND, PROG1, PROG3, STAT1, STAT2, THERM, VBAT, VCC, VIN, VUSB, ~PG
- wire segments 0 -> 99
- no-connect marks 0 -> 2
Other:
- note added: "3.7V"
- note added: "IF VIN EXISTS,\nVCC = VIN (5V-9V)\n\nIF VIN REMOVED,\nVCC = VBAT (3.0V-4.2V)\n\nSEL set to USB\n500mA charge limit\n\n~TE~ low, enables \nsafety timer"
- note added: "TODO: REPLACE WITH LESS AMP VERSION"
- note added: "VPCC\nDISABLED"

Commit message: Added ADS1118 (ADC with temp sensor) to Atmega32u4.
Other:
- note added: "SHEET 4: POWER INPUT"
Changed lines of the file:
@@
 	1    0    0    1
 $EndComp
-Text Notes 4150 2125 0    50   ~ 0
+Text Notes 4150 2275 0    50   ~ 0
 IF VIN EXISTS,\nVCC = VIN (5V-9V)\n\nIF VIN REMOVED,\nVCC = VBAT (3.0V-4.2V)\n\nSEL set to USB\n500mA charge limit\n\n~TE~ low, enables \nsafety timer
 $Comp
@@
 	0    1    1    0
 $EndComp
+Text Notes 1300 1100 0    200  ~ 0
+SHEET 4: POWER INPUT
 $EndSCHEMATC

Commit message: Hooked up pins to ATSAMD21G18 Cortex M0, fixed AGND throughout.
Other:
- note added: "TODO: REPLACE WITH SMALLER LESS AMP VERSION"
- note removed: "TODO: REPLACE WITH LESS AMP VERSION"
Changed lines of the file:
@@
 $EndComp
 $Comp
-L VBAT #PWR078
+L VBAT #PWR083
 U 1 1 59717743
 P 6125 2675
-F 0 "#PWR078" H 6125 2525 50  0001 C CNN
+F 0 "#PWR083" H 6125 2525 50  0001 C CNN
 F 1 "VBAT" H 6125 2815 50  0000 C CNN
 F 2 "" H 6125 2675 50  0000 C CNN
@@
 $EndComp
 $Comp
-L GND #PWR079
+L GND #PWR084
 U 1 1 597178CA
 P 5875 3025
-F 0 "#PWR079" H 5875 2775 50  0001 C CNN
+F 0 "#PWR084" H 5875 2775 50  0001 C CNN
 F 1 "GND" H 5875 2875 50  0000 C CNN
 F 2 "" H 5875 3025 50  0000 C CNN
@@
 $EndComp
 $Comp
-L GND #PWR080
+L GND #PWR085
 U 1 1 597178E6
 P 5550 2425
-F 0 "#PWR080" H 5550 2175 50  0001 C CNN
+F 0 "#PWR085" H 5550 2175 50  0001 C CNN
 F 1 "GND" H 5550 2275 50  0000 C CNN
 F 2 "" H 5550 2425 50  0000 C CNN
@@
 $EndComp
 $Comp
-L GND #PWR081
+L GND #PWR086
 U 1 1 59717A07
 P 1600 3275
-F 0 "#PWR081" H 1600 3025 50  0001 C CNN
+F 0 "#PWR086" H 1600 3025 50  0001 C CNN
 F 1 "GND" H 1600 3125 50  0000 C CNN
 F 2 "" H 1600 3275 50  0000 C CNN
@@
 $EndComp
 $Comp
-L GND #PWR082
+L GND #PWR087
 U 1 1 597180EA
 P 6300 3025
-F 0 "#PWR082" H 6300 2775 50  0001 C CNN
+F 0 "#PWR087" H 6300 2775 50  0001 C CNN
 F 1 "GND" H 6300 2875 50  0000 C CNN
 F 2 "" H 6300 3025 50  0000 C CNN
@@
 NoConn ~ 6775 3200
 $Comp
-L GND #PWR083
+L GND #PWR088
 U 1 1 59718618
 P 5325 4075
-F 0 "#PWR083" H 5325 3825 50  0001 C CNN
+F 0 "#PWR088" H 5325 3825 50  0001 C CNN
 F 1 "GND" H 5325 3925 50  0000 C CNN
 F 2 "" H 5325 4075 50  0000 C CNN
@@
 $EndComp
 $Comp
-L GND #PWR084
+L GND #PWR089
 U 1 1 5972098A
 P 5675 4075
-F 0 "#PWR084" H 5675 3825 50  0001 C CNN
+F 0 "#PWR089" H 5675 3825 50  0001 C CNN
 F 1 "GND" H 5675 3925 50  0000 C CNN
 F 2 "" H 5675 4075 50  0000 C CNN
@@
 $EndComp
 $Comp
-L GND #PWR085
+L GND #PWR090
 U 1 1 597209C2
 P 6175 4075
-F 0 "#PWR085" H 6175 3825 50  0001 C CNN
+F 0 "#PWR090" H 6175 3825 50  0001 C CNN
 F 1 "GND" H 6175 3925 50  0000 C CNN
 F 2 "" H 6175 4075 50  0000 C CNN
@@
 $EndComp
 $Comp
-L GND #PWR086
+L GND #PWR091
 U 1 1 59720A0A
 P 6500 4075
-F 0 "#PWR086" H 6500 3825 50  0001 C CNN
+F 0 "#PWR091" H 6500 3825 50  0001 C CNN
 F 1 "GND" H 6500 3925 50  0000 C CNN
 F 2 "" H 6500 4075 50  0000 C CNN
@@
 $EndComp
 $Comp
-L VIN #PWR087
+L VIN #PWR092
 U 1 1 5975D9CC
 P 4225 2575
-F 0 "#PWR087" H 4225 2425 50  0001 C CNN
+F 0 "#PWR092" H 4225 2425 50  0001 C CNN
 F 1 "VIN" H 4225 2715 50  0000 C CNN
 F 2 "" H 4225 2575 50  0000 C CNN
@@
 $EndComp
 $Comp
-L GND #PWR088
+L GND #PWR093
 U 1 1 5975DBAA
 P 2000 2100
-F 0 "#PWR088" H 2000 1850 50  0001 C CNN
+F 0 "#PWR093" H 2000 1850 50  0001 C CNN
 F 1 "GND" H 2000 1950 50  0000 C CNN
 F 2 "" H 2000 2100 50  0000 C CNN
@@
 $EndComp
 $Comp
-L +3.3V #PWR089
+L +3.3V #PWR094
 U 1 1 59766B20
 P 10675 1925
-F 0 "#PWR089" H 10675 1775 50  0001 C CNN
+F 0 "#PWR094" H 10675 1775 50  0001 C CNN
 F 1 "+3.3V" H 10675 2065 50  0000 C CNN
 F 2 "" H 10675 1925 50  0000 C CNN
@@
 $EndComp
 $Comp
-L +5V #PWR090
+L +5V #PWR095
 U 1 1 59766B5E
 P 8925 1900
-F 0 "#PWR090" H 8925 1750 50  0001 C CNN
+F 0 "#PWR095" H 8925 1750 50  0001 C CNN
 F 1 "+5V" H 8925 2040 50  0000 C CNN
 F 2 "" H 8925 1900 50  0000 C CNN
@@
 $EndComp
 $Comp
-L GND #PWR091
+L GND #PWR096
 U 1 1 59766C20
 P 10150 2625
-F 0 "#PWR091" H 10150 2375 50  0001 C CNN
+F 0 "#PWR096" H 10150 2375 50  0001 C CNN
 F 1 "GND" H 10150 2475 50  0000 C CNN
 F 2 "" H 10150 2625 50  0000 C CNN
@@
 $EndComp
 $Comp
-L GND #PWR092
+L GND #PWR097
 U 1 1 5977A60F
 P 6825 2425
-F 0 "#PWR092" H 6825 2175 50  0001 C CNN
+F 0 "#PWR097" H 6825 2175 50  0001 C CNN
 F 1 "GND" H 6825 2275 50  0000 C CNN
 F 2 "" H 6825 2425 50  0000 C CNN
@@
 $EndComp
 $Comp
-L GND #PWR093
+L GND #PWR098
 U 1 1 5978D873
 P 9750 2575
-F 0 "#PWR093" H 9750 2325 50  0001 C CNN
+F 0 "#PWR098" H 9750 2325 50  0001 C CNN
 F 1 "GND" H 9750 2425 50  0000 C CNN
 F 2 "" H 9750 2575 50  0000 C CNN
@@
 $EndComp
 $Comp
-L GND #PWR094
+L GND #PWR099
 U 1 1 5978D9AF
 P 10675 2575
-F 0 "#PWR094" H 10675 2325 50  0001 C CNN
+F 0 "#PWR099" H 10675 2325 50  0001 C CNN
 F 1 "GND" H 10675 2425 50  0000 C CNN
 F 2 "" H 10675 2575 50  0000 C CNN
@@
 $EndComp
 $Comp
-L GND #PWR095
+L GND #PWR0100
 U 1 1 59790C75
 P 7500 3325
-F 0 "#PWR095" H 7500 3075 50  0001 C CNN
+F 0 "#PWR0100" H 7500 3075 50  0001 C CNN
 F 1 "GND" H 7500 3175 50  0000 C CNN
 F 2 "" H 7500 3325 50  0000 C CNN
@@
 $EndComp
 $Comp
-L GND #PWR096
+L GND #PWR0101
 U 1 1 597910A0
 P 7275 2775
-F 0 "#PWR096" H 7275 2525 50  0001 C CNN
+F 0 "#PWR0101" H 7275 2525 50  0001 C CNN
 F 1 "GND" H 7275 2625 50  0000 C CNN
 F 2 "" H 7275 2775 50  0000 C CNN
@@
 3.7V
 Text Notes 7400 1450 0    50   ~ 0
-TODO: REPLACE WITH LESS AMP VERSION
+TODO: REPLACE WITH SMALLER LESS AMP VERSION
 $Comp
 L RES-1M-5%-1/10W-0603 R45
@@
 STAT2
 $Comp
-L GND #PWR097
+L GND #PWR0102
 U 1 1 59854B48
 P 4100 4050
-F 0 "#PWR097" H 4100 3800 50  0001 C CNN
+F 0 "#PWR0102" H 4100 3800 50  0001 C CNN
 F 1 "GND" H 4100 3900 50  0000 C CNN
 F 2 "" H 4100 4050 50  0000 C CNN

Commit message: All footprints good. Changed op amps slightly for footprints.
Parts:
- removed C46: 4.7uF, Wickerlib:RLC-1206-SMD, symbol CAP-CER-4.7UF-50V-X7R-1206
- removed L2: 1uH 11A, Wickerlib:UNDEFINED, symbol FIXED-IND-1UH-11A-XFL4020-102-SMD
- added C46, C53: 10uF, Wickerlib:RLC-0805-SMD, symbol CAP-CER-10UF-16V-X7R-0805
- added C54, C55, C56: 22uF, Wickerlib:RLC-1210-SMD, symbol CAP-CER-22UF-25V-X7R-1210
- added L2: 1uH 3.3A, Wickerlib:1226AS-H-1R0N, symbol FIXED-IND-1UH-3.3A-1226AS-H-1R0N-SMD
- B1: footprint Wickerlib:UNDEFINED -> (none)
- U10: footprint Wickerlib:QFN-20-1EP-4x4MM_P0.5MM -> Wickerlib:WSON-10-1EP
Connections:
- wire segments 99 -> 109
Other:
- note removed: "TODO: REPLACE WITH SMALLER LESS AMP VERSION"
- moved on the sheet: B1, C43, C44, C45, C47, C48, C49, C50, D4, J8, J9, LED1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

Commit message: Lots more layout work, needs rework.
Connections:
- net ~PG: no longer R41.2, U9.6 (~PG)
- new net ~PG1: R41.2, U9.6 (~PG)
Changed lines of the file:
@@
 $EndComp
 $Comp
-L VBAT #PWR083
+L VBAT #PWR080
 U 1 1 59717743
 P 5550 2675
-F 0 "#PWR083" H 5550 2525 50  0001 C CNN
+F 0 "#PWR080" H 5550 2525 50  0001 C CNN
 F 1 "VBAT" H 5550 2815 50  0000 C CNN
 F 2 "" H 5550 2675 50  0000 C CNN
@@
 $EndComp
 $Comp
-L GND #PWR084
+L GND #PWR081
 U 1 1 597178CA
 P 5300 3025
-F 0 "#PWR084" H 5300 2775 50  0001 C CNN
+F 0 "#PWR081" H 5300 2775 50  0001 C CNN
 F 1 "GND" H 5300 2875 50  0000 C CNN
 F 2 "" H 5300 3025 50  0000 C CNN
@@
 $EndComp
 $Comp
-L GND #PWR085
+L GND #PWR082
 U 1 1 597178E6
 P 4975 2425
-F 0 "#PWR085" H 4975 2175 50  0001 C CNN
+F 0 "#PWR082" H 4975 2175 50  0001 C CNN
 F 1 "GND" H 4975 2275 50  0000 C CNN
 F 2 "" H 4975 2425 50  0000 C CNN
@@
 $EndComp
 $Comp
-L GND #PWR086
+L GND #PWR083
 U 1 1 59717A07
 P 1025 3275
-F 0 "#PWR086" H 1025 3025 50  0001 C CNN
+F 0 "#PWR083" H 1025 3025 50  0001 C CNN
 F 1 "GND" H 1025 3125 50  0000 C CNN
 F 2 "" H 1025 3275 50  0000 C CNN
@@
 $EndComp
 $Comp
-L GND #PWR087
+L GND #PWR084
 U 1 1 597180EA
 P 5725 3025
-F 0 "#PWR087" H 5725 2775 50  0001 C CNN
+F 0 "#PWR084" H 5725 2775 50  0001 C CNN
 F 1 "GND" H 5725 2875 50  0000 C CNN
 F 2 "" H 5725 3025 50  0000 C CNN
@@
 NoConn ~ 6200 3200
 $Comp
-L GND #PWR088
+L GND #PWR085
 U 1 1 59718618
 P 4750 4075
-F 0 "#PWR088" H 4750 3825 50  0001 C CNN
+F 0 "#PWR085" H 4750 3825 50  0001 C CNN
 F 1 "GND" H 4750 3925 50  0000 C CNN
 F 2 "" H 4750 4075 50  0000 C CNN
@@
 $EndComp
 Text Label 3425 3350 0    50   ~ 0
-~PG
+~PG1
 Text Label 3425 3450 0    50   ~ 0
 STAT2
@@
 $EndComp
 $Comp
-L GND #PWR089
+L GND #PWR086
 U 1 1 5972098A
 P 5100 4075
-F 0 "#PWR089" H 5100 3825 50  0001 C CNN
+F 0 "#PWR086" H 5100 3825 50  0001 C CNN
 F 1 "GND" H 5100 3925 50  0000 C CNN
 F 2 "" H 5100 4075 50  0000 C CNN
@@
 $EndComp
 $Comp
-L GND #PWR090
+L GND #PWR087
 U 1 1 597209C2
 P 5600 4075
-F 0 "#PWR090" H 5600 3825 50  0001 C CNN
+F 0 "#PWR087" H 5600 3825 50  0001 C CNN
 F 1 "GND" H 5600 3925 50  0000 C CNN
 F 2 "" H 5600 4075 50  0000 C CNN
@@
 $EndComp
 $Comp
-L GND #PWR091
+L GND #PWR088
 U 1 1 59720A0A
 P 5925 4075
-F 0 "#PWR091" H 5925 3825 50  0001 C CNN
+F 0 "#PWR088" H 5925 3825 50  0001 C CNN
 F 1 "GND" H 5925 3925 50  0000 C CNN
 F 2 "" H 5925 4075 50  0000 C CNN
@@
 $EndComp
 $Comp
-L VIN #PWR092
+L VIN #PWR089
 U 1 1 5975D9CC
 P 3650 2575
-F 0 "#PWR092" H 3650 2425 50  0001 C CNN
+F 0 "#PWR089" H 3650 2425 50  0001 C CNN
 F 1 "VIN" H 3650 2715 50  0000 C CNN
 F 2 "" H 3650 2575 50  0000 C CNN
@@
 $EndComp
 $Comp
-L GND #PWR093
+L GND #PWR090
 U 1 1 5975DBAA
 P 1425 2100
-F 0 "#PWR093" H 1425 1850 50  0001 C CNN
+F 0 "#PWR090" H 1425 1850 50  0001 C CNN
 F 1 "GND" H 1425 1950 50  0000 C CNN
 F 2 "" H 1425 2100 50  0000 C CNN
@@
 $EndComp
 $Comp
-L +3.3V #PWR094
+L +3.3V #PWR091
 U 1 1 59766B20
 P 10650 3475
-F 0 "#PWR094" H 10650 3325 50  0001 C CNN
+F 0 "#PWR091" H 10650 3325 50  0001 C CNN
 F 1 "+3.3V" H 10650 3615 50  0000 C CNN
 F 2 "" H 10650 3475 50  0000 C CNN
@@
 $EndComp
 $Comp
-L +5V #PWR095
+L +5V #PWR092
 U 1 1 59766B5E
 P 8350 1900
-F 0 "#PWR095" H 8350 1750 50  0001 C CNN
+F 0 "#PWR092" H 8350 1750 50  0001 C CNN
 F 1 "+5V" H 8350 2040 50  0000 C CNN
 F 2 "" H 8350 1900 50  0000 C CNN
@@
 $EndComp
 $Comp
-L GND #PWR096
+L GND #PWR093
 U 1 1 59766C20
 P 10125 4175
-F 0 "#PWR096" H 10125 3925 50  0001 C CNN
+F 0 "#PWR093" H 10125 3925 50  0001 C CNN
 F 1 "GND" H 10125 4025 50  0000 C CNN
 F 2 "" H 10125 4175 50  0000 C CNN
@@
 $EndComp
 $Comp
-L GND #PWR097
+L GND #PWR094
 U 1 1 5977A60F
 P 6325 2425
-F 0 "#PWR097" H 6325 2175 50  0001 C CNN
+F 0 "#PWR094" H 6325 2175 50  0001 C CNN
 F 1 "GND" H 6325 2275 50  0000 C CNN
 F 2 "" H 6325 2425 50  0000 C CNN
@@
 $EndComp
 $Comp
-L GND #PWR098
+L GND #PWR095
 U 1 1 5978D873
 P 9625 4125
-F 0 "#PWR098" H 9625 3875 50  0001 C CNN
+F 0 "#PWR095" H 9625 3875 50  0001 C CNN
 F 1 "GND" H 9625 3975 50  0000 C CNN
 F 2 "" H 9625 4125 50  0000 C CNN
@@
 $EndComp
 $Comp
-L GND #PWR099
+L GND #PWR096
 U 1 1 5978D9AF
 P 10650 4125
-F 0 "#PWR099" H 10650 3875 50  0001 C CNN
+F 0 "#PWR096" H 10650 3875 50  0001 C CNN
 F 1 "GND" H 10650 3975 50  0000 C CNN
 F 2 "" H 10650 4125 50  0000 C CNN
@@
 $EndComp
 $Comp
-L GND #PWR0100
+L GND #PWR097
 U 1 1 59790C75
 P 6925 3325
-F 0 "#PWR0100" H 6925 3075 50  0001 C CNN
+F 0 "#PWR097" H 6925 3075 50  0001 C CNN
 F 1 "GND" H 6925 3175 50  0000 C CNN
 F 2 "" H 6925 3325 50  0000 C CNN
@@
 $EndComp
 $Comp
-L GND #PWR0101
+L GND #PWR098
 U 1 1 597910A0
 P 6700 2775
-F 0 "#PWR0101" H 6700 2525 50  0001 C CNN
+F 0 "#PWR098" H 6700 2525 50  0001 C CNN
 F 1 "GND" H 6700 2625 50  0000 C CNN
 F 2 "" H 6700 2775 50  0000 C CNN
@@
 STAT1
 Text Label 2775 3550 0    50   ~ 0
-~PG
+~PG1
 Text Label 2775 3650 0    50   ~ 0
 STAT2
 $Comp
-L GND #PWR0102
+L GND #PWR099
 U 1 1 59854B48
 P 3525 4050
-F 0 "#PWR0102" H 3525 3800 50  0001 C CNN
+F 0 "#PWR099" H 3525 3800 50  0001 C CNN
 F 1 "GND" H 3525 3900 50  0000 C CNN
 F 2 "" H 3525 4050 50  0000 C CNN
@@
 Wire Wire Line
 	5925 3600 4675 3600
-$Comp
-L TEST_1P W1
-U 1 1 5988AA50
-P 5675 3400
-F 0 "W1" V 5675 3625 50  0000 C CNN
-F 1 "TEST_1P" H 5675 3600 50  0001 C CNN
-F 2 "Wickerlib:HOLE-PLATED-40MIL" H 5875 3400 50  0001 C CNN
-F 3 "" H 5875 3400 50  0000 C CNN
-	1    5675 3400
-	0    1    1    0
-$EndComp
 Text Notes 725  1100 0    200  ~ 0
 SHEET 4: POWER INPUT
@@
 	9325 2700 9325 2750
 $Comp
-L GND #PWR0103
+L GND #PWR0100
 U 1 1 597FAAB5
 P 9325 2750
-F 0 "#PWR0103" H 9325 2500 50  0001 C CNN
+F 0 "#PWR0100" H 9325 2500 50  0001 C CNN
 F 1 "GND" H 9325 2600 50  0000 C CNN
 F 2 "" H 9325 2750 50  0000 C CNN
@@
 Connection ~ 9325 2250
 $Comp
-L GND #PWR0104
+L GND #PWR0101
 U 1 1 597FABDB
 P 9700 2750
-F 0 "#PWR0104" H 9700 2500 50  0001 C CNN
+F 0 "#PWR0101" H 9700 2500 50  0001 C CNN
 F 1 "GND" H 9700 2600 50  0000 C CNN
 F 2 "" H 9700 2750 50  0000 C CNN
@@
 $EndComp
 $Comp
-L GND #PWR0105
+L GND #PWR0102
 U 1 1 597FAC49
 P 10075 2750
-F 0 "#PWR0105" H 10075 2500 50  0001 C CNN
+F 0 "#PWR0102" H 10075 2500 50  0001 C CNN
 F 1 "GND" H 10075 2600 50  0000 C CNN
 F 2 "" H 10075 2750 50  0000 C CNN
@@
 Connection ~ 5850 2150
 $Comp
-L GND #PWR0106
+L GND #PWR0103
 U 1 1 597FBFAD
 P 5850 2425
-F 0 "#PWR0106" H 5850 2175 50  0001 C CNN
+F 0 "#PWR0103" H 5850 2175 50  0001 C CNN
 F 1 "GND" H 5850 2275 50  0000 C CNN
 F 2 "" H 5850 2425 50  0000 C CNN
@@
 	0    -1   -1   0
 $EndComp
+$Comp
+L TEST_1P W1
+U 1 1 5988AA50
+P 5675 3400
+F 0 "W1" V 5675 3625 50  0000 C CNN
+F 1 "TEST_1P" H 5675 3600 50  0001 C CNN
+F 2 "Wickerlib:HOLE-PLATED-40MIL" H 5875 3400 50  0001 C CNN
+F 3 "" H 5875 3400 50  0000 C CNN
+	1    5675 3400
+	0    1    1    0
+$EndComp
 $EndSCHEMATC

Commit message: Commit.
Parts:
- C43, C44, C45: MF_Name Taiyo Yuden -> Samsung; MF_PN UMK316AB7475KL-T -> CL31B475KBHNNNE; S1_PN 587-2994-1-ND -> 1276-2789-1-ND
Changed lines of the file:
@@
 EESchema Schematic File Version 2
 LIBS:wickerlib
-LIBS:mcphail-main-board-cache
 EELAYER 25 0
 EELAYER END
@@
 P 4975 2325
 F 0 "C44" H 5075 2375 50  0000 L CNN
-F 1 "4.7uF" H 5075 2275 50  0000 L CNN
-F 2 "Wickerlib:RLC-1206-SMD" H 5600 1925 50  0001 C CIN
-F 3 "http://ds.yuden.co.jp/TYCOMPAS/ut/detail.do?productNo=UMK316AB7475KL-T&fileName=UMK316AB7475KL-T_SS&mode=specSheetDownload" H 5325 2100 50  0001 C CNN
-F 4 "CAP CER 4.7UF 50V X7R 1206" H 5650 2000 50  0001 C CIN "Description"
-F 5 "Taiyo Yuden" H 5175 1825 50  0001 C CIN "MF_Name"
-F 6 "UMK316AB7475KL-T" H 5850 1825 50  0001 C CIN "MF_PN"
-F 7 "Digikey" H 5075 1725 50  0001 C CIN "S1_Name"
-F 8 "587-2994-1-ND" H 5775 1725 50  0001 C CIN "S1_PN"
+F 1 "4.7uF" V 9875 3100 50  0000 C CNN
+F 2 "Wickerlib:RLC-1206-SMD" H 10375 2700 50  0001 C CIN
+F 3 "http://www.samsungsem.com/kr/support/product-search/mlcc/CL31B475KBHNNNE.jsp" H 10100 2875 50  0001 C CNN
+F 4 "CAP CER 4.7UF 50V X7R 1206" H 10425 2775 50  0001 C CIN "Description"
+F 5 "Samsung" H 9950 2600 50  0001 C CIN "MF_Name"
+F 6 "CL31B475KBHNNNE" H 10625 2600 50  0001 C CIN "MF_PN"
+F 7 "Digikey" H 9850 2500 50  0001 C CIN "S1_Name"
+F 8 "1276-2789-1-ND" H 10550 2500 50  0001 C CIN "S1_PN"
 	1    4975 2325
 	1    0    0    -1
@@
 P 5300 2925
 F 0 "C45" H 5400 2975 50  0000 L CNN
-F 1 "4.7uF" H 5400 2875 50  0000 L CNN
-F 2 "Wickerlib:RLC-1206-SMD" H 5925 2525 50  0001 C CIN
-F 3 "http://ds.yuden.co.jp/TYCOMPAS/ut/detail.do?productNo=UMK316AB7475KL-T&fileName=UMK316AB7475KL-T_SS&mode=specSheetDownload" H 5650 2700 50  0001 C CNN
-F 4 "CAP CER 4.7UF 50V X7R 1206" H 5975 2600 50  0001 C CIN "Description"
-F 5 "Taiyo Yuden" H 5500 2425 50  0001 C CIN "MF_Name"
-F 6 "UMK316AB7475KL-T" H 6175 2425 50  0001 C CIN "MF_PN"
-F 7 "Digikey" H 5400 2325 50  0001 C CIN "S1_Name"
-F 8 "587-2994-1-ND" H 6100 2325 50  0001 C CIN "S1_PN"
+F 1 "4.7uF" V 9875 3100 50  0000 C CNN
+F 2 "Wickerlib:RLC-1206-SMD" H 10375 2700 50  0001 C CIN
+F 3 "http://www.samsungsem.com/kr/support/product-search/mlcc/CL31B475KBHNNNE.jsp" H 10100 2875 50  0001 C CNN
+F 4 "CAP CER 4.7UF 50V X7R 1206" H 10425 2775 50  0001 C CIN "Description"
+F 5 "Samsung" H 9950 2600 50  0001 C CIN "MF_Name"
+F 6 "CL31B475KBHNNNE" H 10625 2600 50  0001 C CIN "MF_PN"
+F 7 "Digikey" H 9850 2500 50  0001 C CIN "S1_Name"
+F 8 "1276-2789-1-ND" H 10550 2500 50  0001 C CIN "S1_PN"
 	1    5300 2925
 	1    0    0    -1
@@
 P 1225 3000
 F 0 "C43" H 1325 3050 50  0000 L CNN
-F 1 "4.7uF" H 1325 2950 50  0000 L CNN
-F 2 "Wickerlib:RLC-1206-SMD" H 1850 2600 50  0001 C CIN
-F 3 "http://ds.yuden.co.jp/TYCOMPAS/ut/detail.do?productNo=UMK316AB7475KL-T&fileName=UMK316AB7475KL-T_SS&mode=specSheetDownload" H 1575 2775 50  0001 C CNN
-F 4 "CAP CER 4.7UF 50V X7R 1206" H 1900 2675 50  0001 C CIN "Description"
-F 5 "Taiyo Yuden" H 1425 2500 50  0001 C CIN "MF_Name"
-F 6 "UMK316AB7475KL-T" H 2100 2500 50  0001 C CIN "MF_PN"
-F 7 "Digikey" H 1325 2400 50  0001 C CIN "S1_Name"
-F 8 "587-2994-1-ND" H 2025 2400 50  0001 C CIN "S1_PN"
+F 1 "4.7uF" V 9875 3100 50  0000 C CNN
+F 2 "Wickerlib:RLC-1206-SMD" H 10375 2700 50  0001 C CIN
+F 3 "http://www.samsungsem.com/kr/support/product-search/mlcc/CL31B475KBHNNNE.jsp" H 10100 2875 50  0001 C CNN
+F 4 "CAP CER 4.7UF 50V X7R 1206" H 10425 2775 50  0001 C CIN "Description"
+F 5 "Samsung" H 9950 2600 50  0001 C CIN "MF_Name"
+F 6 "CL31B475KBHNNNE" H 10625 2600 50  0001 C CIN "MF_PN"
+F 7 "Digikey" H 9850 2500 50  0001 C CIN "S1_Name"
+F 8 "1276-2789-1-ND" H 10550 2500 50  0001 C CIN "S1_PN"
 	1    1225 3000
 	1    0    0    -1
