File: hardware/mcphail-main-board/input-power.sch (KiCad schematic (older format))
At the start: 34 parts, among them J8 INPUT 6V-9V, J9 JST PH, U10 BUCK-BOOST 5V TPS63060, U11 MCP1703, U9 MCP73871

Commit message: temp
Parts:
- J9: MF_PN S2B-PH-K-S(LF)(SN) -> S2B-PH-SM4-TB(LF)(SN); S1_PN 455-1719-ND -> 455-1749-1-ND
- U9: MF_PN MCP73871T-2CCI/ML -> MCP73871-2AAI/ML; S1_PN MCP73871T-2CCI/MLCT-ND -> MCP73871-2AAI/ML-ND
Changed lines of the file:
@@
 F 4 "IC USB/AC BATT CHRGR MCP73871 20QFN" H 4225 2850 50  0001 C CIN "Description"
 F 5 "Microchip" H 4225 2850 50  0001 C CIN "MF_Name"
-F 6 "MCP73871T-2CCI/ML" H 4225 2850 50  0001 C CIN "MF_PN"
+F 6 "MCP73871-2AAI/ML" H 4225 2850 50  0001 C CIN "MF_PN"
 F 7 "Digikey" H 4225 2850 50  0001 C CIN "S1_Name"
-F 8 "MCP73871T-2CCI/MLCT-ND" H 4225 2850 50  0001 C CIN "S1_PN"
+F 8 "MCP73871-2AAI/ML-ND" H 4225 2850 50  0001 C CIN "S1_PN"
 	1    4225 3550
 	1    0    0    -1
@@
 F 4 "CONN HEADER PH SIDE 2POS 2MM" H 5900 2450 50  0001 C CIN "Description"
 F 5 "JST" H 5900 2450 50  0001 C CIN "MF_Name"
-F 6 "S2B-PH-K-S(LF)(SN)" H 5900 2450 50  0001 C CIN "MF_PN"
+F 6 "S2B-PH-SM4-TB(LF)(SN)" H 5900 2450 50  0001 C CIN "MF_PN"
 F 7 "Digikey" H 5900 2450 50  0001 C CIN "S1_Name"
-F 8 "455-1719-ND" H 5900 2450 50  0001 C CIN "S1_PN"
+F 8 "455-1749-1-ND" H 5900 2450 50  0001 C CIN "S1_PN"
 	1    5900 2800
 	-1   0    0    -1

Commit message: Fixed clearance issues on McPhail Main v1.1
Changed lines of the file:
@@
 P 4975 2325
 F 0 "C44" H 5075 2375 50  0000 L CNN
-F 1 "4.7uF" V 9875 3100 50  0000 C CNN
+F 1 "4.7uF" H 5175 2300 50  0000 C CNN
 F 2 "Wickerlib:RLC-1206-SMD" H 10375 2700 50  0001 C CIN
 F 3 "http://www.samsungsem.com/kr/support/product-search/mlcc/CL31B475KBHNNNE.jsp" H 10100 2875 50  0001 C CNN
@@
 P 5300 2925
 F 0 "C45" H 5400 2975 50  0000 L CNN
-F 1 "4.7uF" V 9875 3100 50  0000 C CNN
+F 1 "4.7uF" H 5500 2900 50  0000 C CNN
 F 2 "Wickerlib:RLC-1206-SMD" H 10375 2700 50  0001 C CIN
 F 3 "http://www.samsungsem.com/kr/support/product-search/mlcc/CL31B475KBHNNNE.jsp" H 10100 2875 50  0001 C CNN
@@
 P 1225 3000
 F 0 "C43" H 1325 3050 50  0000 L CNN
-F 1 "4.7uF" V 9875 3100 50  0000 C CNN
+F 1 "4.7uF" H 1425 2975 50  0000 C CNN
 F 2 "Wickerlib:RLC-1206-SMD" H 10375 2700 50  0001 C CIN
 F 3 "http://www.samsungsem.com/kr/support/product-search/mlcc/CL31B475KBHNNNE.jsp" H 10100 2875 50  0001 C CNN
