File: hardware/mcphail-main-board/mcphail-main-board.sch (KiCad schematic (older format))
At the start: 0 parts

Commit message: Release main board sch with BOM and layout estimates.
Connections:
- net labels added: +5V, VUSB, ~PG
- wire segments 7 -> 28
Changed lines of the file:
@@
 $EndDescr
 Wire Wire Line
-	2550 4300 2850 4300
-Wire Wire Line
-	2850 4300 2850 4375
+	3925 4125 4225 4125
+Wire Wire Line
+	4225 4125 4225 4200
 $Comp
 L GND #PWR01
 U 1 1 596FA924
-P 2850 4375
-F 0 "#PWR01" H 2850 4125 50  0001 C CNN
-F 1 "GND" H 2850 4225 50  0000 C CNN
-F 2 "" H 2850 4375 50  0000 C CNN
-F 3 "" H 2850 4375 50  0000 C CNN
-	1    2850 4375
-	1    0    0    -1
-$EndComp
-Wire Wire Line
-	2550 3800 2850 3800
-Wire Wire Line
-	2850 3800 2850 3725
+P 4225 4200
+F 0 "#PWR01" H 4225 3950 50  0001 C CNN
+F 1 "GND" H 4225 4050 50  0000 C CNN
+F 2 "" H 4225 4200 50  0000 C CNN
+F 3 "" H 4225 4200 50  0000 C CNN
+	1    4225 4200
+	1    0    0    -1
+$EndComp
+Wire Wire Line
+	3925 3625 4225 3625
+Wire Wire Line
+	4225 3625 4225 3475
 $Comp
 L +3.3V #PWR02
 U 1 1 5971D5F0
-P 2850 3725
-F 0 "#PWR02" H 2850 3575 50  0001 C CNN
-F 1 "+3.3V" H 2850 3865 50  0000 C CNN
-F 2 "" H 2850 3725 50  0000 C CNN
-F 3 "" H 2850 3725 50  0000 C CNN
-	1    2850 3725
-	1    0    0    -1
-$EndComp
-Wire Wire Line
-	2550 3925 3000 3925
-Wire Wire Line
-	2550 4050 3000 4050
-Wire Wire Line
-	2550 4175 3000 4175
-Text Label 2675 3925 0    50   ~ 0
+P 4225 3475
+F 0 "#PWR02" H 4225 3325 50  0001 C CNN
+F 1 "+3.3V" H 4225 3615 50  0000 C CNN
+F 2 "" H 4225 3475 50  0000 C CNN
+F 3 "" H 4225 3475 50  0000 C CNN
+	1    4225 3475
+	1    0    0    -1
+$EndComp
+Wire Wire Line
+	3925 3750 5975 3750
+Wire Wire Line
+	3925 4000 5975 4000
+Text Label 4050 3750 0    50   ~ 0
 A0
-Text Label 2675 4050 0    50   ~ 0
+Text Label 4050 3875 0    50   ~ 0
 A1
-Text Label 2675 4175 0    50   ~ 0
+Text Label 4050 4000 0    50   ~ 0
 A2
 $Sheet
-S 1250 3500 1300 1000
+S 1975 3325 1950 975
 U 596F9466
 F0 "Photodiode Signal Input Conditioning" 50
 F1 "signal-conditioning.sch" 50
-F2 "GND" O R 2550 4300 50
-F3 "3.3V" I R 2550 3800 50
-F4 "A2" O R 2550 4175 50
-F5 "A1" O R 2550 4050 50
-F6 "A0" O R 2550 3925 50
+F2 "GND" O R 3925 4125 50
+F3 "3.3V" I R 3925 3625 50
+F4 "A2" O R 3925 4000 50
+F5 "A1" O R 3925 3875 50
+F6 "A0" O R 3925 3750 50
+F7 "5V" I R 3925 3500 50
 $EndSheet
 $Sheet
-S 3900 3125 1250 2125
+S 5975 2625 1250 2125
 U 5972781D
 F0 "Microcontroller" 50
 F1 "microcontroller.sch" 50
+F2 "VUSB" I L 5975 2850 50
+F3 "GND" O L 5975 4425 50
+F4 "5V" I L 5975 3050 50
+F5 "3.3V" I L 5975 3250 50
+F6 "A0" I L 5975 3750 50
+F7 "A1" I L 5975 3875 50
+F8 "A2" I L 5975 4000 50
+F9 "~PG" I L 5975 3475 50
 $EndSheet
 $Sheet
-S 1275 1450 1500 950
+S 2125 1450 1475 1050
 U 59727832
 F0 "Input Power" 50
 F1 "input-power.sch" 50
+F2 "VUSB" I R 3600 1675 50
+F3 "GND" O R 3600 2300 50
+F4 "5V" O R 3600 1800 50
+F5 "3.3V" O R 3600 1925 50
+F6 "~PG" O R 3600 2050 50
 $EndSheet
+Wire Wire Line
+	3600 2300 3800 2300
+Wire Wire Line
+	3800 2300 3800 2400
+$Comp
+L GND #PWR03
+U 1 1 5975C222
+P 3800 2400
+F 0 "#PWR03" H 3800 2150 50  0001 C CNN
+F 1 "GND" H 3800 2250 50  0000 C CNN
+F 2 "" H 3800 2400 50  0000 C CNN
+F 3 "" H 3800 2400 50  0000 C CNN
+	1    3800 2400
+	1    0    0    -1
+$EndComp
+Wire Wire Line
+	3600 1675 3800 1675
+Wire Wire Line
+	3800 1675 3800 1625
+$Comp
+L VUSB #PWR04
+U 1 1 5975C281
+P 3800 1625
+F 0 "#PWR04" H 3800 1475 50  0001 C CNN
+F 1 "VUSB" H 3800 1765 50  0000 C CNN
+F 2 "" H 3800 1625 50  0000 C CNN
+F 3 "" H 3800 1625 50  0000 C CNN
+	1    3800 1625
+	1    0    0    -1
+$EndComp
+Wire Wire Line
+	5975 4425 5825 4425
+Wire Wire Line
+	5825 4425 5825 4500
+$Comp
+L GND #PWR05
+U 1 1 5975C9F5
+P 5825 4500
+F 0 "#PWR05" H 5825 4250 50  0001 C CNN
+F 1 "GND" H 5825 4350 50  0000 C CNN
+F 2 "" H 5825 4500 50  0000 C CNN
+F 3 "" H 5825 4500 50  0000 C CNN
+	1    5825 4500
+	1    0    0    -1
+$EndComp
+Wire Wire Line
+	5975 2850 5825 2850
+Wire Wire Line
+	5825 2850 5825 2800
+$Comp
+L VUSB #PWR06
+U 1 1 5975CA6A
+P 5825 2800
+F 0 "#PWR06" H 5825 2650 50  0001 C CNN
+F 1 "VUSB" H 5825 2940 50  0000 C CNN
+F 2 "" H 5825 2800 50  0000 C CNN
+F 3 "" H 5825 2800 50  0000 C CNN
+	1    5825 2800
+	1    0    0    -1
+$EndComp
+Wire Wire Line
+	3925 3500 4025 3500
+Wire Wire Line
+	4025 3500 4025 3475
+$Comp
+L +5V #PWR07
+U 1 1 59822623
+P 4025 3475
+F 0 "#PWR07" H 4025 3325 50  0001 C CNN
+F 1 "+5V" H 4025 3615 50  0000 C CNN
+F 2 "" H 4025 3475 50  0000 C CNN
+F 3 "" H 4025 3475 50  0000 C CNN
+	1    4025 3475
+	1    0    0    -1
+$EndComp
+Wire Wire Line
+	3600 1800 3950 1800
+Wire Wire Line
+	3950 1800 3950 1725
+$Comp
+L +5V #PWR08
+U 1 1 5985C6DD
+P 3950 1725
+F 0 "#PWR08" H 3950 1575 50  0001 C CNN
+F 1 "+5V" H 3950 1865 50  0000 C CNN
+F 2 "" H 3950 1725 50  0000 C CNN
+F 3 "" H 3950 1725 50  0000 C CNN
+	1    3950 1725
+	1    0    0    -1
+$EndComp
+Wire Wire Line
+	3600 1925 4125 1925
+Wire Wire Line
+	4125 1925 4125 1825
+$Comp
+L +3.3V #PWR09
+U 1 1 5985C785
+P 4125 1825
+F 0 "#PWR09" H 4125 1675 50  0001 C CNN
+F 1 "+3.3V" H 4125 1965 50  0000 C CNN
+F 2 "" H 4125 1825 50  0000 C CNN
+F 3 "" H 4125 1825 50  0000 C CNN
+	1    4125 1825
+	1    0    0    -1
+$EndComp
+Wire Wire Line
+	3600 2050 4900 2050
+Text Label 3650 2050 0    50   ~ 0
+~PG
+Wire Wire Line
+	5975 3250 5375 3250
+Wire Wire Line
+	5375 3250 5375 3200
+$Comp
+L +3.3V #PWR010
+U 1 1 598615E2
+P 5375 3200
+F 0 "#PWR010" H 5375 3050 50  0001 C CNN
+F 1 "+3.3V" H 5375 3340 50  0000 C CNN
+F 2 "" H 5375 3200 50  0000 C CNN
+F 3 "" H 5375 3200 50  0000 C CNN
+	1    5375 3200
+	1    0    0    -1
+$EndComp
+Wire Wire Line
+	5975 3050 5600 3050
+Wire Wire Line
+	5600 3050 5600 2975
+$Comp
+L +5V #PWR011
+U 1 1 598617B5
+P 5600 2975
+F 0 "#PWR011" H 5600 2825 50  0001 C CNN
+F 1 "+5V" H 5600 3115 50  0000 C CNN
+F 2 "" H 5600 2975 50  0000 C CNN
+F 3 "" H 5600 2975 50  0000 C CNN
+	1    5600 2975
+	1    0    0    -1
+$EndComp
+Wire Wire Line
+	3925 3875 5975 3875
+Wire Wire Line
+	5975 3475 4900 3475
+Wire Wire Line
+	4900 3475 4900 2050
+Text Label 5600 3475 0    50   ~ 0
+~PG
+Text Label 5600 3750 0    50   ~ 0
+A0
+Text Label 5600 3875 0    50   ~ 0
+A1
+Text Label 5600 4000 0    50   ~ 0
+A2
 $EndSCHEMATC

Commit message: Hooked up pins to ATSAMD21G18 Cortex M0, fixed AGND throughout.
Changed lines of the file:
@@
 F0 "Microcontroller" 50
 F1 "microcontroller.sch" 50
-F2 "VUSB" I L 5975 2850 50
+F2 "VUSB" O L 5975 2850 50
 F3 "GND" O L 5975 4425 50
 F4 "5V" I L 5975 3050 50
@@
 F8 "A2" I L 5975 4000 50
 F9 "~PG" I L 5975 3475 50
+F10 "AGND" O L 5975 4325 50
 $EndSheet
 $Sheet
@@
 Text Label 5600 4000 0    50   ~ 0
 A2
+$Comp
+L AGND #PWR012
+U 1 1 59864395
+P 5550 4500
+F 0 "#PWR012" H 5550 4250 50  0001 C CNN
+F 1 "AGND" H 5550 4350 50  0000 C CNN
+F 2 "" H 5550 4500 50  0000 C CNN
+F 3 "" H 5550 4500 50  0000 C CNN
+	1    5550 4500
+	1    0    0    -1
+$EndComp
+Wire Wire Line
+	5550 4500 5550 4325
+Wire Wire Line
+	5550 4325 5975 4325
 $EndSCHEMATC

Commit message: Sch passes rule check. Final netlist. Starting layout.
Changed lines of the file:
@@
 Wire Wire Line
 	4225 4125 4225 4200
-$Comp
-L GND #PWR7
-U 1 1 596FA924
-P 4225 4200
-F 0 "#PWR7" H 4225 3950 50  0001 C CNN
-F 1 "GND" H 4225 4050 50  0000 C CNN
-F 2 "" H 4225 4200 50  0000 C CNN
-F 3 "" H 4225 4200 50  0000 C CNN
-	1    4225 4200
-	1    0    0    -1
-$EndComp
 Wire Wire Line
 	3925 3625 4225 3625
@@
 	4225 3625 4225 3475
 $Comp
-L +3.3V #PWR6
+L +3.3V #PWR01
 U 1 1 5971D5F0
 P 4225 3475
-F 0 "#PWR6" H 4225 3325 50  0001 C CNN
+F 0 "#PWR01" H 4225 3325 50  0001 C CNN
 F 1 "+3.3V" H 4225 3615 50  0000 C CNN
 F 2 "" H 4225 3475 50  0000 C CNN
@@
 F0 "Photodiode Signal Input Conditioning" 50
 F1 "signal-conditioning.sch" 50
-F2 "GND" O R 3925 4125 50
-F3 "3.3V" I R 3925 3625 50
-F4 "A2" O R 3925 4000 50
-F5 "A1" O R 3925 3875 50
-F6 "A0" O R 3925 3750 50
-F7 "5V" I R 3925 3500 50
+F2 "3.3V" I R 3925 3625 50
+F3 "A2" O R 3925 4000 50
+F4 "A1" O R 3925 3875 50
+F5 "A0" O R 3925 3750 50
+F6 "5V" I R 3925 3500 50
+F7 "AGND" O R 3925 4125 50
 $EndSheet
 $Sheet
@@
 	3800 2300 3800 2400
 $Comp
-L GND #PWR2
+L GND #PWR02
 U 1 1 5975C222
 P 3800 2400
-F 0 "#PWR2" H 3800 2150 50  0001 C CNN
+F 0 "#PWR02" H 3800 2150 50  0001 C CNN
 F 1 "GND" H 3800 2250 50  0000 C CNN
 F 2 "" H 3800 2400 50  0000 C CNN
@@
 	3800 1675 3800 1625
 $Comp
-L VUSB #PWR1
+L VUSB #PWR03
 U 1 1 5975C281
 P 3800 1625
-F 0 "#PWR1" H 3800 1475 50  0001 C CNN
+F 0 "#PWR03" H 3800 1475 50  0001 C CNN
 F 1 "VUSB" H 3800 1765 50  0000 C CNN
 F 2 "" H 3800 1625 50  0000 C CNN
@@
 	5825 4425 5825 4500
 $Comp
-L GND #PWR12
+L GND #PWR04
 U 1 1 5975C9F5
 P 5825 4500
-F 0 "#PWR12" H 5825 4250 50  0001 C CNN
+F 0 "#PWR04" H 5825 4250 50  0001 C CNN
 F 1 "GND" H 5825 4350 50  0000 C CNN
 F 2 "" H 5825 4500 50  0000 C CNN
@@
 	5825 2850 5825 2800
 $Comp
-L VUSB #PWR11
+L VUSB #PWR05
 U 1 1 5975CA6A
 P 5825 2800
-F 0 "#PWR11" H 5825 2650 50  0001 C CNN
+F 0 "#PWR05" H 5825 2650 50  0001 C CNN
 F 1 "VUSB" H 5825 2940 50  0000 C CNN
 F 2 "" H 5825 2800 50  0000 C CNN
@@
 	4025 3500 4025 3475
 $Comp
-L +5V #PWR4
+L +5V #PWR06
 U 1 1 59822623
 P 4025 3475
-F 0 "#PWR4" H 4025 3325 50  0001 C CNN
+F 0 "#PWR06" H 4025 3325 50  0001 C CNN
 F 1 "+5V" H 4025 3615 50  0000 C CNN
 F 2 "" H 4025 3475 50  0000 C CNN
@@
 	3950 1800 3950 1725
 $Comp
-L +5V #PWR3
+L +5V #PWR07
 U 1 1 5985C6DD
 P 3950 1725
-F 0 "#PWR3" H 3950 1575 50  0001 C CNN
+F 0 "#PWR07" H 3950 1575 50  0001 C CNN
 F 1 "+5V" H 3950 1865 50  0000 C CNN
 F 2 "" H 3950 1725 50  0000 C CNN
@@
 	4125 1925 4125 1825
 $Comp
-L +3.3V #PWR5
+L +3.3V #PWR08
 U 1 1 5985C785
 P 4125 1825
-F 0 "#PWR5" H 4125 1675 50  0001 C CNN
+F 0 "#PWR08" H 4125 1675 50  0001 C CNN
 F 1 "+3.3V" H 4125 1965 50  0000 C CNN
 F 2 "" H 4125 1825 50  0000 C CNN
@@
 	5375 3250 5375 3200
 $Comp
-L +3.3V #PWR8
+L +3.3V #PWR09
 U 1 1 598615E2
 P 5375 3200
-F 0 "#PWR8" H 5375 3050 50  0001 C CNN
+F 0 "#PWR09" H 5375 3050 50  0001 C CNN
 F 1 "+3.3V" H 5375 3340 50  0000 C CNN
 F 2 "" H 5375 3200 50  0000 C CNN
@@
 	5600 3050 5600 2975
 $Comp
-L +5V #PWR10
+L +5V #PWR010
 U 1 1 598617B5
 P 5600 2975
-F 0 "#PWR10" H 5600 2825 50  0001 C CNN
+F 0 "#PWR010" H 5600 2825 50  0001 C CNN
 F 1 "+5V" H 5600 3115 50  0000 C CNN
 F 2 "" H 5600 2975 50  0000 C CNN
@@
 A2
 $Comp
-L AGND #PWR9
+L AGND #PWR011
 U 1 1 59864395
 P 5550 4500
-F 0 "#PWR9" H 5550 4250 50  0001 C CNN
+F 0 "#PWR011" H 5550 4250 50  0001 C CNN
 F 1 "AGND" H 5550 4350 50  0000 C CNN
 F 2 "" H 5550 4500 50  0000 C CNN
@@
 Wire Wire Line
 	5550 4325 5975 4325
+$Comp
+L AGND #PWR012
+U 1 1 5983011F
+P 4225 4200
+F 0 "#PWR012" H 4225 3950 50  0001 C CNN
+F 1 "AGND" H 4225 4050 50  0000 C CNN
+F 2 "" H 4225 4200 50  0000 C CNN
+F 3 "" H 4225 4200 50  0000 C CNN
+	1    4225 4200
+	1    0    0    -1
+$EndComp
 $EndSCHEMATC

Commit message: Reworking main board, power rails routed next.
Changed lines of the file:
@@
 Comment4 ""
 $EndDescr
-Wire Wire Line
-	3925 4125 4225 4125
-Wire Wire Line
-	4225 4125 4225 4200
-Wire Wire Line
-	3925 3625 4225 3625
-Wire Wire Line
-	4225 3625 4225 3475
-$Comp
-L +3.3V #PWR01
-U 1 1 5971D5F0
-P 4225 3475
-F 0 "#PWR01" H 4225 3325 50  0001 C CNN
-F 1 "+3.3V" H 4225 3615 50  0000 C CNN
-F 2 "" H 4225 3475 50  0000 C CNN
-F 3 "" H 4225 3475 50  0000 C CNN
-	1    4225 3475
-	1    0    0    -1
-$EndComp
-Wire Wire Line
-	3925 3750 5975 3750
-Wire Wire Line
-	3925 4000 5975 4000
 Text Label 4050 3750 0    50   ~ 0
 A0
@@
 F0 "Photodiode Signal Input Conditioning" 50
 F1 "signal-conditioning.sch" 50
-F2 "3.3V" I R 3925 3625 50
+F2 "VDDANA" I R 3925 3625 50
 F3 "A2" O R 3925 4000 50
 F4 "A1" O R 3925 3875 50
@@
 F9 "~PG" I L 5975 3475 50
 F10 "AGND" O L 5975 4325 50
+F11 "VDDANA" O L 5975 3625 50
 $EndSheet
 $Sheet
@@
 F6 "~PG" O R 3600 2050 50
 $EndSheet
-Wire Wire Line
-	3600 2300 3800 2300
-Wire Wire Line
-	3800 2300 3800 2400
-$Comp
-L GND #PWR02
+$Comp
+L GND #PWR01
 U 1 1 5975C222
 P 3800 2400
-F 0 "#PWR02" H 3800 2150 50  0001 C CNN
+F 0 "#PWR01" H 3800 2150 50  0001 C CNN
 F 1 "GND" H 3800 2250 50  0000 C CNN
 F 2 "" H 3800 2400 50  0000 C CNN
@@
 	1    0    0    -1
 $EndComp
-Wire Wire Line
-	3600 1675 3800 1675
-Wire Wire Line
-	3800 1675 3800 1625
-$Comp
-L VUSB #PWR03
+$Comp
+L VUSB #PWR02
 U 1 1 5975C281
 P 3800 1625
-F 0 "#PWR03" H 3800 1475 50  0001 C CNN
+F 0 "#PWR02" H 3800 1475 50  0001 C CNN
 F 1 "VUSB" H 3800 1765 50  0000 C CNN
 F 2 "" H 3800 1625 50  0000 C CNN
@@
 	1    0    0    -1
 $EndComp
-Wire Wire Line
-	5975 4425 5825 4425
-Wire Wire Line
-	5825 4425 5825 4500
-$Comp
-L GND #PWR04
+$Comp
+L GND #PWR03
 U 1 1 5975C9F5
 P 5825 4500
-F 0 "#PWR04" H 5825 4250 50  0001 C CNN
+F 0 "#PWR03" H 5825 4250 50  0001 C CNN
 F 1 "GND" H 5825 4350 50  0000 C CNN
 F 2 "" H 5825 4500 50  0000 C CNN
@@
 	1    0    0    -1
 $EndComp
-Wire Wire Line
-	5975 2850 5825 2850
-Wire Wire Line
-	5825 2850 5825 2800
-$Comp
-L VUSB #PWR05
+$Comp
+L VUSB #PWR04
 U 1 1 5975CA6A
 P 5825 2800
-F 0 "#PWR05" H 5825 2650 50  0001 C CNN
+F 0 "#PWR04" H 5825 2650 50  0001 C CNN
 F 1 "VUSB" H 5825 2940 50  0000 C CNN
 F 2 "" H 5825 2800 50  0000 C CNN
@@
 	1    0    0    -1
 $EndComp
-Wire Wire Line
-	3925 3500 4025 3500
-Wire Wire Line
-	4025 3500 4025 3475
-$Comp
-L +5V #PWR06
+$Comp
+L +5V #PWR05
 U 1 1 59822623
 P 4025 3475
-F 0 "#PWR06" H 4025 3325 50  0001 C CNN
+F 0 "#PWR05" H 4025 3325 50  0001 C CNN
 F 1 "+5V" H 4025 3615 50  0000 C CNN
 F 2 "" H 4025 3475 50  0000 C CNN
@@
 	1    0    0    -1
 $EndComp
-Wire Wire Line
-	3600 1800 3950 1800
-Wire Wire Line
-	3950 1800 3950 1725
-$Comp
-L +5V #PWR07
+$Comp
+L +5V #PWR06
 U 1 1 5985C6DD
 P 3950 1725
-F 0 "#PWR07" H 3950 1575 50  0001 C CNN
+F 0 "#PWR06" H 3950 1575 50  0001 C CNN
 F 1 "+5V" H 3950 1865 50  0000 C CNN
 F 2 "" H 3950 1725 50  0000 C CNN
@@
 	1    0    0    -1
 $EndComp
-Wire Wire Line
-	3600 1925 4125 1925
-Wire Wire Line
-	4125 1925 4125 1825
-$Comp
-L +3.3V #PWR08
+$Comp
+L +3.3V #PWR07
 U 1 1 5985C785
 P 4125 1825
-F 0 "#PWR08" H 4125 1675 50  0001 C CNN
+F 0 "#PWR07" H 4125 1675 50  0001 C CNN
 F 1 "+3.3V" H 4125 1965 50  0000 C CNN
 F 2 "" H 4125 1825 50  0000 C CNN
@@
 	1    0    0    -1
 $EndComp
-Wire Wire Line
-	3600 2050 4900 2050
 Text Label 3650 2050 0    50   ~ 0
 ~PG
-Wire Wire Line
-	5975 3250 5375 3250
-Wire Wire Line
-	5375 3250 5375 3200
-$Comp
-L +3.3V #PWR09
-U 1 1 598615E2
-P 5375 3200
-F 0 "#PWR09" H 5375 3050 50  0001 C CNN
-F 1 "+3.3V" H 5375 3340 50  0000 C CNN
-F 2 "" H 5375 3200 50  0000 C CNN
-F 3 "" H 5375 3200 50  0000 C CNN
-	1    5375 3200
-	1    0    0    -1
-$EndComp
-Wire Wire Line
-	5975 3050 5600 3050
-Wire Wire Line
-	5600 3050 5600 2975
-$Comp
-L +5V #PWR010
+$Comp
+L +5V #PWR08
 U 1 1 598617B5
 P 5600 2975
-F 0 "#PWR010" H 5600 2825 50  0001 C CNN
+F 0 "#PWR08" H 5600 2825 50  0001 C CNN
 F 1 "+5V" H 5600 3115 50  0000 C CNN
 F 2 "" H 5600 2975 50  0000 C CNN
@@
 	1    0    0    -1
 $EndComp
-Wire Wire Line
-	3925 3875 5975 3875
-Wire Wire Line
-	5975 3475 4900 3475
-Wire Wire Line
-	4900 3475 4900 2050
 Text Label 5600 3475 0    50   ~ 0
 ~PG
@@
 A2
 $Comp
-L AGND #PWR011
+L AGND #PWR09
 U 1 1 59864395
 P 5550 4500
-F 0 "#PWR011" H 5550 4250 50  0001 C CNN
+F 0 "#PWR09" H 5550 4250 50  0001 C CNN
 F 1 "AGND" H 5550 4350 50  0000 C CNN
 F 2 "" H 5550 4500 50  0000 C CNN
@@
 	1    0    0    -1
 $EndComp
-Wire Wire Line
-	5550 4500 5550 4325
-Wire Wire Line
-	5550 4325 5975 4325
-$Comp
-L AGND #PWR012
+$Comp
+L AGND #PWR010
 U 1 1 5983011F
 P 4225 4200
-F 0 "#PWR012" H 4225 3950 50  0001 C CNN
+F 0 "#PWR010" H 4225 3950 50  0001 C CNN
 F 1 "AGND" H 4225 4050 50  0000 C CNN
 F 2 "" H 4225 4200 50  0000 C CNN
@@
 	1    0    0    -1
 $EndComp
+Text Label 4050 3625 0    50   ~ 0
+VDDANA
+Wire Wire Line
+	3925 4125 4225 4125
+Wire Wire Line
+	4225 4125 4225 4200
+Wire Wire Line
+	3925 3625 5975 3625
+Wire Wire Line
+	3925 3750 5975 3750
+Wire Wire Line
+	3925 4000 5975 4000
+Wire Wire Line
+	3600 2300 3800 2300
+Wire Wire Line
+	3800 2300 3800 2400
+Wire Wire Line
+	3600 1675 3800 1675
+Wire Wire Line
+	3800 1675 3800 1625
+Wire Wire Line
+	5975 4425 5825 4425
+Wire Wire Line
+	5825 4425 5825 4500
+Wire Wire Line
+	5975 2850 5825 2850
+Wire Wire Line
+	5825 2850 5825 2800
+Wire Wire Line
+	3925 3500 4025 3500
+Wire Wire Line
+	4025 3500 4025 3475
+Wire Wire Line
+	3600 1800 3950 1800
+Wire Wire Line
+	3950 1800 3950 1725
+Wire Wire Line
+	3600 1925 4125 1925
+Wire Wire Line
+	4125 1925 4125 1825
+Wire Wire Line
+	3600 2050 4900 2050
+Wire Wire Line
+	5975 3250 5375 3250
+Wire Wire Line
+	5975 3050 5600 3050
+Wire Wire Line
+	5600 3050 5600 2975
+Wire Wire Line
+	3925 3875 5975 3875
+Wire Wire Line
+	5975 3475 4900 3475
+Wire Wire Line
+	4900 3475 4900 2050
+Wire Wire Line
+	5550 4500 5550 4325
+Wire Wire Line
+	5550 4325 5975 4325
+Wire Wire Line
+	5375 3250 5375 3200
+$Comp
+L +3.3V #PWR011
+U 1 1 598615E2
+P 5375 3200
+F 0 "#PWR011" H 5375 3050 50  0001 C CNN
+F 1 "+3.3V" H 5375 3340 50  0000 C CNN
+F 2 "" H 5375 3200 50  0000 C CNN
+F 3 "" H 5375 3200 50  0000 C CNN
+	1    5375 3200
+	1    0    0    -1
+$EndComp
