File: hardware/mcphail-zero-analog-shield/mcphail-zero-analog-shield.kicad_pcb (KiCad board)
At the start: 2 copper layers, 80.6 x 56.6 mm, 143 parts, among them J1 INSECT DETECTION, J2 EMITTERS, J3 BREAKOUT, J4 MICRO SD, J5 MICRO USB, J6 PROG/BOOT, J7 FONA 808, J8 INPUT 6V-9V, J9 JST PH, U1 MCP6004, U10 BUCK-BOOST 5V TPS63060, U11 MCP1703, U2 MCP6004, U3 TLV274, U4 MCP6001, U5 ADS1118, U6 ATSAMD21G18A, U7 24AA1025 EEPROM, U8 MCP7940N RTC, U9 MCP73871, X1 16MHz, X2 32.768kHz

Commit message: Only comps we need left on board. Needs routed.
Parts:
- removed BAT1: 3V, Wickerlib:BATT-HOLDER-CR1220-BK-916
- removed C30, C36, C37, C38, C39, C47, C51, C52: 100nF, Wickerlib:RLC-0603-SMD
- removed C31, C46, C53: 10uF, Wickerlib:RLC-0805-SMD
- removed C33, C35: 22pF, Wickerlib:RLC-0603-SMD
- removed C34, C49, C50: 1uF, Wickerlib:RLC-0805-SMD
- removed C40, C42: 2pF, Wickerlib:RLC-0603-SMD
- removed C41: 100pF, Wickerlib:RLC-0603-SMD
- removed C43, C44, C45: 4.7uF, Wickerlib:RLC-1206-SMD
- removed C48: 10pF, Wickerlib:RLC-0603-SMD
- removed C54, C55, C56: 22uF, Wickerlib:RLC-1210-SMD
- removed D1, D4: 20V 1A, Wickerlib:DIODE-SMA
- removed D2, D3: CG0603MLC-05E, Wickerlib:RLC-0603-SMD
- removed F1: 500mA, Wickerlib:RLC-1812-SMD
- removed FID1, FID2, FID3: FIDUCIAL, Wickerlib:FIDUCIAL-2MM
- removed J4: MICRO SD, Wickerlib:CONN-SD-MICRO-MOLEX-0475710001
- removed J5: MICRO USB, Wickerlib:CONN-USB-MICRO-B-AMPHENOL-10118193-0001LF
- removed J6: PROG/BOOT, Wickerlib:CONN-HEADER-STRAIGHT-P2.54MM-2x03
- removed J7: FONA 808, Wickerlib:BREAKOUT-ADAFRUIT-FONA808-CELL-GPS
- removed J8: INPUT 6V-9V, Wickerlib:CONN-BARREL-JACK-2.5x5.5MM-TH
- removed J9: JST PH, Wickerlib:CONN-JST-S2B-PH-SM4-TB
- removed L1, L3, L4, L5: FERRITE, Wickerlib:RLC-0805-SMD
- removed L2: 1uH 3.3A, Wickerlib:1226AS-H-1R0N
- removed LED2, LED3: AMBER, Wickerlib:LED-0603-SMD
- removed R33, R36: 10K, Wickerlib:RLC-0603-SMD
- removed R34, R35, R43: 2K, Wickerlib:RLC-0603-SMD
- removed R37: 1K, Wickerlib:RLC-0603-SMD
- removed R38: 0 ohm, Wickerlib:RLC-0603-SMD
- removed R39, R40, R41: 470, Wickerlib:RLC-0603-SMD
- removed R42: NTC 10K, Wickerlib:RLC-0402-SMD
- removed R44: 100K, Wickerlib:RLC-0603-SMD
- removed R45, R47: 1M, Wickerlib:RLC-0603-SMD
- removed R46: 111K, Wickerlib:RLC-0603-SMD
- removed U1, U2: MCP6004, Wickerlib:SOIC-14-3.9x8.7MM-P1.27MM
- removed U11: MCP1703, Wickerlib:SOT-23-3
- removed U5: ADS1118, Wickerlib:MSOP-10-3x3MM-P0.5MM
- removed U8: MCP7940N RTC, Wickerlib:SOIC-8-3.9x4.9MM-P1.27MM
- removed U9: MCP73871, Wickerlib:QFN-20-1EP-4x4MM_P0.5MM
- removed W1: TEST_1P, Wickerlib:HOLE-PLATED-40MIL
- removed X1: 16MHz, Wickerlib:CRYSTAL-CTS-4SMD
- removed X2: 32.768kHz, Wickerlib:CRYSTAL-HC49-TH
- J3: value BREAKOUT -> VREF; footprint Wickerlib:CONN-HEADER-STRAIGHT-P2.54MM-1x06 -> Wickerlib:CONN-HEADER-STRAIGHT-P2.54MM-1x01
- R31: value 330 -> 0 ohm
- R32: value 1K -> 220
- U10: value BUCK-BOOST 5V TPS63060 -> ARDUINO-101-SHIELD; footprint Wickerlib:WSON-10-1EP -> Wickerlib:ARDUINO-UNO-SHIELD
- U6: value ATSAMD21G18A -> MCP6004; footprint Wickerlib:TQFP-48_7x7mm_Pitch0.5mm -> Wickerlib:SOIC-14-3.9x8.7MM-P1.27MM
- U7: value 24AA1025 EEPROM -> MCP6004; footprint Wickerlib:SOIC-8-3.9x4.9MM-P1.27MM -> Wickerlib:SOIC-14-3.9x8.7MM-P1.27MM
- moved U10 131.1 mm to (31.0, 172.6), turned to 0 degrees
Connections:
- net /Photodiode Signal Input Conditioning/PHOTO_K renamed /PHOTO_K
- C10 pad 2: /Photodiode Signal Input Conditioning/VREF -> /VREF
- C14 pad 2: AGND -> GND
- C18 pad 1: /Photodiode Signal Input Conditioning/LINE_IN -> /LINE_IN
- C22 pad 2: /Photodiode Signal Input Conditioning/LINE_IN -> /LINE_IN
- C25 pad 1: /VDDANA -> +3V3
- C25 pad 2: AGND -> GND
- C26 pad 1: /VDDANA -> +3V3
- C26 pad 2: AGND -> GND
- C27 pad 2: /Photodiode Signal Input Conditioning/VREF -> /VREF
- C29 pad 2: AGND -> GND
- C3 pad 2: AGND -> GND
- C4 pad 2: AGND -> GND
- C5 pad 2: /Photodiode Signal Input Conditioning/VREF -> /VREF
- C6 pad 1: /Photodiode Signal Input Conditioning/VREF -> /VREF
- C6 pad 2: AGND -> GND
- C9 pad 1: /Photodiode Signal Input Conditioning/VREF -> /VREF
- C9 pad 2: AGND -> GND
- J1 pad 2: AGND -> GND
- J3 pad 1: +5V -> /VREF
- LED1 pad 2: VIN -> Net-(LED1-Pad2)
- R14 pad 2: /Photodiode Signal Input Conditioning/VREF -> /VREF
- R15 pad 1: /Photodiode Signal Input Conditioning/LINE_IN -> /LINE_IN
- R17 pad 2: /Photodiode Signal Input Conditioning/VREF -> /VREF
- R18 pad 1: /VDDANA -> +3V3
- R19 pad 2: AGND -> GND
- R20 pad 1: /VDDANA -> +3V3
- R31 pad 1: /Microcontroller/~RESET -> +3V3
- R32 pad 1: +3V3 -> Net-(LED1-Pad1)
- R32 pad 2: /Microcontroller/SWCLK -> GND
- R4 pad 2: AGND -> GND
- R7 pad 1: /Photodiode Signal Input Conditioning/VREF -> /VREF
- R9 pad 2: /Photodiode Signal Input Conditioning/VREF -> /VREF
- S1 pad 1: Net-(R31-Pad2) -> Net-(S1-Pad1)
- U3 pad 11: AGND -> GND
- U3 pad 4: /VDDANA -> +3V3
- U4 pad 2: AGND -> GND
- U4 pad 3: AGND -> GND
- U6 pad 1: (no net) -> Net-(C13-Pad1)
- U6 pad 10: /A2 -> /VREF
- U6 pad 11: /A1 -> GND
- U6 pad 12: /A0 -> Net-(C4-Pad1)
- U6 pad 13: /Microcontroller/D4_CS -> Net-(R7-Pad2)
- U6 pad 14: /Microcontroller/SCLK -> Net-(R7-Pad2)
- U6 pad 2: (no net) -> Net-(C11-Pad1)
- U6 pad 3: (no net) -> /VREF
- U6 pad 4: (no net) -> +5V
- U6 pad 5: AGND -> /VREF
- U6 pad 6: /VDDANA -> Net-(C8-Pad2)
- U6 pad 7: (no net) -> Net-(C8-Pad1)
- U6 pad 8: (no net) -> Net-(C12-Pad1)
- U6 pad 9: (no net) -> Net-(C12-Pad2)
- U7 pad 1: /Microcontroller/EEPROM_ADD0 -> Net-(C28-Pad1)
- U7 pad 2: /Microcontroller/EEPROM_ADD1 -> Net-(C28-Pad2)
- U7 pad 3: /Microcontroller/EEPROM_ADD2 -> /VREF
- U7 pad 4: GND -> +5V
- U7 pad 5: /Microcontroller/SDA -> /VREF
- U7 pad 6: /Microcontroller/SCL -> Net-(C17-Pad1)
- U7 pad 7: GND -> Net-(C19-Pad1)
- U7 pad 8: +3V3 -> Net-(C24-Pad1)
Routing:
- net (no net): track 0.00 -> 967.4 mm, vias 1 -> 102
- net /VREF: track 0.00 -> 83.4 mm, vias 0 -> 6
- net AGND: track 75.7 -> 0.00 mm, vias 32 -> 0
- net +3V3: track 152.2 -> 76.8 mm, vias 10 -> 3
- net +5V: track 205.6 -> 132.0 mm, vias 9 -> 7
- net Net-(C12-Pad2): track 4.39 -> 74.0 mm, vias 0 -> 5
- net /Photodiode Signal Input Conditioning/VREF: track 69.5 -> 0.00 mm, vias 4 -> 0
- net GND: track 167.8 -> 111.3 mm, vias 53 -> 27
- net /Microcontroller/D-: track 54.6 -> 0.00 mm, vias 2 -> 0
- net /Microcontroller/D+: track 53.1 -> 0.00 mm, vias 2 -> 0
- net /Microcontroller/FONA_PS: track 52.2 -> 0.00 mm, vias 5 -> 0
- net /VDDANA: track 50.2 -> 0.00 mm, vias 2 -> 0
- net /Microcontroller/SCLK: track 45.9 -> 0.00 mm, vias 3 -> 0
- net Net-(BAT1-Pad1): track 38.7 -> 0.00 mm, vias 1 -> 0
- net /Input Power/VCC: track 38.3 -> 0.00 mm
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- removed copper zone on B.Cu, net AGND
- removed copper zone on F.Cu, net AGND
Other:
- board outline removed

Commit message: Parts on board with no traces, clean. Ready to layout.
Parts:
- moved S1 111.6 mm to (53.9, 169.2), turned to 180 degrees
- moved U6 88.2 mm to (51.8, 154.8), turned to 180 degrees
- moved U7 78.9 mm to (52.3, 138.0), turned to 90 degrees
- moved R31 72.0 mm to (77.0, 133.1)
- moved LED1 71.7 mm to (77.7, 126.1)
- moved R32 71.7 mm to (77.7, 128.6), turned to 180 degrees
- moved C17 68.2 mm to (62.4, 152.8)
- moved C2 68.2 mm to (79.1, 154.8)
- moved C21 68.2 mm to (61.0, 145.8)
- moved C22 68.2 mm to (58.3, 139.4)
- moved C23 68.2 mm to (46.6, 150.5)
- moved C27 68.2 mm to (41.7, 153.5)
- moved R13 68.2 mm to (58.3, 136.2)
- moved R15 68.2 mm to (55.3, 143.0)
- moved R17 68.2 mm to (51.0, 149.0)
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Routing:
- net (no net): track 967.4 -> 0.00 mm, vias 102 -> 0
- net +5V: track 132.0 -> 0.00 mm, vias 7 -> 0
- net GND: track 111.3 -> 0.00 mm, vias 27 -> 0
- net /VREF: track 83.4 -> 0.00 mm, vias 6 -> 0
- net +3V3: track 76.8 -> 0.00 mm, vias 3 -> 0
- net Net-(C12-Pad2): track 74.0 -> 0.00 mm, vias 5 -> 0
- net /A0: track 44.8 -> 0.00 mm
- net /A2: track 38.2 -> 0.00 mm, vias 2 -> 0
- net Net-(LED1-Pad2): track 37.3 -> 0.00 mm, vias 2 -> 0
- net Net-(C17-Pad1): track 35.2 -> 0.00 mm
- net Net-(C18-Pad2): track 31.5 -> 0.00 mm
- net /A1: track 29.7 -> 0.00 mm, vias 2 -> 0
- net Net-(U3-Pad12): track 15.8 -> 0.00 mm
- net /PHOTO_K: track 14.3 -> 0.00 mm
- net Net-(C11-Pad2): track 14.3 -> 0.00 mm
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Other:
- board text added: "McPhail Zero Analog Shield v1.0 Kyle Birchard and Jenner Hanni"
- board text removed: "3.3V"
- board text removed: "5V"
- board text removed: "McPhail Trap Main Board v1.1 Kyle Birchard and Jenner Hanni"
- board text removed: "PIN1"

Commit message: Starting layout.
Parts:
- moved R1 25.5 mm to (82.3, 129.3), turned to 0 degrees
- moved J2 22.5 mm to (90.6, 133.2), turned to 0 degrees
- moved C1 15.8 mm to (82.4, 134.9), turned to 270 degrees
- moved R31 5.24 mm to (71.8, 134.2)
- moved R32 4.84 mm to (82.4, 127.3), turned to 0 degrees
- moved LED1 1.17 mm to (77.7, 127.3)
Routing:
- net Net-(LED1-Pad2): track 0.00 -> 5.95 mm
- net Net-(LED1-Pad1): track 0.00 -> 3.18 mm

Commit message: More placement.
Parts:
- moved C1 65.1 mm to (17.2, 136.2)
- moved J2 65.1 mm to (25.4, 134.5)
- moved R1 65.1 mm to (17.2, 130.6)
- moved J1 59.8 mm to (16.5, 160.9), turned to 180 degrees
- moved C2 55.7 mm to (24.1, 163.6), turned to 180 degrees
- moved U4 54.8 mm to (20.3, 159.7), turned to 270 degrees
- moved C3 53.0 mm to (22.8, 160.3), turned to 90 degrees
- moved R2 49.6 mm to (24.9, 158.9), turned to 270 degrees
- moved C7 49.2 mm to (21.7, 155.4), turned to 0 degrees
- moved R21 23.5 mm to (81.8, 160.5)
- moved R18 23.5 mm to (80.1, 152.7)
- moved R24 23.5 mm to (83.4, 151.8)
- moved R19 23.5 mm to (80.2, 149.0)
- moved C21 23.5 mm to (79.3, 160.5)
- moved C25 23.5 mm to (80.7, 154.7)
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Routing:
- net Net-(LED1-Pad2): track 5.95 -> 20.3 mm
- net Net-(LED1-Pad1): track 3.18 -> 2.14 mm
Other:
- board text removed: "SIGOUT"

Commit message: Re-import netlist, override existing.
Parts:
- removed U10: ARDUINO-101-SHIELD, Wickerlib:ARDUINO-UNO-SHIELD
- removed U6, U7: MCP6004, Wickerlib:SOIC-14-3.9x8.7MM-P1.27MM
- added U1: MCP6001, Wickerlib:SOT-23-5, F.Cu at (19.1, 101.2)
- added U2: MCP6004, Wickerlib:SOIC-14-3.9x8.7MM-P1.27MM, F.Cu at (19.1, 101.2)
- added U5: ARDUINO-101-SHIELD, Wickerlib:ARDUINO-UNO-SHIELD, F.Cu at (31.1, 172.4)
- U3: value TLV274 -> MCP6004
- U4: value MCP6001 -> TLV274; footprint Wickerlib:SOT-23-5 -> Wickerlib:SOIC-14-3.9x8.7MM-P1.27MM
Connections:
- U3 pad 1: Net-(R24-Pad1) -> Net-(C28-Pad1)
- U3 pad 10: (no net) -> /VREF
- U3 pad 12: Net-(U3-Pad12) -> /VREF
- U3 pad 13: /A1 -> Net-(C18-Pad2)
- U3 pad 14: /A2 -> /LINE_IN
- U3 pad 2: Net-(R22-Pad1) -> Net-(C28-Pad2)
- U3 pad 3: Net-(U3-Pad12) -> /VREF
- U3 pad 4: +3V3 -> +5V
- U3 pad 5: Net-(C21-Pad1) -> /VREF
- U3 pad 6: Net-(U3-Pad12) -> Net-(C17-Pad1)
- U3 pad 7: Net-(U3-Pad12) -> Net-(C19-Pad1)
- U3 pad 8: (no net) -> Net-(C24-Pad1)
- U3 pad 9: (no net) -> Net-(C23-Pad1)
- U4 pad 1: Net-(C2-Pad1) -> Net-(R24-Pad1)
- U4 pad 2: GND -> Net-(R22-Pad1)
- U4 pad 3: GND -> Net-(U4-Pad12)
- U4 pad 4: /PHOTO_K -> +3V3
- U4 pad 5: +5V -> Net-(C21-Pad1)
Other:
- board text removed: "GND"

Commit message: Arduino Zero Shield v1.0 layout done.
Parts:
- J1, J2: footprint Wickerlib:CONN-HEADER-STRAIGHT-P2.54MM-1x02 -> Wickerlib:CONN-ONSHORE-SCREW-GREEN-2PIN-TH
- U1: value MCP6001 -> MCP6004; footprint Wickerlib:SOT-23-5 -> Wickerlib:SOIC-14-3.9x8.7MM-P1.27MM
- U3: value MCP6004 -> TLV274
- U4: value TLV274 -> MCP6001; footprint Wickerlib:SOIC-14-3.9x8.7MM-P1.27MM -> Wickerlib:SOT-23-5
- moved U2 70.4 mm to (79.9, 136.7), turned to 180 degrees
- moved U1 66.6 mm to (65.0, 149.5)
- moved R27 44.7 mm to (87.4, 143.7), turned to 270 degrees
- moved R29 42.9 mm to (85.7, 143.6), turned to 270 degrees
- moved R30 37.7 mm to (83.0, 142.8), turned to 0 degrees
- moved C28 36.8 mm to (84.8, 140.2), turned to 90 degrees
- moved R6 34.7 mm to (79.7, 142.8), turned to 0 degrees
- moved C1 34.7 mm to (51.8, 133.3)
- moved C27 34.2 mm to (76.0, 153.2), turned to 90 degrees
- moved R8 34.2 mm to (76.4, 144.6), turned to 0 degrees
- moved C29 34.0 mm to (85.0, 136.6), turned to 90 degrees
- moved C18 33.4 mm to (86.6, 132.9), turned to 270 degrees
- moved R25 32.2 mm to (75.0, 156.9), turned to 180 degrees
- moved C8 32.0 mm to (76.3, 142.8), turned to 180 degrees
- moved R15 31.2 mm to (84.8, 132.9), turned to 270 degrees
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Connections:
- C22 pad 1: /A0 -> /A2
- R18 pad 2: /A0 -> /A2
- R19 pad 1: /A0 -> /A2
- R22 pad 2: /A0 -> /A2
- R28 pad 1: /A2 -> /A0
- U1 pad 1: Net-(C2-Pad1) -> Net-(C13-Pad1)
- U1 pad 2: GND -> Net-(C11-Pad1)
- U1 pad 3: GND -> /VREF
- U1 pad 4: /PHOTO_K -> +5V
- U1 pad 5: +5V -> /VREF
- U2 pad 1: Net-(C13-Pad1) -> Net-(C28-Pad1)
- U2 pad 12: Net-(C4-Pad1) -> /VREF
- U2 pad 13: Net-(R7-Pad2) -> Net-(C8-Pad2)
- U2 pad 14: Net-(R7-Pad2) -> Net-(C8-Pad1)
- U2 pad 2: Net-(C11-Pad1) -> Net-(C28-Pad2)
- U2 pad 6: Net-(C8-Pad2) -> Net-(C18-Pad2)
- U2 pad 7: Net-(C8-Pad1) -> /LINE_IN
- U3 pad 1: Net-(C28-Pad1) -> Net-(R24-Pad1)
- U3 pad 10: /VREF -> (no net)
- U3 pad 12: /VREF -> Net-(U3-Pad12)
- U3 pad 13: Net-(C18-Pad2) -> /A1
- U3 pad 14: /LINE_IN -> /A0
- U3 pad 2: Net-(C28-Pad2) -> Net-(R22-Pad1)
- U3 pad 3: /VREF -> Net-(U3-Pad12)
- U3 pad 4: +5V -> +3V3
- U3 pad 5: /VREF -> Net-(C21-Pad1)
- U3 pad 6: Net-(C17-Pad1) -> Net-(U3-Pad12)
- U3 pad 7: Net-(C19-Pad1) -> Net-(U3-Pad12)
- U3 pad 8: Net-(C24-Pad1) -> (no net)
- U3 pad 9: Net-(C23-Pad1) -> (no net)
- U4 pad 1: Net-(R24-Pad1) -> Net-(C2-Pad1)
- U4 pad 2: Net-(R22-Pad1) -> GND
- U4 pad 3: Net-(U4-Pad12) -> GND
- U4 pad 4: +3V3 -> /PHOTO_K
- U4 pad 5: Net-(C21-Pad1) -> +5V
Routing:
- net +5V: track 0.00 -> 123.1 mm, vias 0 -> 6
- net /VREF: track 0.00 -> 86.1 mm, vias 0 -> 2
- net GND: track 0.00 -> 45.7 mm, vias 0 -> 18
- net +3V3: track 0.00 -> 32.9 mm
- net /LINE_IN: track 0.00 -> 24.0 mm
- net /A2: track 0.00 -> 23.9 mm
- net Net-(C27-Pad1): track 0.00 -> 22.7 mm
- net /PHOTO_K: track 0.00 -> 19.0 mm
- net /A1: track 0.00 -> 18.7 mm
- net Net-(C11-Pad2): track 0.00 -> 16.7 mm
- net Net-(C10-Pad1): track 0.00 -> 16.4 mm
- net /A0: track 0.00 -> 16.1 mm
- net Net-(C5-Pad1): track 0.00 -> 15.3 mm
- net Net-(R31-Pad2): track 0.00 -> 14.5 mm
- net Net-(C13-Pad1): track 0.00 -> 14.0 mm
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Other:
- board outline added: 70.9 x 53.3 mm
- board text added: "+ -"
- board text added: "- +"
- board text added: "DETECTORS"
- board text added: "EMITTERS"
- board text added: "RESET"
- board text added: "VREF"
- board text removed: "5V VA A2 A1 A0 AG"
- board text removed: "AGND"
- board text removed: "SIGIN"

Commit message: Add datasheet. Fix footprint.
Parts:
- C16, C17, C19, C22: footprint Wickerlib:RLC-1210-SMD -> Wickerlib:RLC-0805-SMD
