File: hardware/mcphail-zero-analog-shield/mcphail-zero-analog-shield.sch (KiCad schematic (older format))
At the start: 72 parts, among them J1 INSECT DETECTION, J2 EMITTERS, J3 VREF, U1 HOLE, U2 HOLE, U3 TLV274, U4 MCP6001, U5 ARDUINO-101-SHIELD, U6 MCP6004, U7 MCP6004, U8 HOLE, U9 HOLE

Commit message: Schematic ref des seems okay.
Parts:
- added LED1: AMBER, Wickerlib:LED-0603-SMD, symbol LED-AMBER-0603-SMT-L296-Q2R2
- added R32: 220, Wickerlib:RLC-0603-SMD, symbol RES-220-5%-1/10W-0603
- added S1: RESET, Wickerlib:SWITCH-OMRON-MOMENTARY-SMD-B3U-1000P, symbol SWITCH-MOMENT-SPST-NO-0.05A-12V-SMT-B3U-1000P
- renumbered U5 to U10, U8 to U11, U9 to U12, U2 to U13, U1 to U14
Connections:
- net labels removed: A3, A4, A5, AGND, D0, D1, D10, D11, D12, D13, D2, D3, D4, D5, D6, D7, D8, D9, IOREF, RESET
- wire segments 234 -> 219
- no-connect marks 1 -> 21

Commit message: Only comps we need left on board. Needs routed.
Parts:
- U11, U12, U13, U14: footprint ARDUINO-MOUNTING-HOLE -> Wickerlib:ARDUINO-MOUNTING-HOLE
Changed lines of the file:
@@
 F 0 "U14" H 15450 3225 50  0001 L CNN
 F 1 "HOLE" V 15400 3275 50  0001 L CNN
-F 2 "ARDUINO-MOUNTING-HOLE" H 15600 3375 50  0001 C CIN
+F 2 "Wickerlib:ARDUINO-MOUNTING-HOLE" H 15600 3375 50  0001 C CIN
 F 3 "https://www.adafruit.com/products/50" H 15600 3725 10  0001 C CNN
 F 4 "Arduino" H 15600 3375 50  0001 C CIN "MF_Name"
@@
 F 0 "U13" H 15350 3225 50  0001 L CNN
 F 1 "HOLE" V 15300 3275 50  0001 L CNN
-F 2 "ARDUINO-MOUNTING-HOLE" H 15500 3375 50  0001 C CIN
+F 2 "Wickerlib:ARDUINO-MOUNTING-HOLE" H 15500 3375 50  0001 C CIN
 F 3 "https://www.adafruit.com/products/50" H 15500 3725 5   0001 C CNN
 F 4 "ARDU-101SHIELD" H 15500 3375 50  0001 C CIN "Package"
@@
 F 0 "U12" H 15250 3225 50  0001 L CNN
 F 1 "HOLE" V 15200 3275 50  0001 L CNN
-F 2 "ARDUINO-MOUNTING-HOLE" H 15400 3375 50  0001 C CIN
+F 2 "Wickerlib:ARDUINO-MOUNTING-HOLE" H 15400 3375 50  0001 C CIN
 F 3 "https://www.adafruit.com/products/50" H 15400 3725 5   0001 C CNN
 F 4 "ARDU-101SHIELD" H 15400 3375 50  0001 C CIN "Package"
@@
 F 0 "U11" H 15150 3225 50  0001 L CNN
 F 1 "HOLE" V 15100 3275 50  0001 L CNN
-F 2 "ARDUINO-MOUNTING-HOLE" H 15300 3375 50  0001 C CIN
+F 2 "Wickerlib:ARDUINO-MOUNTING-HOLE" H 15300 3375 50  0001 C CIN
 F 3 "https://www.adafruit.com/products/50" H 15300 3725 5   0001 C CNN
 F 4 "ARDU-101SHIELD" H 15300 3375 50  0001 C CIN "Package"

Commit message: Parts on board with no traces, clean. Ready to layout.
Parts:
- removed U11, U12, U13, U14: HOLE, Wickerlib:ARDUINO-MOUNTING-HOLE, symbol ARDUINO-101-SHIELD
Other:
- note removed: "Arduino Zero Shield\nMounting Holes"
Changed lines of the file:
@@
 $EndDescr
-$Comp
-L ARDUINO-101-SHIELD U14
-U 5 1 57282130
-P 15600 3725
-F 0 "U14" H 15450 3225 50  0001 L CNN
-F 1 "HOLE" V 15400 3275 50  0001 L CNN
-F 2 "Wickerlib:ARDUINO-MOUNTING-HOLE" H 15600 3375 50  0001 C CIN
-F 3 "https://www.adafruit.com/products/50" H 15600 3725 10  0001 C CNN
-F 4 "Arduino" H 15600 3375 50  0001 C CIN "MF_Name"
-F 5 "101" H 15600 3375 50  0001 C CIN "MF_PN"
-F 6 "Adafruit" H 15600 3375 50  0001 C CIN "S1_Name"
-F 7 "50" H 15600 3375 50  0001 C CIN "S1_PN"
-F 8 "ARDUINO 101" H 15600 3375 50  0001 C CIN "Description"
-	5    15600 3725
-	-1   0    0    -1
-$EndComp
-Text Notes 15700 3475 2    60   ~ 0
-Arduino Zero Shield\nMounting Holes
-$Comp
-L ARDUINO-101-SHIELD U13
-U 5 1 57290D61
-P 15500 3725
-F 0 "U13" H 15350 3225 50  0001 L CNN
-F 1 "HOLE" V 15300 3275 50  0001 L CNN
-F 2 "Wickerlib:ARDUINO-MOUNTING-HOLE" H 15500 3375 50  0001 C CIN
-F 3 "https://www.adafruit.com/products/50" H 15500 3725 5   0001 C CNN
-F 4 "ARDU-101SHIELD" H 15500 3375 50  0001 C CIN "Package"
-F 5 "Arduino" H 15500 3375 50  0001 C CIN "MF_Name"
-F 6 "101" H 15500 3375 50  0001 C CIN "MF_PN"
-F 7 "Adafruit" H 15500 3375 50  0001 C CIN "S1_Name"
-F 8 "50" H 15500 3375 50  0001 C CIN "S1_PN"
-F 9 "ARDUINO 101" H 15500 3375 50  0001 C CIN "Description"
-F 10 "Not Verified" H 15500 3375 50  0001 C CIN "Verified"
-	5    15500 3725
-	-1   0    0    -1
-$EndComp
-$Comp
-L ARDUINO-101-SHIELD U12
-U 5 1 57290D9E
-P 15400 3725
-F 0 "U12" H 15250 3225 50  0001 L CNN
-F 1 "HOLE" V 15200 3275 50  0001 L CNN
-F 2 "Wickerlib:ARDUINO-MOUNTING-HOLE" H 15400 3375 50  0001 C CIN
-F 3 "https://www.adafruit.com/products/50" H 15400 3725 5   0001 C CNN
-F 4 "ARDU-101SHIELD" H 15400 3375 50  0001 C CIN "Package"
-F 5 "Arduino" H 15400 3375 50  0001 C CIN "MF_Name"
-F 6 "101" H 15400 3375 50  0001 C CIN "MF_PN"
-F 7 "Adafruit" H 15400 3375 50  0001 C CIN "S1_Name"
-F 8 "50" H 15400 3375 50  0001 C CIN "S1_PN"
-F 9 "ARDUINO 101" H 15400 3375 50  0001 C CIN "Description"
-F 10 "Not Verified" H 15400 3375 50  0001 C CIN "Verified"
-	5    15400 3725
-	-1   0    0    -1
-$EndComp
-$Comp
-L ARDUINO-101-SHIELD U11
-U 5 1 57290DDB
-P 15300 3725
-F 0 "U11" H 15150 3225 50  0001 L CNN
-F 1 "HOLE" V 15100 3275 50  0001 L CNN
-F 2 "Wickerlib:ARDUINO-MOUNTING-HOLE" H 15300 3375 50  0001 C CIN
-F 3 "https://www.adafruit.com/products/50" H 15300 3725 5   0001 C CNN
-F 4 "ARDU-101SHIELD" H 15300 3375 50  0001 C CIN "Package"
-F 5 "Arduino" H 15300 3375 50  0001 C CIN "MF_Name"
-F 6 "101" H 15300 3375 50  0001 C CIN "MF_PN"
-F 7 "Adafruit" H 15300 3375 50  0001 C CIN "S1_Name"
-F 8 "50" H 15300 3375 50  0001 C CIN "S1_PN"
-F 9 "ARDUINO 101" H 15300 3375 50  0001 C CIN "Description"
-F 10 "Not Verified" H 15300 3375 50  0001 C CIN "Verified"
-	5    15300 3725
-	-1   0    0    -1
-$EndComp
 $Comp
 L +5V #PWR01

Commit message: Re-import netlist, override existing.
Parts:
- renumbered U4 to U1, U6 to U2, U7 to U3, U3 to U4, U10 to U5
Changed lines of the file:
@@
 $EndComp
 $Comp
-L ARDUINO-101-SHIELD U10
+L ARDUINO-101-SHIELD U5
 U 1 1 572986CB
 P 15550 4875
-F 0 "U10" H 15400 4375 50  0000 L CNN
+F 0 "U5" H 15400 4375 50  0000 L CNN
 F 1 "ARDUINO-101-SHIELD" V 15350 4425 50  0001 L CNN
 F 2 "Wickerlib:ARDUINO-UNO-SHIELD" H 15550 4525 50  0001 C CIN
@@
 $EndComp
 $Comp
-L ARDUINO-101-SHIELD U10
+L ARDUINO-101-SHIELD U5
 U 2 1 572988F2
 P 15550 5775
-F 0 "U10" H 15400 5275 50  0000 L CNN
+F 0 "U5" H 15400 5275 50  0000 L CNN
 F 1 "ARDUINO-101-SHIELD" V 15350 5325 50  0001 L CNN
 F 2 "Wickerlib:ARDUINO-UNO-SHIELD" H 15550 5425 50  0001 C CIN
@@
 $EndComp
 $Comp
-L ARDUINO-101-SHIELD U10
+L ARDUINO-101-SHIELD U5
 U 3 1 57298950
 P 15550 6875
-F 0 "U10" H 15400 6375 50  0000 L CNN
+F 0 "U5" H 15400 6375 50  0000 L CNN
 F 1 "ARDUINO-101-SHIELD" V 15350 6425 50  0001 L CNN
 F 2 "Wickerlib:ARDUINO-UNO-SHIELD" H 15550 6525 50  0001 C CIN
@@
 $EndComp
 $Comp
-L ARDUINO-101-SHIELD U10
+L ARDUINO-101-SHIELD U5
 U 4 1 572989D0
 P 15550 8150
-F 0 "U10" H 15400 7650 50  0000 L CNN
+F 0 "U5" H 15400 7650 50  0000 L CNN
 F 1 "ARDUINO-101-SHIELD" V 15350 7700 50  0001 L CNN
 F 2 "Wickerlib:ARDUINO-UNO-SHIELD" H 15550 7800 50  0001 C CIN
@@
 $EndComp
 $Comp
-L IC-OPAMP-QUAD-MCP6004-SOIC14 U6
+L IC-OPAMP-QUAD-MCP6004-SOIC14 U2
 U 1 1 596FCA3F
 P 6550 3975
-AR Path="/596FCA3F" Ref="U6"  Part="1"
-AR Path="/596F9466/596FCA3F" Ref="U1"  Part="1"
-F 0 "U6" H 6600 4125 50  0000 L CNN
+AR Path="/596FCA3F" Ref="U2"  Part="1"
+AR Path="/596F9466/596FCA3F" Ref="U?"  Part="1"
+F 0 "U2" H 6600 4125 50  0000 L CNN
 F 1 "MCP6004" H 6600 3825 50  0000 L CNN
 F 2 "Wickerlib:SOIC-14-3.9x8.7MM-P1.27MM" H 6550 3625 50  0001 C CIN
@@
 $EndComp
 $Comp
-L IC-OPAMP-QUAD-MCP6004-SOIC14 U7
+L IC-OPAMP-QUAD-MCP6004-SOIC14 U3
 U 2 1 596FCA4B
 P 8325 3975
-AR Path="/596FCA4B" Ref="U7"  Part="2"
-AR Path="/596F9466/596FCA4B" Ref="U1"  Part="2"
-F 0 "U7" H 8375 4125 50  0000 L CNN
+AR Path="/596FCA4B" Ref="U3"  Part="2"
+AR Path="/596F9466/596FCA4B" Ref="U?"  Part="2"
+F 0 "U3" H 8375 4125 50  0000 L CNN
 F 1 "MCP6004" H 8375 3825 50  0000 L CNN
 F 2 "Wickerlib:SOIC-14-3.9x8.7MM-P1.27MM" H 8325 3625 50  0001 C CIN
@@
 $EndComp
 $Comp
-L IC-OPAMP-QUAD-MCP6004-SOIC14 U7
+L IC-OPAMP-QUAD-MCP6004-SOIC14 U3
 U 3 1 596FCB0B
 P 10025 3975
-AR Path="/596FCB0B" Ref="U7"  Part="3"
-AR Path="/596F9466/596FCB0B" Ref="U1"  Part="3"
-F 0 "U7" H 10075 4125 50  0000 L CNN
+AR Path="/596FCB0B" Ref="U3"  Part="3"
+AR Path="/596F9466/596FCB0B" Ref="U?"  Part="3"
+F 0 "U3" H 10075 4125 50  0000 L CNN
 F 1 "MCP6004" H 10075 3825 50  0000 L CNN
 F 2 "Wickerlib:SOIC-14-3.9x8.7MM-P1.27MM" H 10025 3625 50  0001 C CIN
@@
 VREF
 $Comp
-L IC-OPAMP-QUAD-MCP6004-SOIC14 U6
+L IC-OPAMP-QUAD-MCP6004-SOIC14 U2
 U 4 1 596FCB31
 P 4525 4675
-AR Path="/596FCB31" Ref="U6"  Part="4"
-AR Path="/596F9466/596FCB31" Ref="U1"  Part="4"
-F 0 "U6" H 4575 4825 50  0000 L CNN
+AR Path="/596FCB31" Ref="U2"  Part="4"
+AR Path="/596F9466/596FCB31" Ref="U?"  Part="4"
+F 0 "U2" H 4575 4825 50  0000 L CNN
 F 1 "MCP6004" H 4575 4525 50  0000 L CNN
 F 2 "Wickerlib:SOIC-14-3.9x8.7MM-P1.27MM" H 4525 4325 50  0001 C CIN
@@
 $EndComp
 $Comp
-L IC-OPAMP-QUAD-MCP6004-SOIC14 U7
+L IC-OPAMP-QUAD-MCP6004-SOIC14 U3
 U 1 1 596FEA2E
 P 12425 3975
-AR Path="/596FEA2E" Ref="U7"  Part="1"
-AR Path="/596F9466/596FEA2E" Ref="U2"  Part="1"
-F 0 "U7" H 12475 4125 50  0000 L CNN
+AR Path="/596FEA2E" Ref="U3"  Part="1"
+AR Path="/596F9466/596FEA2E" Ref="U?"  Part="1"
+F 0 "U3" H 12475 4125 50  0000 L CNN
 F 1 "MCP6004" H 12475 3825 50  0000 L CNN
 F 2 "Wickerlib:SOIC-14-3.9x8.7MM-P1.27MM" H 12425 3625 50  0001 C CIN
@@
 $EndComp
 $Comp
-L IC-OPAMP-QUAD-MCP6004-SOIC14 U6
+L IC-OPAMP-QUAD-MCP6004-SOIC14 U2
 U 2 1 596FEB1E
 P 4850 7500
-AR Path="/596FEB1E" Ref="U6"  Part="2"
-AR Path="/596F9466/596FEB1E" Ref="U2"  Part="4"
-F 0 "U6" H 4900 7650 50  0000 L CNN
+AR Path="/596FEB1E" Ref="U2"  Part="2"
+AR Path="/596F9466/596FEB1E" Ref="U?"  Part="4"
+F 0 "U2" H 4900 7650 50  0000 L CNN
 F 1 "MCP6004" H 4900 7350 50  0000 L CNN
 F 2 "Wickerlib:SOIC-14-3.9x8.7MM-P1.27MM" H 4850 7150 50  0001 C CIN
@@
 $EndComp
 $Comp
-L IC-OPAMP-QUAD-MCP6004-SOIC14 U6
+L IC-OPAMP-QUAD-MCP6004-SOIC14 U2
 U 3 1 596FEBC9
 P 6500 7525
-AR Path="/596FEBC9" Ref="U6"  Part="3"
-AR Path="/596F9466/596FEBC9" Ref="U2"  Part="3"
-F 0 "U6" H 6550 7675 50  0000 L CNN
+AR Path="/596FEBC9" Ref="U2"  Part="3"
+AR Path="/596F9466/596FEBC9" Ref="U?"  Part="3"
+F 0 "U2" H 6550 7675 50  0000 L CNN
 F 1 "MCP6004" H 6550 7375 50  0000 L CNN
 F 2 "Wickerlib:SOIC-14-3.9x8.7MM-P1.27MM" H 6500 7175 50  0001 C CIN
@@
 $EndComp
 $Comp
-L IC-OPAMP-QUAD-MCP6004-SOIC14 U7
+L IC-OPAMP-QUAD-MCP6004-SOIC14 U3
 U 4 1 596FEC6B
 P 8125 7975
-AR Path="/596FEC6B" Ref="U7"  Part="4"
-AR Path="/596F9466/596FEC6B" Ref="U2"  Part="2"
-F 0 "U7" H 8175 8125 50  0000 L CNN
+AR Path="/596FEC6B" Ref="U3"  Part="4"
+AR Path="/596F9466/596FEC6B" Ref="U?"  Part="2"
+F 0 "U3" H 8175 8125 50  0000 L CNN
 F 1 "MCP6004" H 8175 7825 50  0000 L CNN
 F 2 "Wickerlib:SOIC-14-3.9x8.7MM-P1.27MM" H 8125 7625 50  0001 C CIN
@@
 Photodiode \nConditioned \nOutput
 $Comp
-L IC-OPAMP-QUAD-TLV274-SOIC14 U3
+L IC-OPAMP-QUAD-TLV274-SOIC14 U4
 U 1 1 59722096
 P 10425 7875
-F 0 "U3" H 10475 8025 50  0000 L CNN
+F 0 "U4" H 10475 8025 50  0000 L CNN
 F 1 "TLV274" H 10475 7725 50  0000 L CNN
 F 2 "Wickerlib:SOIC-14-3.9x8.7MM-P1.27MM" H 10425 7525 50  0001 C CIN
@@
 $EndComp
 $Comp
-L IC-OPAMP-QUAD-TLV274-SOIC14 U3
+L IC-OPAMP-QUAD-TLV274-SOIC14 U4
 U 2 1 597222BE
 P 10650 6475
-F 0 "U3" H 10700 6625 50  0000 L CNN
+F 0 "U4" H 10700 6625 50  0000 L CNN
 F 1 "TLV274" H 10700 6325 50  0000 L CNN
 F 2 "Wickerlib:SOIC-14-3.9x8.7MM-P1.27MM" H 10650 6125 50  0001 C CIN
@@
 $EndComp
 $Comp
-L IC-OPAMP-QUAD-TLV274-SOIC14 U3
+L IC-OPAMP-QUAD-TLV274-SOIC14 U4
 U 4 1 59722405
 P 11825 7925
-F 0 "U3" H 11875 8075 50  0000 L CNN
+F 0 "U4" H 11875 8075 50  0000 L CNN
 F 1 "TLV274" H 11875 7775 50  0000 L CNN
 F 2 "Wickerlib:SOIC-14-3.9x8.7MM-P1.27MM" H 11825 7575 50  0001 C CIN
@@
 VREF
 $Comp
-L IC-OPAMP-MCP6001SOT-23-5 U4
+L IC-OPAMP-MCP6001SOT-23-5 U1
 U 1 1 59818A3C
 P 2725 3350
-F 0 "U4" H 2775 3500 50  0000 L CNN
+F 0 "U1" H 2775 3500 50  0000 L CNN
 F 1 "MCP6001" H 2775 3200 50  0000 L CNN
 F 2 "Wickerlib:SOT-23-5" H 2725 3000 50  0001 C CIN

Commit message: Arduino Zero Shield v1.0 layout done.
Parts:
- removed J1: INSECT DETECTION, Wickerlib:CONN-HEADER-STRAIGHT-P2.54MM-1x02, symbol HEADER-MALE-2POS-TH-1x02-P0.1IN
- removed J2: EMITTERS, Wickerlib:CONN-HEADER-STRAIGHT-P2.54MM-1x02, symbol HEADER-MALE-2POS-TH-1x02-P0.1IN
- added J1: INSECT DETECTION, Wickerlib:CONN-ONSHORE-SCREW-GREEN-2PIN-TH, symbol CONN-TERM-SCREW-GREEN-2.54MM-2POS-TH
- added J2: EMITTERS, Wickerlib:CONN-ONSHORE-SCREW-GREEN-2PIN-TH, symbol CONN-TERM-SCREW-GREEN-2.54MM-2POS-TH
- renumbered U2 to U1, U3 to U1, U3 to U2, U4 to U3, U1 to U4
Connections:
- net A0: now also R28.1, U3.14; no longer C22.1, R18.2, R19.1, R22.2
- net A2: now also C22.1, R18.2, R19.1, R22.2; no longer R28.1, U3.14
- net GND: now also J1.2 (P2), J2.2 (P2)
- net LINE_IN: now also U2.7; no longer U2.14
- net PHOTO_K: now also J1.1 (P1)
- net VREF: now also U2.12 (+), U2.5 (+); no longer U2.12 (+), U2.5 (+)
- net at C8.2, R5.1: now also U2.13 (-); no longer U2.6 (-)
- net at C8.1, R6.1, R8.2: now also U2.14; no longer U2.7
- net at C18.2, R13.2, R15.2: now also U2.6 (-); no longer U2.13 (-)
- net at R1.2: now also J2.1 (P1)
Other:
- note added: "NOTE: use a jumper \nfrom 5V or 3.3V\n or VREF to AREF\nas appropriate"
- note removed: "Jumper from 5V or 3.3V\n or VREF to AREF"
Changed lines of the file:
@@
 L GND #PWR03
 U 1 1 57283670
-P 15250 8600
-F 0 "#PWR03" H 15250 8350 50  0001 C CNN
-F 1 "GND" H 15250 8450 50  0000 C CNN
-F 2 "" H 15250 8600 50  0000 C CNN
-F 3 "" H 15250 8600 50  0000 C CNN
-	1    15250 8600
+P 14350 8600
+F 0 "#PWR03" H 14350 8350 50  0001 C CNN
+F 1 "GND" H 14350 8450 50  0000 C CNN
+F 2 "" H 14350 8600 50  0000 C CNN
+F 3 "" H 14350 8600 50  0000 C CNN
+	1    14350 8600
 	-1   0    0    -1
 $EndComp
@@
 $EndComp
 $Comp
-L IC-OPAMP-QUAD-MCP6004-SOIC14 U2
+L IC-OPAMP-QUAD-MCP6004-SOIC14 U1
 U 1 1 596FCA3F
 P 6550 3975
-AR Path="/596FCA3F" Ref="U2"  Part="1"
+AR Path="/596FCA3F" Ref="U1"  Part="1"
 AR Path="/596F9466/596FCA3F" Ref="U?"  Part="1"
-F 0 "U2" H 6600 4125 50  0000 L CNN
+F 0 "U1" H 6600 4125 50  0000 L CNN
 F 1 "MCP6004" H 6600 3825 50  0000 L CNN
 F 2 "Wickerlib:SOIC-14-3.9x8.7MM-P1.27MM" H 6550 3625 50  0001 C CIN
@@
 $EndComp
 $Comp
-L IC-OPAMP-QUAD-MCP6004-SOIC14 U3
+L IC-OPAMP-QUAD-MCP6004-SOIC14 U1
 U 2 1 596FCA4B
 P 8325 3975
-AR Path="/596FCA4B" Ref="U3"  Part="2"
+AR Path="/596FCA4B" Ref="U1"  Part="2"
 AR Path="/596F9466/596FCA4B" Ref="U?"  Part="2"
-F 0 "U3" H 8375 4125 50  0000 L CNN
+F 0 "U1" H 8375 4125 50  0000 L CNN
 F 1 "MCP6004" H 8375 3825 50  0000 L CNN
 F 2 "Wickerlib:SOIC-14-3.9x8.7MM-P1.27MM" H 8325 3625 50  0001 C CIN
@@
 $EndComp
 $Comp
-L IC-OPAMP-QUAD-MCP6004-SOIC14 U3
+L IC-OPAMP-QUAD-MCP6004-SOIC14 U1
 U 3 1 596FCB0B
 P 10025 3975
-AR Path="/596FCB0B" Ref="U3"  Part="3"
+AR Path="/596FCB0B" Ref="U1"  Part="3"
 AR Path="/596F9466/596FCB0B" Ref="U?"  Part="3"
-F 0 "U3" H 10075 4125 50  0000 L CNN
+F 0 "U1" H 10075 4125 50  0000 L CNN
 F 1 "MCP6004" H 10075 3825 50  0000 L CNN
 F 2 "Wickerlib:SOIC-14-3.9x8.7MM-P1.27MM" H 10025 3625 50  0001 C CIN
@@
 VREF
 $Comp
-L IC-OPAMP-QUAD-MCP6004-SOIC14 U2
+L IC-OPAMP-QUAD-MCP6004-SOIC14 U1
 U 4 1 596FCB31
 P 4525 4675
-AR Path="/596FCB31" Ref="U2"  Part="4"
+AR Path="/596FCB31" Ref="U1"  Part="4"
 AR Path="/596F9466/596FCB31" Ref="U?"  Part="4"
-F 0 "U2" H 4575 4825 50  0000 L CNN
+F 0 "U1" H 4575 4825 50  0000 L CNN
 F 1 "MCP6004" H 4575 4525 50  0000 L CNN
 F 2 "Wickerlib:SOIC-14-3.9x8.7MM-P1.27MM" H 4525 4325 50  0001 C CIN
@@
 $EndComp
 $Comp
-L IC-OPAMP-QUAD-MCP6004-SOIC14 U3
+L IC-OPAMP-QUAD-MCP6004-SOIC14 U2
 U 1 1 596FEA2E
 P 12425 3975
-AR Path="/596FEA2E" Ref="U3"  Part="1"
+AR Path="/596FEA2E" Ref="U2"  Part="1"
 AR Path="/596F9466/596FEA2E" Ref="U?"  Part="1"
-F 0 "U3" H 12475 4125 50  0000 L CNN
+F 0 "U2" H 12475 4125 50  0000 L CNN
 F 1 "MCP6004" H 12475 3825 50  0000 L CNN
 F 2 "Wickerlib:SOIC-14-3.9x8.7MM-P1.27MM" H 12425 3625 50  0001 C CIN
@@
 $Comp
 L IC-OPAMP-QUAD-MCP6004-SOIC14 U2
-U 2 1 596FEB1E
+U 4 1 596FEB1E
 P 4850 7500
-AR Path="/596FEB1E" Ref="U2"  Part="2"
+AR Path="/596FEB1E" Ref="U2"  Part="4"
 AR Path="/596F9466/596FEB1E" Ref="U?"  Part="4"
 F 0 "U2" H 4900 7650 50  0000 L CNN
@@
 F 7 "Digikey" H 4850 7150 50  0001 C CIN "S1_Name"
 F 8 "MCP6004T-I/SLCT-ND" H 4850 7150 50  0001 C CIN "S1_PN"
-	2    4850 7500
+	4    4850 7500
 	1    0    0    -1
 $EndComp
@@
 $EndComp
 $Comp
-L IC-OPAMP-QUAD-MCP6004-SOIC14 U3
-U 4 1 596FEC6B
+L IC-OPAMP-QUAD-MCP6004-SOIC14 U2
+U 2 1 596FEC6B
 P 8125 7975
-AR Path="/596FEC6B" Ref="U3"  Part="4"
+AR Path="/596FEC6B" Ref="U2"  Part="2"
 AR Path="/596F9466/596FEC6B" Ref="U?"  Part="2"
-F 0 "U3" H 8175 8125 50  0000 L CNN
+F 0 "U2" H 8175 8125 50  0000 L CNN
 F 1 "MCP6004" H 8175 7825 50  0000 L CNN
 F 2 "Wickerlib:SOIC-14-3.9x8.7MM-P1.27MM" H 8125 7625 50  0001 C CIN
@@
 F 7 "Digikey" H 8125 7625 50  0001 C CIN "S1_Name"
 F 8 "MCP6004T-I/SLCT-ND" H 8125 7625 50  0001 C CIN "S1_PN"
-	4    8125 7975
+	2    8125 7975
 	1    0    0    -1
 $EndComp
@@
 Photodiode \nConditioned \nOutput
 $Comp
-L IC-OPAMP-QUAD-TLV274-SOIC14 U4
+L IC-OPAMP-QUAD-TLV274-SOIC14 U3
 U 1 1 59722096
 P 10425 7875
-F 0 "U4" H 10475 8025 50  0000 L CNN
+F 0 "U3" H 10475 8025 50  0000 L CNN
 F 1 "TLV274" H 10475 7725 50  0000 L CNN
 F 2 "Wickerlib:SOIC-14-3.9x8.7MM-P1.27MM" H 10425 7525 50  0001 C CIN
@@
 $EndComp
 $Comp
-L IC-OPAMP-QUAD-TLV274-SOIC14 U4
+L IC-OPAMP-QUAD-TLV274-SOIC14 U3
 U 2 1 597222BE
 P 10650 6475
-F 0 "U4" H 10700 6625 50  0000 L CNN
+F 0 "U3" H 10700 6625 50  0000 L CNN
 F 1 "TLV274" H 10700 6325 50  0000 L CNN
 F 2 "Wickerlib:SOIC-14-3.9x8.7MM-P1.27MM" H 10650 6125 50  0001 C CIN
@@
 $EndComp
 $Comp
-L IC-OPAMP-QUAD-TLV274-SOIC14 U4
+L IC-OPAMP-QUAD-TLV274-SOIC14 U3
 U 4 1 59722405
 P 11825 7925
-F 0 "U4" H 11875 8075 50  0000 L CNN
+F 0 "U3" H 11875 8075 50  0000 L CNN
 F 1 "TLV274" H 11875 7775 50  0000 L CNN
 F 2 "Wickerlib:SOIC-14-3.9x8.7MM-P1.27MM" H 11825 7575 50  0001 C CIN
@@
 $EndComp
 $Comp
-L HEADER-MALE-2POS-TH-1x02-P0.1IN J1
-U 1 1 5974EE73
-P 1175 3200
-F 0 "J1" H 1075 3350 50  0000 L CNN
-F 1 "INSECT DETECTION" H 1075 3050 50  0000 L CNN
-F 2 "Wickerlib:CONN-HEADER-STRAIGHT-P2.54MM-1x02" H 1175 2850 50  0001 C CIN
-F 3 "https://cdn.harwin.com/pdfs/60page140.pdf" H 1125 3200 5   0001 C CNN
-F 4 "HEADER MALE 2POS TH 1x02 0.1IN" H 1175 2850 50  0001 C CIN "Description"
-F 5 "Harwin" H 1175 2850 50  0001 C CIN "MF_Name"
-F 6 "M20-9990246" H 1175 2850 50  0001 C CIN "MF_PN"
-F 7 "Digikey" H 1175 2850 50  0001 C CIN "S1_Name"
-F 8 "952-2262-ND" H 1175 2850 50  0001 C CIN "S1_PN"
-	1    1175 3200
-	1    0    0    -1
-$EndComp
-$Comp
 L +5V #PWR07
 U 1 1 5974FCB7
@@
 Text Notes 875  1025 0    100  ~ 0
 EMITTER\nOUTPUT
-$Comp
-L HEADER-MALE-2POS-TH-1x02-P0.1IN J2
-U 1 1 597520CD
-P 1400 1375
-F 0 "J2" H 1300 1525 50  0000 L CNN
-F 1 "EMITTERS" H 1300 1225 50  0000 L CNN
-F 2 "Wickerlib:CONN-HEADER-STRAIGHT-P2.54MM-1x02" H 1400 1025 50  0001 C CIN
-F 3 "https://cdn.harwin.com/pdfs/60page140.pdf" H 1350 1375 5   0001 C CNN
-F 4 "HEADER MALE 2POS TH 1x02 0.1IN" H 1400 1025 50  0001 C CIN "Description"
-F 5 "Harwin" H 1400 1025 50  0001 C CIN "MF_Name"
-F 6 "M20-9990246" H 1400 1025 50  0001 C CIN "MF_PN"
-F 7 "Digikey" H 1400 1025 50  0001 C CIN "S1_Name"
-F 8 "952-2262-ND" H 1400 1025 50  0001 C CIN "S1_PN"
-	1    1400 1375
-	1    0    0    -1
-$EndComp
 $Comp
 L RES-220-5%-1/10W-0603 R1
@@
 VREF
 $Comp
-L IC-OPAMP-MCP6001SOT-23-5 U1
+L IC-OPAMP-MCP6001SOT-23-5 U4
 U 1 1 59818A3C
 P 2725 3350
-F 0 "U1" H 2775 3500 50  0000 L CNN
+F 0 "U4" H 2775 3500 50  0000 L CNN
 F 1 "MCP6001" H 2775 3200 50  0000 L CNN
 F 2 "Wickerlib:SOT-23-5" H 2725 3000 50  0001 C CIN
@@
 	1    0    0    -1
 $EndComp
-Wire Wire Line
-	13725 8675 13725 5675
 Wire Notes Line
 	4125 4550 4175 4550
@@
 	12400 7925 12400 8475
 Wire Wire Line
-	11825 8475 13925 8475
+	11825 8475 13725 8475
 Connection ~ 12400 8475
 Wire Wire Line
@@
 	9825 8225 9825 8675
 Wire Wire Line
-	9825 8675 13725 8675
+	9825 8675 13925 8675
 Wire Wire Line
 	9825 8225 9525 7975
@@
 	2275 2050 2275 3450
 Wire Wire Line
-	1325 3250 2425 3250
+	1250 3250 2425 3250
 Wire Wire Line
 	1900 3250 1900 3500
@@
 Connection ~ 3500 3350
 Wire Wire Line
-	2275 3150 1325 3150
+	2275 3150 1250 3150
 Connection ~ 2275 3150
 Connection ~ 13025 3975
@@
 Connection ~ 11400 8475
 Wire Wire Line
-	15250 8250 15250 8600
-Wire Wire Line
-	15400 8250 15250 8250
+	14350 8250 14350 8600
+Wire Wire Line
+	15400 8250 14350 8250
 Wire Wire Line
 	13925 5875 15400 5875
@@
 Wire Wire Line
 	13825 8575 13825 5775
-Wire Wire Line
-	13925 8475 13925 5875
 NoConn ~ 15400 8350
-Text Notes 14150 8400 0    50   ~ 0
-Jumper from 5V or 3.3V\n or VREF to AREF
+Text Notes 14575 8800 0    50   ~ 0
+NOTE: use a jumper \nfrom 5V or 3.3V\n or VREF to AREF\nas appropriate
 $Comp
 L HEADER-MALE-1POS-TH-1x01 J3
@@
 	14925 7825 14925 7775
 NoConn ~ 15400 4625
+Wire Notes Line
+	15325 8350 14900 8450
+Wire Wire Line
+	13925 8675 13925 5875
+Wire Wire Line
+	13725 8475 13725 5675
+$Comp
+L CONN-TERM-SCREW-GREEN-2.54MM-2POS-TH J2
+U 1 1 59D6B378
+P 1350 1375
+F 0 "J2" H 1300 1525 50  0000 L CNN
+F 1 "EMITTERS" H 1300 1225 50  0000 L CNN
+F 2 "Wickerlib:CONN-ONSHORE-SCREW-GREEN-2PIN-TH" H 1350 1025 50  0001 C CIN
+F 3 "http://www.on-shore.com/sites/default/files/manuals/ostvnxxa150.pdf" H 1350 1375 5   0001 C CNN
+F 4 "CONN TERM SCREW GREEN 2.54MM 2POS TH" H 1350 1025 50  0001 C CIN "Description"
+F 5 "OnShoreTech" H 1350 1025 50  0001 C CIN "MF_Name"
+F 6 "OSTVN02A150" H 1350 1025 50  0001 C CIN "MF_PN"
+F 7 "Digikey" H 1350 1025 50  0001 C CIN "S1_Name"
+F 8 "ED10561-ND" H 1350 1025 50  0001 C CIN "S1_PN"
+	1    1350 1375
+	1    0    0    -1
+$EndComp
+$Comp
+L CONN-TERM-SCREW-GREEN-2.54MM-2POS-TH J1
+U 1 1 59D6B954
+P 1050 3200
+F 0 "J1" H 1000 3350 50  0000 L CNN
+F 1 "INSECT DETECTION" H 1000 3050 50  0000 L CNN
+F 2 "Wickerlib:CONN-ONSHORE-SCREW-GREEN-2PIN-TH" H 1050 2850 50  0001 C CIN
+F 3 "http://www.on-shore.com/sites/default/files/manuals/ostvnxxa150.pdf" H 1050 3200 5   0001 C CNN
+F 4 "CONN TERM SCREW GREEN 2.54MM 2POS TH" H 1050 2850 50  0001 C CIN "Description"
+F 5 "OnShoreTech" H 1050 2850 50  0001 C CIN "MF_Name"
+F 6 "OSTVN02A150" H 1050 2850 50  0001 C CIN "MF_PN"
+F 7 "Digikey" H 1050 2850 50  0001 C CIN "S1_Name"
+F 8 "ED10561-ND" H 1050 2850 50  0001 C CIN "S1_PN"
+	1    1050 3200
+	1    0    0    -1
+$EndComp
 $EndSCHEMATC
