File: hardware/mcphail-zero-analog-shield/mcphail-zero-analog-shield.sch (KiCad schematic (older format))
At the start: 71 parts, among them J1 INSECT DETECTION, J2 EMITTERS, J3 VREF, U1 MCP6004, U2 MCP6004, U3 TLV274, U4 MCP6001, U5 ARDUINO-101-SHIELD

Commit message: Zero shield v1.0 ready to order.
Parts:
- U5: Description ARDUINO 101 SHIELD -> ARDUINO ZERO SHIELD; MF_PN UNO R3 -> ARDUINO ZERO; S1_PN 50 -> 2843
Other:
- note added: "TEST POINT"
- note removed: "SHEET 2: SIGNAL CONDITIONING"
Changed lines of the file:
@@
 F 3 "https://www.adafruit.com/products/3033" H 15550 4875 5   0001 C CNN
 F 4 "Arduino" H 15550 4525 50  0001 C CIN "MF_Name"
-F 5 "UNO R3" H 15550 4525 50  0001 C CIN "MF_PN"
+F 5 "ARDUINO ZERO" H 15550 4525 50  0001 C CIN "MF_PN"
 F 6 "Adafruit" H 15550 4525 50  0001 C CIN "S1_Name"
-F 7 "50" H 15550 4525 50  0001 C CIN "S1_PN"
-F 8 "ARDUINO 101 SHIELD" H 15550 4525 50  0001 C CIN "Description"
+F 7 "2843" H 15550 4525 50  0001 C CIN "S1_PN"
+F 8 "ARDUINO ZERO SHIELD" H 15550 4525 50  0001 C CIN "Description"
 	1    15550 4875
 	-1   0    0    -1
@@
 F 3 "https://www.adafruit.com/products/3033" H 15550 5775 5   0001 C CNN
 F 4 "Arduino" H 15550 5425 50  0001 C CIN "MF_Name"
-F 5 "UNO R3" H 15550 5425 50  0001 C CIN "MF_PN"
+F 5 "ARDUINO ZERO" H 15550 5425 50  0001 C CIN "MF_PN"
 F 6 "Adafruit" H 15550 5425 50  0001 C CIN "S1_Name"
-F 7 "50" H 15550 5425 50  0001 C CIN "S1_PN"
-F 8 "ARDUINO 101 SHIELD" H 15550 5425 50  0001 C CIN "Description"
+F 7 "2843" H 15550 5425 50  0001 C CIN "S1_PN"
+F 8 "ARDUINO ZERO SHIELD" H 15550 5425 50  0001 C CIN "Description"
 	2    15550 5775
 	-1   0    0    -1
@@
 F 3 "https://www.adafruit.com/products/3033" H 15550 6875 5   0001 C CNN
 F 4 "Arduino" H 15550 6525 50  0001 C CIN "MF_Name"
-F 5 "UNO R3" H 15550 6525 50  0001 C CIN "MF_PN"
+F 5 "ARDUINO ZERO" H 15550 6525 50  0001 C CIN "MF_PN"
 F 6 "Adafruit" H 15550 6525 50  0001 C CIN "S1_Name"
-F 7 "50" H 15550 6525 50  0001 C CIN "S1_PN"
-F 8 "ARDUINO 101 SHIELD" H 15550 6525 50  0001 C CIN "Description"
+F 7 "2843" H 15550 6525 50  0001 C CIN "S1_PN"
+F 8 "ARDUINO ZERO SHIELD" H 15550 6525 50  0001 C CIN "Description"
 	3    15550 6875
 	-1   0    0    -1
@@
 F 3 "https://www.adafruit.com/products/3033" H 15550 8150 5   0001 C CNN
 F 4 "Arduino" H 15550 7800 50  0001 C CIN "MF_Name"
-F 5 "UNO R3" H 15550 7800 50  0001 C CIN "MF_PN"
+F 5 "ARDUINO ZERO" H 15550 7800 50  0001 C CIN "MF_PN"
 F 6 "Adafruit" H 15550 7800 50  0001 C CIN "S1_Name"
-F 7 "50" H 15550 7800 50  0001 C CIN "S1_PN"
-F 8 "ARDUINO 101 SHIELD" H 15550 7800 50  0001 C CIN "Description"
+F 7 "2843" H 15550 7800 50  0001 C CIN "S1_PN"
+F 8 "ARDUINO ZERO SHIELD" H 15550 7800 50  0001 C CIN "Description"
 	4    15550 8150
 	-1   0    0    -1
@@
 	0    1    1    0
 $EndComp
-Text Notes 4400 1425 0    200  ~ 0
-SHEET 2: SIGNAL CONDITIONING
 $Comp
 L CAP-CER-220NF-25V-X7R-0603 C3
@@
 	1    0    0    -1
 $EndComp
+Text Notes 10150 5125 0    50   ~ 0
+TEST POINT
 $EndSCHEMATC

Commit message: Add datasheet. Fix footprint.
Parts:
- C16, C17, C19, C22: footprint Wickerlib:RLC-1210-SMD -> Wickerlib:RLC-0805-SMD
Changed lines of the file:
@@
 F 0 "C16" V 7150 3975 50  0000 C CNN
 F 1 "2.2uF" V 7400 3975 50  0000 C CNN
-F 2 "Wickerlib:RLC-1210-SMD" H 7900 3575 50  0001 C CIN
+F 2 "Wickerlib:RLC-0805-SMD" H 7900 3575 50  0001 C CIN
 F 3 "http://media.digikey.com/pdf/Data%20Sheets/Samsung%20PDFs/CL21B225KAFNFNE_Spec.pdf" H 7625 3750 10  0001 C CNN
 F 4 "CAP CER 2.2UF 25V X7R 0805" H 7950 3650 50  0001 C CIN "Description"
@@
 F 0 "C17" V 7475 4075 50  0000 C CNN
 F 1 "2.2uF" V 7725 4075 50  0000 C CNN
-F 2 "Wickerlib:RLC-1210-SMD" H 8225 3675 50  0001 C CIN
+F 2 "Wickerlib:RLC-0805-SMD" H 8225 3675 50  0001 C CIN
 F 3 "http://media.digikey.com/pdf/Data%20Sheets/Samsung%20PDFs/CL21B225KAFNFNE_Spec.pdf" H 7950 3850 10  0001 C CNN
 F 4 "CAP CER 2.2UF 25V X7R 0805" H 8275 3750 50  0001 C CIN "Description"
@@
 F 0 "C19" V 8075 3000 50  0000 C CNN
 F 1 "2.2uF" V 8325 3000 50  0000 C CNN
-F 2 "Wickerlib:RLC-1210-SMD" H 8825 2600 50  0001 C CIN
+F 2 "Wickerlib:RLC-0805-SMD" H 8825 2600 50  0001 C CIN
 F 3 "http://media.digikey.com/pdf/Data%20Sheets/Samsung%20PDFs/CL21B225KAFNFNE_Spec.pdf" H 8550 2775 10  0001 C CNN
 F 4 "CAP CER 2.2UF 25V X7R 0805" H 8875 2675 50  0001 C CIN "Description"
@@
 F 0 "C22" V 9125 7975 50  0000 C CNN
 F 1 "2.2uF" V 9375 7975 50  0000 C CNN
-F 2 "Wickerlib:RLC-1210-SMD" H 9875 7575 50  0001 C CIN
+F 2 "Wickerlib:RLC-0805-SMD" H 9875 7575 50  0001 C CIN
 F 3 "http://media.digikey.com/pdf/Data%20Sheets/Samsung%20PDFs/CL21B225KAFNFNE_Spec.pdf" H 9600 7750 10  0001 C CNN
 F 4 "CAP CER 2.2UF 25V X7R 0805" H 9925 7650 50  0001 C CIN "Description"
